File: hardware/voltage_input.sch (KiCad schematic (older format))
At the start: 15 parts, among them U2 MP1584EN

Commit message: Implement next hardware revision
Parts:
- removed C4: 10uF, Capacitor_SMD:C_0805_2012Metric_Pad1.15x1.40mm_HandSolder, symbol Device:C
- removed C5: 100nF, Capacitor_SMD:C_0603_1608Metric_Pad1.05x0.95mm_HandSolder, symbol Device:C
- removed C6: 150pF, Capacitor_SMD:C_0603_1608Metric_Pad1.05x0.95mm_HandSolder, symbol Device:C
- removed C7: 47uF, Capacitor_SMD:C_0805_2012Metric_Pad1.15x1.40mm_HandSolder, symbol Device:C
- removed D10: DS34W, Diode_SMD:D_SOD-123F, symbol Device:D_Schottky
- removed L1: 15uH, CSAB0630-100M:INDC6060X300, symbol Device:L
- removed R6, R7: 100k, Resistor_SMD:R_0603_1608Metric_Pad1.05x0.95mm_HandSolder, symbol Device:R
- removed R8: 40.2k, Resistor_SMD:R_0603_1608Metric_Pad1.05x0.95mm_HandSolder, symbol Device:R
- removed R9: 210k, Resistor_SMD:R_0603_1608Metric_Pad1.05x0.95mm_HandSolder, symbol Device:R
- removed U2: MP1584EN, Package_SO:SOIC-8-1EP_3.9x4.9mm_P1.27mm_EP2.35x2.35mm, symbol pi-supercap-ups-rescue:MP1584EN-Custom-raspi-supercap-ups-rescue
- added D?: D_TVS, symbol Device:D_TVS
- R5: value 3k -> 4.7k
Connections:
- net labels removed: BST, COMP, FB, FREQ, SW, Vin
- wire segments 27 -> 7
- no-connect marks 1 -> 0
