File: hardware/voltage_output.sch (KiCad schematic (older format))
At the start: 8 parts, among them U3 MT3608

Commit message: Add an output cap to the MT3608.
Parts:
- added C?: 47uF, Capacitor_SMD:C_0805_2012Metric_Pad1.15x1.40mm_HandSolder, symbol Device:C
Connections:
- wire segments 22 -> 25
Other:
- moved on the sheet: C8
Changed lines of the file:
@@
 L Device:C C?
 U 1 1 5C3482DB
-P 3800 1550
+P 3550 1550
 AR Path="/5C3482DB" Ref="C?"  Part="1"
 AR Path="/5C3480BB/5C3482DB" Ref="C8"  Part="1"
-F 0 "C8" H 3918 1596 50  0000 L CNN
-F 1 "47uF" H 3918 1505 50  0000 L CNN
-F 2 "Capacitor_SMD:C_0805_2012Metric_Pad1.15x1.40mm_HandSolder" H 3838 1400 50  0001 C CNN
-F 3 "~" H 3800 1550 50  0001 C CNN
-	1    3800 1550
+F 0 "C8" H 3668 1596 50  0000 L CNN
+F 1 "47uF" H 3668 1505 50  0000 L CNN
+F 2 "Capacitor_SMD:C_0805_2012Metric_Pad1.15x1.40mm_HandSolder" H 3588 1400 50  0001 C CNN
+F 3 "~" H 3550 1550 50  0001 C CNN
+	1    3550 1550
 	1    0    0    -1
 $EndComp
@@
 L power:GND #PWR?
 U 1 1 5C3482E2
-P 3800 2050
+P 3550 2050
 AR Path="/5C3482E2" Ref="#PWR?"  Part="1"
 AR Path="/5C3480BB/5C3482E2" Ref="#PWR029"  Part="1"
-F 0 "#PWR029" H 3800 1800 50  0001 C CNN
-F 1 "GND" H 3805 1877 50  0000 C CNN
-F 2 "" H 3800 2050 50  0001 C CNN
-F 3 "" H 3800 2050 50  0001 C CNN
-	1    3800 2050
+F 0 "#PWR029" H 3550 1800 50  0001 C CNN
+F 1 "GND" H 3555 1877 50  0000 C CNN
+F 2 "" H 3550 2050 50  0001 C CNN
+F 3 "" H 3550 2050 50  0001 C CNN
+	1    3550 2050
 	1    0    0    -1
 $EndComp
@@
 	3200 2050 3200 2000
 Wire Wire Line
-	3800 2050 3800 1700
-Wire Wire Line
-	3800 1400 3800 1000
+	3550 2050 3550 1700
+Wire Wire Line
+	3550 1400 3550 1000
 Connection ~ 3200 1000
 Wire Wire Line
@@
 Wire Wire Line
 	1050 1000 1700 1000
-Connection ~ 3800 1000
-Wire Wire Line
-	3800 1000 4450 1000
-Wire Wire Line
-	3200 1000 3800 1000
+Wire Wire Line
+	3200 1000 3550 1000
 Text Label 2500 1000 0    50   ~ 0
 SW
 Text Label 2900 1600 0    50   ~ 0
 FB
+Connection ~ 3550 1000
+Wire Wire Line
+	3550 1000 4100 1000
+$Comp
+L Device:C C?
+U 1 1 5C897351
+P 4100 1550
+AR Path="/5C897351" Ref="C?"  Part="1"
+AR Path="/5C3480BB/5C897351" Ref="C?"  Part="1"
+F 0 "C?" H 4218 1596 50  0000 L CNN
+F 1 "47uF" H 4218 1505 50  0000 L CNN
+F 2 "Capacitor_SMD:C_0805_2012Metric_Pad1.15x1.40mm_HandSolder" H 4138 1400 50  0001 C CNN
+F 3 "~" H 4100 1550 50  0001 C CNN
+	1    4100 1550
+	1    0    0    -1
+$EndComp
+$Comp
+L power:GND #PWR?
+U 1 1 5C897357
+P 4100 2050
+AR Path="/5C897357" Ref="#PWR?"  Part="1"
+AR Path="/5C3480BB/5C897357" Ref="#PWR?"  Part="1"
+F 0 "#PWR?" H 4100 1800 50  0001 C CNN
+F 1 "GND" H 4105 1877 50  0000 C CNN
+F 2 "" H 4100 2050 50  0001 C CNN
+F 3 "" H 4100 2050 50  0001 C CNN
+	1    4100 2050
+	1    0    0    -1
+$EndComp
+Wire Wire Line
+	4100 2050 4100 1700
+Wire Wire Line
+	4100 1400 4100 1000
+Connection ~ 4100 1000
+Wire Wire Line
+	4100 1000 4450 1000
 $EndSCHEMATC

Commit message: Implement next hardware revision
Parts:
- L2: value 4.7uH -> 5.6uH
- R12: value 1k -> 2.2k
- U3: symbol pi-supercap-ups-rescue:MT3608-Custom-raspi-supercap-ups-rescue -> pi-supercap-ups:MT3608
Changed lines of the file:
@@
 $Descr A4 11693 8268
 encoding utf-8
-Sheet 5 7
+Sheet 5 8
 Title ""
 Date ""
@@
 AR Path="/5C3480BB/5C359B99" Ref="R12"  Part="1"
 F 0 "R12" H 4520 1396 50  0000 L CNN
-F 1 "1k" H 4520 1305 50  0000 L CNN
+F 1 "2.2k" H 4520 1305 50  0000 L CNN
 F 2 "Resistor_SMD:R_0603_1608Metric_Pad1.05x0.95mm_HandSolder" V 4380 1350 50  0001 C CNN
 F 3 "~" H 4450 1350 50  0001 C CNN
@@
 $EndComp
 $Comp
-L pi-supercap-ups-rescue:MT3608-Custom-raspi-supercap-ups-rescue U3
+L pi-supercap-ups:MT3608 U3
 U 1 1 5C35E3F1
 P 2300 1550
+AR Path="/5C35E3F1" Ref="U3"  Part="1"
+AR Path="/5C3480BB/5C35E3F1" Ref="U3"  Part="1"
 F 0 "U3" H 2300 1865 50  0000 C CNN
 F 1 "MT3608" H 2300 1774 50  0000 C CNN
@@
 P 2250 1000
 F 0 "L2" V 2440 1000 50  0000 C CNN
-F 1 "4.7uH" V 2349 1000 50  0000 C CNN
+F 1 "5.6uH" V 2349 1000 50  0000 C CNN
 F 2 "Inductor_SMD:L_4.5x4.8_H3_Handsolder" H 2250 1000 50  0001 C CNN
 F 3 "~" H 2250 1000 50  0001 C CNN
