File: current_limiting.sch (KiCad schematic (older format))
At the start: 9 parts, among them U6 MT9700, U7 MT9700

Commit message: Rename to Sailor Hat
Parts:
- U6, U7: symbol pi-supercap-ups:MT9700 -> sailor-hat-rescue:MT9700-sailor-hat
Changed lines of the file:
@@
-EESchema Schematic File Version 5
-LIBS:pi-supercap-ups-cache
+EESchema Schematic File Version 4
 EELAYER 30 0
 EELAYER END
@@
 Comment3 ""
 Comment4 ""
-Comment5 ""
-Comment6 ""
-Comment7 ""
-Comment8 ""
-Comment9 ""
 $EndDescr
 Text HLabel 4900 2000 2    50   Output ~ 0
@@
 $EndComp
 $Comp
-L pi-supercap-ups:MT9700 U7
+L sailor-hat-rescue:MT9700-sailor-hat U7
 U 1 1 5D58745D
 P 3200 2350
@@
 	3350 1600 3700 1600
 $Comp
-L pi-supercap-ups:MT9700 U6
+L sailor-hat-rescue:MT9700-sailor-hat U6
 U 1 1 5D58745E
 P 2950 1550
