File: voltage_output.sch (KiCad schematic (older format))
At the start: 9 parts, among them U3 MT3608

Commit message: Rename to Sailor Hat
Parts:
- U3: symbol pi-supercap-ups:MT3608 -> sailor-hat:MT3608
Changed lines of the file:
@@
 EESchema Schematic File Version 4
-LIBS:pi-supercap-ups-cache
+LIBS:sailor-hat-cache
 EELAYER 26 0
 EELAYER END
@@
 $EndComp
 $Comp
-L pi-supercap-ups:MT3608 U3
+L sailor-hat:MT3608 U3
 U 1 1 5C35E3F1
 P 2300 1550
