File: canbus.sch (KiCad schematic (older format))
At the start: 17 parts, among them U5 MCP2515-xST, U6 ISO1050DUB, U7 H7550-H#, Y1 TAXM8M4RFDCET2T

Commit message: Parts updated to match JLCPCB availability
Parts:
- C1, C3: value 22p -> 22pF; LCSC (none) -> C1653
- D14: value SDM10U45-7 -> PSBD521S-40; LCSC (none) -> C168633
- U5: LCSC (none) -> C15193
- U6: LCSC (none) -> C16428
- U7: LCSC (none) -> C277875
- Y1: value TAXM8M4RFDCET2T -> 1C208000BC0R; LCSC C403948 -> C57131
Changed lines of the file:
@@
 F 2 "Package_SO:TSSOP-20_4.4x6.5mm_P0.65mm" H 2750 1450 50  0001 C CIN
 F 3 "http://ww1.microchip.com/downloads/en/DeviceDoc/21801e.pdf" H 2850 1550 50  0001 C CNN
+F 4 "C15193" H 2750 2350 50  0001 C CNN "LCSC"
 	1    2750 2350
 	1    0    0    -1
@@
 P 1550 3250
 F 0 "Y1" H 1744 3296 50  0000 L CNN
-F 1 "TAXM8M4RFDCET2T" H 1744 3205 50  0000 L CNN
+F 1 "1C208000BC0R" H 1744 3205 50  0000 L CNN
 F 2 "Crystal:Crystal_SMD_3225-4Pin_3.2x2.5mm" H 1550 3250 50  0001 C CNN
 F 3 "~" H 1550 3250 50  0001 C CNN
-F 4 "C403948" H 1550 3250 50  0001 C CNN "LCSC"
+F 4 "C57131" H 1550 3250 50  0001 C CNN "LCSC"
 	1    1550 3250
 	1    0    0    -1
@@
 P 1300 3600
 F 0 "C1" H 1050 3650 50  0000 L CNN
-F 1 "22p" H 1050 3550 50  0000 L CNN
+F 1 "22pF" H 1050 3550 50  0000 L CNN
 F 2 "Capacitor_SMD:C_0603_1608Metric" H 1338 3450 50  0001 C CNN
 F 3 "~" H 1300 3600 50  0001 C CNN
-F 4 "" H 1300 3600 50  0001 C CNN "LCSC"
+F 4 "C1653" H 1300 3600 50  0001 C CNN "LCSC"
 	1    1300 3600
 	1    0    0    -1
@@
 P 1800 3600
 F 0 "C3" H 1915 3646 50  0000 L CNN
-F 1 "22p" H 1915 3555 50  0000 L CNN
+F 1 "22pF" H 1915 3555 50  0000 L CNN
 F 2 "Capacitor_SMD:C_0603_1608Metric" H 1838 3450 50  0001 C CNN
 F 3 "~" H 1800 3600 50  0001 C CNN
-F 4 "" H 1800 3600 50  0001 C CNN "LCSC"
+F 4 "C1653" H 1800 3600 50  0001 C CNN "LCSC"
 	1    1800 3600
 	1    0    0    -1
@@
 F 2 "Package_TO_SOT_SMD:SOT-23" H 9500 1975 50  0001 C CIN
 F 3 "" H 9500 1750 50  0001 C CNN
+F 4 "C277875" H 9500 1650 50  0001 C CNN "LCSC"
 	1    9500 1650
 	1    0    0    -1
@@
 P 8300 1550
 F 0 "D14" H 8300 1334 50  0000 C CNN
-F 1 "SDM10U45-7" H 8300 1425 50  0000 C CNN
+F 1 "PSBD521S-40" H 8300 1425 50  0000 C CNN
 F 2 "Diode_SMD:D_SOD-523" H 8300 1550 50  0001 C CNN
 F 3 "~" H 8300 1550 50  0001 C CNN
+F 4 "C168633" H 8300 1550 50  0001 C CNN "LCSC"
 	1    8300 1550
 	-1   0    0    1
@@
 F 2 "Package_SO:SOP-8_6.62x9.15mm_P2.54mm" H 4700 1400 50  0001 C CIN
 F 3 "http://www.ti.com/lit/ds/symlink/iso1050.pdf" H 4700 1700 50  0001 C CNN
+F 4 "C16428" H 4700 1750 50  0001 C CNN "LCSC"
 	1    4700 1750
 	1    0    0    -1
