File: canbus.sch (KiCad schematic (older format))
At the start: 21 parts, among them J801 Screw_Terminal_01x04, U801 RCLAMP0524P-N, U802 H7550-H#, U803 MCP2515-xST, U804 ISO1050DUB, Y801 1C208000CE0Q

Commit message: Redesigned layout to take EMC issues better into account
Parts:
- added TP801: OSC1, TestPoint:TestPoint_Pad_D1.5mm, symbol Connector:TestPoint
- added TP802: CAN_5V, TestPoint:TestPoint_Keystone_5000-5004_Miniature, symbol Connector:TestPoint
- C803, C804: footprint Capacitor_SMD:C_0603_1608Metric -> Capacitor_SMD:C_0402_1005Metric; LCSC C1653 -> C1555
- C806, C807, C808: footprint Capacitor_SMD:C_0603_1608Metric -> Capacitor_SMD:C_0402_1005Metric; LCSC C14663 -> C1525
- J801: footprint custom:TerminalBlock_WJ15EDGRC-3.81-4P -> Connector_Phoenix_MC:PhoenixContact_MC_1,5_4-G-3.81_1x04_P3.81mm_Horizontal
- R802: footprint Resistor_SMD:R_0603_1608Metric -> Resistor_SMD:R_0402_1005Metric; LCSC C25804 -> C25744
- U801: footprint (none) -> Package_DFN_QFN:Diodes_UDFN-10_1.0x2.5mm_P0.5mm
Connections:
- net labels added: +3.3V
- net labels removed: 3.3V
- wire segments 81 -> 92
- no-connect marks 10 -> 6
Changed lines of the file:
@@
 $Descr A4 11693 8268
 encoding utf-8
-Sheet 8 8
+Sheet 8 9
 Title "Sailor Hat for Raspberry Pi"
 Date ""
@@
 F 0 "C803" H 4700 4150 50  0000 L CNN
 F 1 "22pF" H 4700 4050 50  0000 L CNN
-F 2 "Capacitor_SMD:C_0603_1608Metric" H 4988 3950 50  0001 C CNN
+F 2 "Capacitor_SMD:C_0402_1005Metric" H 4988 3950 50  0001 C CNN
 F 3 "~" H 4950 4100 50  0001 C CNN
-F 4 "C1653" H 4950 4100 50  0001 C CNN "LCSC"
+F 4 "C1555" H 4950 4100 50  0001 C CNN "LCSC"
 	1    4950 4100
 	1    0    0    -1
@@
 F 0 "C804" H 5565 4146 50  0000 L CNN
 F 1 "22pF" H 5565 4055 50  0000 L CNN
-F 2 "Capacitor_SMD:C_0603_1608Metric" H 5488 3950 50  0001 C CNN
+F 2 "Capacitor_SMD:C_0402_1005Metric" H 5488 3950 50  0001 C CNN
 F 3 "~" H 5450 4100 50  0001 C CNN
-F 4 "C1653" H 5450 4100 50  0001 C CNN "LCSC"
+F 4 "C1555" H 5450 4100 50  0001 C CNN "LCSC"
 	1    5450 4100
 	1    0    0    -1
@@
 F 0 "R802" V 7093 3450 50  0000 C CNN
 F 1 "10k" V 7184 3450 50  0000 C CNN
-F 2 "Resistor_SMD:R_0603_1608Metric" V 7230 3450 50  0001 C CNN
+F 2 "Resistor_SMD:R_0402_1005Metric" V 7230 3450 50  0001 C CNN
 F 3 "~" H 7300 3450 50  0001 C CNN
-F 4 "C25804" H 7300 3450 50  0001 C CNN "LCSC"
+F 4 "C25744" H 7300 3450 50  0001 C CNN "LCSC"
 	1    7300 3450
 	0    1    1    0
 $EndComp
-Text GLabel 7550 3300 1    50   Input ~ 0
-3.3V
 Wire Wire Line
 	7550 3450 7450 3450
 Wire Wire Line
 	7150 3450 7000 3450
-Text GLabel 6400 1300 1    50   Input ~ 0
-3.3V
 $Comp
 L power:GND #PWR0804
@@
 Wire Wire Line
 	7750 1300 7750 1500
-Text GLabel 7750 1300 1    50   Input ~ 0
-3.3V
 Wire Wire Line
 	7850 2450 7950 2450
@@
 F 0 "C806" H 6715 1596 50  0000 L CNN
 F 1 "100nF" H 6715 1505 50  0000 L CNN
-F 2 "Capacitor_SMD:C_0603_1608Metric" H 6638 1400 50  0001 C CNN
+F 2 "Capacitor_SMD:C_0402_1005Metric" H 6638 1400 50  0001 C CNN
 F 3 "~" H 6600 1550 50  0001 C CNN
-F 4 "C14663" H 6600 1550 50  0001 C CNN "LCSC"
+F 4 "C1525" H 6600 1550 50  0001 C CNN "LCSC"
 	1    6600 1550
 	1    0    0    -1
@@
 F 0 "C807" H 7615 1796 50  0000 L CNN
 F 1 "100nF" H 7615 1705 50  0000 L CNN
-F 2 "Capacitor_SMD:C_0603_1608Metric" H 7538 1600 50  0001 C CNN
+F 2 "Capacitor_SMD:C_0402_1005Metric" H 7538 1600 50  0001 C CNN
 F 3 "~" H 7500 1750 50  0001 C CNN
-F 4 "C14663" H 7500 1750 50  0001 C CNN "LCSC"
+F 4 "C1525" H 7500 1750 50  0001 C CNN "LCSC"
 	1    7500 1750
 	1    0    0    -1
@@
 F 0 "C808" H 9515 2446 50  0000 L CNN
 F 1 "100nF" H 9515 2355 50  0000 L CNN
-F 2 "Capacitor_SMD:C_0603_1608Metric" H 9438 2250 50  0001 C CNN
+F 2 "Capacitor_SMD:C_0402_1005Metric" H 9438 2250 50  0001 C CNN
 F 3 "~" H 9400 2400 50  0001 C CNN
-F 4 "C14663" H 9400 2400 50  0001 C CNN "LCSC"
+F 4 "C1525" H 9400 2400 50  0001 C CNN "LCSC"
 	1    9400 2400
 	1    0    0    -1
@@
 F 0 "J801" H 1320 1225 50  0000 C CNN
 F 1 "Screw_Terminal_01x04" H 1320 1316 50  0000 C CNN
-F 2 "custom:TerminalBlock_WJ15EDGRC-3.81-4P" H 1400 1650 50  0001 C CNN
+F 2 "Connector_Phoenix_MC:PhoenixContact_MC_1,5_4-G-3.81_1x04_P3.81mm_Horizontal" H 1400 1650 50  0001 C CNN
 F 3 "~" H 1400 1650 50  0001 C CNN
 F 4 "C7245" H 1400 1650 50  0001 C CNN "LCSC"
@@
 	5700 6300 5700 6100
 Wire Wire Line
-	5700 6100 5350 6100
+	5700 6100 5550 6100
 Wire Wire Line
 	6000 6100 5700 6100
@@
 F 0 "U801" H 2950 2825 50  0000 C CNN
 F 1 "RCLAMP0524P-N" H 2950 2734 50  0000 C CNN
-F 2 "" H 2950 2300 50  0001 C CNN
+F 2 "Package_DFN_QFN:Diodes_UDFN-10_1.0x2.5mm_P0.5mm" H 2950 2300 50  0001 C CNN
 F 3 "" H 2950 2300 50  0001 C CNN
 	1    2950 2400
@@
 	1600 1750 2500 1750
 Wire Wire Line
-	1600 1850 2550 1850
-Wire Wire Line
-	3300 2200 3350 2200
-Wire Wire Line
-	3350 2200 3350 1850
-Connection ~ 3350 1850
-Wire Wire Line
-	3350 1850 3500 1850
-Wire Wire Line
 	3300 2300 3400 2300
 Wire Wire Line
-	3400 2300 3400 1750
+	3400 2300 3400 2200
 Connection ~ 3400 1750
 Wire Wire Line
 	3400 1750 3500 1750
 Wire Wire Line
-	2600 2200 2550 2200
-Wire Wire Line
-	2550 2200 2550 1850
-Connection ~ 2550 1850
-Wire Wire Line
-	2550 1850 3350 1850
-Wire Wire Line
 	2600 2300 2500 2300
 Wire Wire Line
-	2500 2300 2500 1750
+	2500 2300 2500 2200
 Connection ~ 2500 1750
 Wire Wire Line
 	2500 1750 3400 1750
-NoConn ~ 3300 2400
-NoConn ~ 3300 2500
-NoConn ~ 2600 2500
-NoConn ~ 2600 2400
 Text Label 2900 2850 3    50   ~ 0
 CAN0_GND
@@
 Wire Wire Line
 	2800 6100 3450 6100
+Wire Wire Line
+	2600 2200 2500 2200
+Connection ~ 2500 2200
+Wire Wire Line
+	2500 2200 2500 1750
+Wire Wire Line
+	1600 1850 2450 1850
+Wire Wire Line
+	3300 2200 3400 2200
+Connection ~ 3400 2200
+Wire Wire Line
+	3400 2200 3400 1750
+Wire Wire Line
+	3300 2400 3450 2400
+Wire Wire Line
+	3450 2400 3450 1850
+Connection ~ 3450 1850
+Wire Wire Line
+	3450 1850 3500 1850
+Wire Wire Line
+	3300 2500 3450 2500
+Wire Wire Line
+	3450 2500 3450 2400
+Connection ~ 3450 2400
+Wire Wire Line
+	2600 2500 2450 2500
+Wire Wire Line
+	2450 2500 2450 2400
+Connection ~ 2450 1850
+Wire Wire Line
+	2450 1850 3450 1850
+Wire Wire Line
+	2600 2400 2450 2400
+Connection ~ 2450 2400
+Wire Wire Line
+	2450 2400 2450 1850
+$Comp
+L Connector:TestPoint TP802
+U 1 1 5FB14C6B
+P 5550 6100
+F 0 "TP802" H 5600 6300 50  0000 L CNN
+F 1 "CAN_5V" H 5600 6200 50  0000 L CNN
+F 2 "TestPoint:TestPoint_Keystone_5000-5004_Miniature" H 5750 6100 50  0001 C CNN
+F 3 "~" H 5750 6100 50  0001 C CNN
+	1    5550 6100
+	1    0    0    -1
+$EndComp
+Connection ~ 5550 6100
+Wire Wire Line
+	5550 6100 5350 6100
+$Comp
+L Connector:TestPoint TP801
+U 1 1 5FB18FAE
+P 5350 2900
+F 0 "TP801" H 5408 3018 50  0000 L CNN
+F 1 "OSC1" H 5408 2927 50  0000 L CNN
+F 2 "TestPoint:TestPoint_Pad_D1.5mm" H 5550 2900 50  0001 C CNN
+F 3 "~" H 5550 2900 50  0001 C CNN
+	1    5350 2900
+	1    0    0    -1
+$EndComp
+Wire Wire Line
+	5350 2900 5350 3150
+Wire Wire Line
+	5350 3150 5450 3150
+Connection ~ 5450 3150
+$Comp
+L power:+3.3V #PWR0105
+U 1 1 5FB649C2
+P 7550 3300
+F 0 "#PWR0105" H 7550 3150 50  0001 C CNN
+F 1 "+3.3V" H 7565 3473 50  0000 C CNN
+F 2 "" H 7550 3300 50  0001 C CNN
+F 3 "" H 7550 3300 50  0001 C CNN
+	1    7550 3300
+	1    0    0    -1
+$EndComp
+$Comp
+L power:+3.3V #PWR0106
+U 1 1 5FB6765D
+P 6400 1300
+F 0 "#PWR0106" H 6400 1150 50  0001 C CNN
+F 1 "+3.3V" H 6415 1473 50  0000 C CNN
+F 2 "" H 6400 1300 50  0001 C CNN
+F 3 "" H 6400 1300 50  0001 C CNN
+	1    6400 1300
+	1    0    0    -1
+$EndComp
+$Comp
+L power:+3.3V #PWR0107
+U 1 1 5FB67D37
+P 7750 1300
+F 0 "#PWR0107" H 7750 1150 50  0001 C CNN
+F 1 "+3.3V" H 7765 1473 50  0000 C CNN
+F 2 "" H 7750 1300 50  0001 C CNN
+F 3 "" H 7750 1300 50  0001 C CNN
+	1    7750 1300
+	1    0    0    -1
+$EndComp
 $EndSCHEMATC

Commit message: Change CAN termination jumper to a solder jumper
Parts:
- JP801: footprint Connector_PinHeader_2.54mm:PinHeader_1x02_P2.54mm_Vertical -> custom:SolderJumper-2_P1.3mm_Open_TrianglePad_Narrow; symbol Jumper:Jumper_2_Open -> Jumper:SolderJumper_2_Open
Connections:
- wire segments 92 -> 94
Changed lines of the file:
@@
 	1650 4100 1650 3950
 $Comp
-L Jumper:Jumper_2_Open JP801
+L Jumper:SolderJumper_2_Open JP801
 U 1 1 5C35395F
 P 2300 3750
 F 0 "JP801" H 2300 3893 50  0000 C CNN
 F 1 "Term" H 2300 3894 50  0001 C CNN
-F 2 "Connector_PinHeader_2.54mm:PinHeader_1x02_P2.54mm_Vertical" H 2300 3750 50  0001 C CNN
+F 2 "custom:SolderJumper-2_P1.3mm_Open_TrianglePad_Narrow" H 2300 3750 50  0001 C CNN
 F 3 "~" H 2300 3750 50  0001 C CNN
 	1    2300 3750
@@
 	1    0    0    -1
 $EndComp
+Wire Wire Line
+	2300 3550 2300 3600
+Wire Wire Line
+	2300 3950 2300 3900
 $EndSCHEMATC

Commit message: Add missing LCSC part numbers
Parts:
- U801: LCSC (none) -> C316044
Changed lines of the file:
@@
 F 2 "Package_DFN_QFN:Diodes_UDFN-10_1.0x2.5mm_P0.5mm" H 2950 2300 50  0001 C CNN
 F 3 "" H 2950 2300 50  0001 C CNN
+F 4 "C316044" H 2950 2400 50  0001 C CNN "LCSC"
 	1    2950 2400
 	1    0    0    -1

Commit message: Rename project files to follow the conventions in SH-ESP32
Parts:
- JP801: footprint custom:SolderJumper-2_P1.3mm_Open_TrianglePad_Narrow -> SH-RPi:SolderJumper-2_P1.3mm_Open_TrianglePad_Narrow
- U801: symbol sailor-hat:RCLAMP0524P-N -> SH-RPi:RCLAMP0524P-N
- U802: symbol sailor-hat:HT75xx-1-SOT23 -> SH-RPi:HT75xx-1-SOT23
Changed lines of the file:
@@
 F 0 "JP801" H 2300 3893 50  0000 C CNN
 F 1 "Term" H 2300 3894 50  0001 C CNN
-F 2 "custom:SolderJumper-2_P1.3mm_Open_TrianglePad_Narrow" H 2300 3750 50  0001 C CNN
+F 2 "SH-RPi:SolderJumper-2_P1.3mm_Open_TrianglePad_Narrow" H 2300 3750 50  0001 C CNN
 F 3 "~" H 2300 3750 50  0001 C CNN
 	1    2300 3750
@@
 	1600 1650 2200 1650
 $Comp
-L sailor-hat:HT75xx-1-SOT23 U802
+L SH-RPi:HT75xx-1-SOT23 U802
 U 1 1 5FB27765
 P 5050 6200
@@
 	1850 1550 2200 1550
 $Comp
-L sailor-hat:RCLAMP0524P-N U801
+L SH-RPi:RCLAMP0524P-N U801
 U 1 1 5FB46A7F
 P 2950 2400

Commit message: Extend the PCB size to provide space for an onboard supercapacitor
The PCB was extended to the left by 21mm to provide room for a
18x40mm (max 18x42mm) 50/60F supercapacitor. The supercapacitor
is lodged in a slot on the PCB to provide mechanical stability and limit
the maximum height of the assembly. It now requires 14mm of headroom.

Additionally, the following changes were made:

- the external supercap connector was removed
- the power and CAN connectors were swapped to JST XH
- there is space for a wire link between CAN and power conx
- power protection circuitry was moved to the edge of the board
- 3.3V regulator was moved to improve the layout
- a 100pF cap was added to the boost feedback to improve loop stability
- rectangles were drawn around ground pins on the GPIO connector
Parts:
- added J802: Wire Link, SH-RPi:WireLink_1x02_P2.54mm, symbol Connector_Generic:Conn_01x02
- J801: value Screw_Terminal_01x04 -> JST XH horiz; footprint Connector_Phoenix_MC:PhoenixContact_MC_1,5_4-G-3.81_1x04_P3.81mm_Horizontal -> SH-RPi:Boomelec_XH-4AW_1x04_P2.50mm_Horizontal; symbol Connector:Screw_Terminal_01x04 -> Connector_Generic:Conn_01x04; LCSC C7245 -> C21273
Connections:
- wire segments 94 -> 97
Changed lines of the file:
@@
 Title "Sailor Hat for Raspberry Pi"
 Date ""
-Rev "revL"
+Rev "revM"
 Comp "Hat Laboratories"
 Comment1 "https://creativecommons.org/licenses/by-sa/4.0"
@@
 	9400 2150 8750 2150
 $Comp
-L Connector:Screw_Terminal_01x04 J?
+L Connector_Generic:Conn_01x04 J?
 U 1 1 5FB016D7
 P 1400 1650
@@
 AR Path="/5C348474/5FB016D7" Ref="J801"  Part="1"
 F 0 "J801" H 1320 1225 50  0000 C CNN
-F 1 "Screw_Terminal_01x04" H 1320 1316 50  0000 C CNN
-F 2 "Connector_Phoenix_MC:PhoenixContact_MC_1,5_4-G-3.81_1x04_P3.81mm_Horizontal" H 1400 1650 50  0001 C CNN
+F 1 "JST XH horiz" H 1320 1316 50  0000 C CNN
+F 2 "SH-RPi:Boomelec_XH-4AW_1x04_P2.50mm_Horizontal" H 1400 1650 50  0001 C CNN
 F 3 "~" H 1400 1650 50  0001 C CNN
-F 4 "C7245" H 1400 1650 50  0001 C CNN "LCSC"
+F 4 "C21273" H 1400 1650 50  0001 C CNN "LCSC"
 	1    1400 1650
 	-1   0    0    -1
@@
 L power:PWR_FLAG #FLG?
 U 1 1 5FB016DE
-P 1850 1550
+P 2250 1450
 AR Path="/5FB016DE" Ref="#FLG?"  Part="1"
 AR Path="/5FAD80E5/5FB016DE" Ref="#FLG?"  Part="1"
 AR Path="/5C348474/5FB016DE" Ref="#FLG0801"  Part="1"
-F 0 "#FLG0801" H 1850 1625 50  0001 C CNN
-F 1 "PWR_FLAG" H 1850 1723 50  0000 C CNN
-F 2 "" H 1850 1550 50  0001 C CNN
-F 3 "~" H 1850 1550 50  0001 C CNN
-	1    1850 1550
+F 0 "#FLG0801" H 2250 1525 50  0001 C CNN
+F 1 "PWR_FLAG" H 2250 1623 50  0000 C CNN
+F 2 "" H 2250 1450 50  0001 C CNN
+F 3 "~" H 2250 1450 50  0001 C CNN
+	1    2250 1450
 	1    0    0    -1
 $EndComp
@@
 Text Label 3500 1850 0    50   ~ 0
 CAN0_L
-Text Label 2200 1550 0    50   ~ 0
+Text Label 2450 1650 0    50   ~ 0
 CAN0_12V
-Text Label 2200 1650 0    50   ~ 0
-CAN0_GND
-Wire Wire Line
-	1600 1650 2200 1650
+Text Label 1650 1550 0    50   ~ 0
+CAN0_GND
 $Comp
 L SH-RPi:HT75xx-1-SOT23 U802
@@
 Text Label 6000 6100 0    50   ~ 0
 CAN_5V
-Connection ~ 1850 1550
-Wire Wire Line
-	1850 1550 1600 1550
-Wire Wire Line
-	1850 1550 2200 1550
 $Comp
 L SH-RPi:RCLAMP0524P-N U801
@@
 Wire Wire Line
 	2300 3950 2300 3900
+Wire Wire Line
+	1600 1550 1650 1550
+Wire Wire Line
+	2250 1650 2250 1450
+Connection ~ 2250 1650
+Wire Wire Line
+	2250 1650 2450 1650
+Wire Wire Line
+	1600 1650 2250 1650
+$Comp
+L Connector_Generic:Conn_01x02 J802
+U 1 1 5FD00858
+P 4900 1150
+F 0 "J802" H 4980 1142 50  0000 L CNN
+F 1 "Wire Link" H 4980 1051 50  0000 L CNN
+F 2 "SH-RPi:WireLink_1x02_P2.54mm" H 4900 1150 50  0001 C CNN
+F 3 "~" H 4900 1150 50  0001 C CNN
+	1    4900 1150
+	1    0    0    -1
+$EndComp
+Text Label 4600 1150 2    50   ~ 0
+CAN0_GND
+Wire Wire Line
+	4700 1150 4600 1150
+Text Label 4600 1250 2    50   ~ 0
+CAN0_12V
+Wire Wire Line
+	4700 1250 4600 1250
 $EndSCHEMATC
