File: power_bank.sch (KiCad schematic (older format))
At the start: 7 parts

Commit message: Rename project files to follow the conventions in SH-ESP32
Parts:
- C3, C4, C5, C6: footprint custom:CP_Radial_D10.0mm_P5.00mm_flat -> SH-RPi:CP_Radial_D10.0mm_P5.00mm_flat
Changed lines of the file:
@@
 F 0 "C3" H 3568 2396 50  0000 L CNN
 F 1 "10F" H 3568 2305 50  0000 L CNN
-F 2 "custom:CP_Radial_D10.0mm_P5.00mm_flat" H 3488 2200 50  0001 C CNN
+F 2 "SH-RPi:CP_Radial_D10.0mm_P5.00mm_flat" H 3488 2200 50  0001 C CNN
 F 3 "~" H 3450 2350 50  0001 C CNN
 	1    3450 2350
@@
 F 0 "C4" H 3568 3046 50  0000 L CNN
 F 1 "10F" H 3568 2955 50  0000 L CNN
-F 2 "custom:CP_Radial_D10.0mm_P5.00mm_flat" H 3488 2850 50  0001 C CNN
+F 2 "SH-RPi:CP_Radial_D10.0mm_P5.00mm_flat" H 3488 2850 50  0001 C CNN
 F 3 "~" H 3450 3000 50  0001 C CNN
 	1    3450 3000
@@
 F 0 "C5" H 4168 2396 50  0000 L CNN
 F 1 "10F" H 4168 2305 50  0000 L CNN
-F 2 "custom:CP_Radial_D10.0mm_P5.00mm_flat" H 4088 2200 50  0001 C CNN
+F 2 "SH-RPi:CP_Radial_D10.0mm_P5.00mm_flat" H 4088 2200 50  0001 C CNN
 F 3 "~" H 4050 2350 50  0001 C CNN
 	1    4050 2350
@@
 F 0 "C6" H 4168 3046 50  0000 L CNN
 F 1 "10F" H 4168 2955 50  0000 L CNN
-F 2 "custom:CP_Radial_D10.0mm_P5.00mm_flat" H 4088 2850 50  0001 C CNN
+F 2 "SH-RPi:CP_Radial_D10.0mm_P5.00mm_flat" H 4088 2850 50  0001 C CNN
 F 3 "~" H 4050 3000 50  0001 C CNN
 	1    4050 3000
