File: control_mcu.sch (KiCad schematic (older format))
At the start: 11 parts, among them J601 Conn_02x07_Counter_Clockwise, U601 ATtiny841-SSU

Commit message: Redesigned layout to take EMC issues better into account
Parts:
- C601, C602: footprint Capacitor_SMD:C_0603_1608Metric -> Capacitor_SMD:C_0402_1005Metric; LCSC C14663 -> C1525
- R602: footprint Resistor_SMD:R_0603_1608Metric -> Resistor_SMD:R_0402_1005Metric; LCSC C4190 -> C25879
- R603: footprint Resistor_SMD:R_0603_1608Metric -> Resistor_SMD:R_0402_1005Metric; LCSC C25804 -> C25744
- R604: value 200k -> 300k; footprint Resistor_SMD:R_0603_1608Metric -> Resistor_SMD:R_0402_1005Metric; LCSC C25811 -> C25774
- R605: value 130k -> 200k; footprint Resistor_SMD:R_0603_1608Metric -> Resistor_SMD:R_0402_1005Metric; LCSC C22795 -> C25764
Connections:
- net labels added: +3.3V, VinS
- net labels removed: 3.3V, V12s
Other:
- note added: "Clamp VinS to always\nless than ATT_Vcc"
- note added: "VcapS is scaled from 2.75V to 1.1V\n(this will also drain the cap over time)"
- note added: "VinS scaled to provide 1.1V for 32V input"
- note removed: "Clamp V12s to always\nless than ATT_Vcc"
- note removed: "V12s scaled to provide 1.1V for 32V input"
- note removed: "VcapS is scaled from 2.8V to 1.1V\n(this will also drain the cap over time)"
Changed lines of the file:
@@
 $Descr A4 11693 8268
 encoding utf-8
-Sheet 6 8
+Sheet 6 9
 Title "Sailor Hat for Raspberry Pi"
 Date ""
@@
 	1    0    0    -1
 $EndComp
-Text GLabel 4100 2600 2    50   Input ~ 0
-3.3V
 Wire Wire Line
 	5800 5100 5500 5100
@@
 F 0 "C602" H 4315 3296 50  0000 L CNN
 F 1 "100nF" H 4315 3205 50  0000 L CNN
-F 2 "Capacitor_SMD:C_0603_1608Metric" H 4238 3100 50  0001 C CNN
+F 2 "Capacitor_SMD:C_0402_1005Metric" H 4238 3100 50  0001 C CNN
 F 3 "~" H 4200 3250 50  0001 C CNN
-F 4 "C14663" H 4200 3250 50  0001 C CNN "LCSC"
+F 4 "C1525" H 4200 3250 50  0001 C CNN "LCSC"
 	1    4200 3250
 	1    0    0    -1
@@
 F 0 "R603" H 5570 4896 50  0000 L CNN
 F 1 "10k" H 5570 4805 50  0000 L CNN
-F 2 "Resistor_SMD:R_0603_1608Metric" V 5430 4850 50  0001 C CNN
+F 2 "Resistor_SMD:R_0402_1005Metric" V 5430 4850 50  0001 C CNN
 F 3 "~" H 5500 4850 50  0001 C CNN
-F 4 "C25804" H 5500 4850 50  0001 C CNN "LCSC"
+F 4 "C25744" H 5500 4850 50  0001 C CNN "LCSC"
 	1    5500 4850
 	1    0    0    -1
@@
 	4650 4100 4400 4100
 Text Notes 650  3300 0    50   ~ 0
-Clamp V12s to always\nless than ATT_Vcc
+Clamp VinS to always\nless than ATT_Vcc
 $Comp
 L Device:D_Schottky D601
@@
 ATT_Vcc
 Text Notes 750  4000 0    50   ~ 0
-V12s scaled to provide 1.1V for 32V input
+VinS scaled to provide 1.1V for 32V input
 Wire Wire Line
 	2250 3050 2400 3050
@@
 F 0 "R602" H 2320 3346 50  0000 L CNN
 F 1 "2.2k" H 2320 3255 50  0000 L CNN
-F 2 "Resistor_SMD:R_0603_1608Metric" V 2180 3300 50  0001 C CNN
+F 2 "Resistor_SMD:R_0402_1005Metric" V 2180 3300 50  0001 C CNN
 F 3 "~" H 2250 3300 50  0001 C CNN
-F 4 "C4190" H 2250 3300 50  0001 C CNN "LCSC"
+F 4 "C25879" H 2250 3300 50  0001 C CNN "LCSC"
 	1    2250 3300
 	1    0    0    -1
@@
 F 0 "C601" H 1765 3346 50  0000 L CNN
 F 1 "100nF" H 1765 3255 50  0000 L CNN
-F 2 "Capacitor_SMD:C_0603_1608Metric" H 1688 3150 50  0001 C CNN
+F 2 "Capacitor_SMD:C_0402_1005Metric" H 1688 3150 50  0001 C CNN
 F 3 "~" H 1650 3300 50  0001 C CNN
-F 4 "C14663" H 1650 3300 50  0001 C CNN "LCSC"
+F 4 "C1525" H 1650 3300 50  0001 C CNN "LCSC"
 	1    1650 3300
 	1    0    0    -1
@@
 RESET
 Text Label 6100 1800 0    50   ~ 0
-V12s
+VinS
 $Comp
 L power:GND #PWR?
@@
 	8000 3050 8000 3250
 Text Notes 6350 3650 0    50   ~ 0
-VcapS is scaled from 2.8V to 1.1V\n(this will also drain the cap over time)
+VcapS is scaled from 2.75V to 1.1V\n(this will also drain the cap over time)
 $Comp
 L Device:R R?
@@
 AR Path="/5C33FF90/5FAFDE9B" Ref="R605"  Part="1"
 F 0 "R605" H 8070 3946 50  0000 L CNN
-F 1 "130k" H 8070 3855 50  0000 L CNN
-F 2 "Resistor_SMD:R_0603_1608Metric" V 7930 3900 50  0001 C CNN
+F 1 "200k" H 8070 3855 50  0000 L CNN
+F 2 "Resistor_SMD:R_0402_1005Metric" V 7930 3900 50  0001 C CNN
 F 3 "~" H 8000 3900 50  0001 C CNN
-F 4 "C22795" H 8000 3900 50  0001 C CNN "LCSC"
+F 4 "C25764" H 8000 3900 50  0001 C CNN "LCSC"
 	1    8000 3900
 	1    0    0    -1
@@
 AR Path="/5C33FF90/5FAFDEAF" Ref="R604"  Part="1"
 F 0 "R604" H 8070 3446 50  0000 L CNN
-F 1 "200k" H 8070 3355 50  0000 L CNN
-F 2 "Resistor_SMD:R_0603_1608Metric" V 7930 3400 50  0001 C CNN
+F 1 "300k" H 8070 3355 50  0000 L CNN
+F 2 "Resistor_SMD:R_0402_1005Metric" V 7930 3400 50  0001 C CNN
 F 3 "~" H 8000 3400 50  0001 C CNN
-F 4 "C25811" H 8000 3400 50  0001 C CNN "LCSC"
+F 4 "C25774" H 8000 3400 50  0001 C CNN "LCSC"
 	1    8000 3400
 	1    0    0    -1
@@
 Vcap
 Text Label 2400 3050 0    50   ~ 0
-V12s
+VinS
 Text Label 4650 4000 0    50   ~ 0
-V12s
+VinS
 Text Label 4650 3900 0    50   ~ 0
 PA0
@@
 Text Label 5800 5100 0    50   ~ 0
 RESET
+$Comp
+L power:+3.3V #PWR0102
+U 1 1 5FB5EC9E
+P 4100 2600
+F 0 "#PWR0102" H 4100 2450 50  0001 C CNN
+F 1 "+3.3V" V 4115 2728 50  0000 L CNN
+F 2 "" H 4100 2600 50  0001 C CNN
+F 3 "" H 4100 2600 50  0001 C CNN
+	1    4100 2600
+	0    1    1    0
+$EndComp
 $EndSCHEMATC

Commit message: Add missing LCSC part numbers
Parts:
- J601: LCSC (none) -> C492424
Changed lines of the file:
@@
 F 2 "custom:PinHeader_2x07_P2.54mm_Vertical_CounterClockwise" H 5800 1900 50  0001 C CNN
 F 3 "~" H 5800 1900 50  0001 C CNN
+F 4 "C492424" H 5800 1900 50  0001 C CNN "LCSC"
 	1    5800 1900
 	1    0    0    -1

Commit message: Rename project files to follow the conventions in SH-ESP32
Parts:
- J601: footprint custom:PinHeader_2x07_P2.54mm_Vertical_CounterClockwise -> SH-RPi:PinHeader_2x07_P2.54mm_Vertical_CounterClockwise
Changed lines of the file:
@@
 F 0 "J601" H 5850 2417 50  0000 C CNN
 F 1 "Conn_02x07_Counter_Clockwise" H 5850 2326 50  0000 C CNN
-F 2 "custom:PinHeader_2x07_P2.54mm_Vertical_CounterClockwise" H 5800 1900 50  0001 C CNN
+F 2 "SH-RPi:PinHeader_2x07_P2.54mm_Vertical_CounterClockwise" H 5800 1900 50  0001 C CNN
 F 3 "~" H 5800 1900 50  0001 C CNN
 F 4 "C492424" H 5800 1900 50  0001 C CNN "LCSC"

Commit message: Update the BAT54C part number according to availability
Parts:
- D602: LCSC C375703 -> C37704
Changed lines of the file:
@@
 F 2 "Package_TO_SOT_SMD:SOT-23" H 3875 2725 50  0001 L CNN
 F 3 "http://www.diodes.com/_files/datasheets/ds11005.pdf" H 3720 2600 50  0001 C CNN
-F 4 "C375703" H 3800 2600 50  0001 C CNN "LCSC"
+F 4 "C37704" H 3800 2600 50  0001 C CNN "LCSC"
 	1    3800 2600
 	1    0    0    -1
