File: control_mcu.sch (KiCad schematic (older format))
At the start: 11 parts, among them J601 Conn_02x07_Counter_Clockwise, U601 ATtiny841-SSU

Commit message: Route I2C to unique pins
Also:
- Connect RTC interrupt to ATtiny
- Break out the interrupt pin to a connector for external signaling
Parts:
- added C603: 33pF/50V, Capacitor_SMD:C_0603_1608Metric, symbol Device:C
- added C604: 33pF, Capacitor_SMD:C_0402_1005Metric, symbol Device:C
- added FB601: GZ2012D101TF, Inductor_SMD:L_0805_2012Metric, symbol Device:Ferrite_Bead
- added J602: Conn_01x02, Connector_PinHeader_2.54mm:PinHeader_1x02_P2.54mm_Vertical, symbol Connector_Generic:Conn_01x02
- added R606: 100R, Resistor_SMD:R_0603_1608Metric, symbol Device:R
- added U602: RCLAMP0524P-N, Package_DFN_QFN:Diodes_UDFN-10_1.0x2.5mm_P0.5mm, symbol SH-RPi:RCLAMP0524P-N
Connections:
- net labels added: PB0_CONN, PB0_INT
- net labels removed: PB0
- wire segments 37 -> 54
- no-connect marks 0 -> 4
Changed lines of the file:
@@
 PB2_LED1
 Text Label 5600 1700 2    50   ~ 0
-PB0
+PB0_INT
 Text Label 5600 1800 2    50   ~ 0
 PB1_LED0
@@
 Text Label 4650 3900 0    50   ~ 0
 PA0
-Text Label 4650 4400 0    50   ~ 0
-PA5
-Text Label 4650 4800 0    50   ~ 0
-PB0
 Text Label 3800 3450 2    50   ~ 0
 ATT_Vcc
@@
 	0    1    1    0
 $EndComp
+$Comp
+L SH-RPi:RCLAMP0524P-N U602
+U 1 1 5FD9547B
+P 2200 1700
+F 0 "U602" H 2200 2125 50  0000 C CNN
+F 1 "RCLAMP0524P-N" H 2200 2034 50  0000 C CNN
+F 2 "Package_DFN_QFN:Diodes_UDFN-10_1.0x2.5mm_P0.5mm" H 2200 1600 50  0001 C CNN
+F 3 "" H 2200 1600 50  0001 C CNN
+	1    2200 1700
+	1    0    0    -1
+$EndComp
+$Comp
+L Connector_Generic:Conn_01x02 J602
+U 1 1 5FD961DC
+P 850 1150
+F 0 "J602" H 768 1367 50  0000 C CNN
+F 1 "Conn_01x02" H 768 1276 50  0000 C CNN
+F 2 "Connector_PinHeader_2.54mm:PinHeader_1x02_P2.54mm_Vertical" H 850 1150 50  0001 C CNN
+F 3 "~" H 850 1150 50  0001 C CNN
+	1    850  1150
+	-1   0    0    -1
+$EndComp
+$Comp
+L power:GND #PWR0607
+U 1 1 5FD96F07
+P 1250 1500
+F 0 "#PWR0607" H 1250 1250 50  0001 C CNN
+F 1 "GND" H 1255 1327 50  0000 C CNN
+F 2 "" H 1250 1500 50  0001 C CNN
+F 3 "" H 1250 1500 50  0001 C CNN
+	1    1250 1500
+	1    0    0    -1
+$EndComp
+Wire Wire Line
+	1050 1250 1250 1250
+Wire Wire Line
+	1250 1250 1250 1500
+Wire Wire Line
+	1050 1150 1850 1150
+NoConn ~ 1850 1700
+NoConn ~ 1850 1800
+NoConn ~ 2550 1800
+NoConn ~ 2550 1700
+$Comp
+L power:GND #PWR0608
+U 1 1 5FD9AA4E
+P 2150 2150
+F 0 "#PWR0608" H 2150 1900 50  0001 C CNN
+F 1 "GND" H 2155 1977 50  0000 C CNN
+F 2 "" H 2150 2150 50  0001 C CNN
+F 3 "" H 2150 2150 50  0001 C CNN
+	1    2150 2150
+	1    0    0    -1
+$EndComp
+$Comp
+L power:GND #PWR0609
+U 1 1 5FD9AF64
+P 2250 2150
+F 0 "#PWR0609" H 2250 1900 50  0001 C CNN
+F 1 "GND" H 2255 1977 50  0000 C CNN
+F 2 "" H 2250 2150 50  0001 C CNN
+F 3 "" H 2250 2150 50  0001 C CNN
+	1    2250 2150
+	1    0    0    -1
+$EndComp
+Wire Wire Line
+	2550 1150 3000 1150
+Text Label 4650 4400 0    50   ~ 0
+PA5
+Text HLabel 4650 4800 2    50   Input ~ 0
+PB0_INT
+Text Label 2000 1150 0    50   ~ 0
+PB0_CONN
+Wire Wire Line
+	2550 1150 1850 1150
+Connection ~ 2550 1150
+Connection ~ 1850 1150
+Wire Wire Line
+	1850 1600 1850 1500
+Connection ~ 1850 1500
+Wire Wire Line
+	1850 1150 1850 1500
+Wire Wire Line
+	2550 1150 2550 1500
+Connection ~ 2550 1500
+Wire Wire Line
+	2550 1500 2550 1600
+$Comp
+L Device:C C603
+U 1 1 5FDA159A
+P 3000 1500
+F 0 "C603" H 3115 1546 50  0000 L CNN
+F 1 "33pF/50V" H 3115 1455 50  0000 L CNN
+F 2 "Capacitor_SMD:C_0603_1608Metric" H 3038 1350 50  0001 C CNN
+F 3 "~" H 3000 1500 50  0001 C CNN
+F 4 "C1663" H 3000 1500 50  0001 C CNN "LCSC"
+	1    3000 1500
+	1    0    0    -1
+$EndComp
+$Comp
+L Device:C C604
+U 1 1 5FDA1F07
+P 3600 1500
+F 0 "C604" H 3715 1546 50  0000 L CNN
+F 1 "33pF" H 3715 1455 50  0000 L CNN
+F 2 "Capacitor_SMD:C_0402_1005Metric" H 3638 1350 50  0001 C CNN
+F 3 "~" H 3600 1500 50  0001 C CNN
+F 4 "C1562" H 3600 1500 50  0001 C CNN "LCSC"
+	1    3600 1500
+	1    0    0    -1
+$EndComp
+$Comp
+L Device:Ferrite_Bead FB601
+U 1 1 5FDA284B
+P 3300 1150
+F 0 "FB601" V 3026 1150 50  0000 C CNN
+F 1 "GZ2012D101TF" V 3117 1150 50  0000 C CNN
+F 2 "Inductor_SMD:L_0805_2012Metric" V 3230 1150 50  0001 C CNN
+F 3 "~" H 3300 1150 50  0001 C CNN
+F 4 "C1017" V 3300 1150 50  0001 C CNN "LCSC"
+	1    3300 1150
+	0    1    1    0
+$EndComp
+Wire Wire Line
+	3000 1350 3000 1150
+Connection ~ 3000 1150
+Wire Wire Line
+	3000 1150 3150 1150
+Wire Wire Line
+	3600 1350 3600 1150
+Wire Wire Line
+	3600 1150 3450 1150
+Wire Wire Line
+	3000 1650 3000 1750
+Wire Wire Line
+	3600 1750 3600 1650
+$Comp
+L power:GND #PWR0610
+U 1 1 5FDA6E85
+P 3000 1750
+F 0 "#PWR0610" H 3000 1500 50  0001 C CNN
+F 1 "GND" H 3005 1577 50  0000 C CNN
+F 2 "" H 3000 1750 50  0001 C CNN
+F 3 "" H 3000 1750 50  0001 C CNN
+	1    3000 1750
+	1    0    0    -1
+$EndComp
+$Comp
+L power:GND #PWR0611
+U 1 1 5FDA72F7
+P 3600 1750
+F 0 "#PWR0611" H 3600 1500 50  0001 C CNN
+F 1 "GND" H 3605 1577 50  0000 C CNN
+F 2 "" H 3600 1750 50  0001 C CNN
+F 3 "" H 3600 1750 50  0001 C CNN
+	1    3600 1750
+	1    0    0    -1
+$EndComp
+Wire Wire Line
+	3600 1150 3900 1150
+Connection ~ 3600 1150
+Text Label 4500 1150 0    50   ~ 0
+PB0_INT
+$Comp
+L Device:R R606
+U 1 1 5FDC878A
+P 4050 1150
+F 0 "R606" V 3843 1150 50  0000 C CNN
+F 1 "100R" V 3934 1150 50  0000 C CNN
+F 2 "Resistor_SMD:R_0603_1608Metric" V 3980 1150 50  0001 C CNN
+F 3 "~" H 4050 1150 50  0001 C CNN
+F 4 "C22775" V 4050 1150 50  0001 C CNN "LCSC"
+	1    4050 1150
+	0    1    1    0
+$EndComp
+Wire Wire Line
+	4200 1150 4500 1150
 $EndSCHEMATC

Commit message: Split the 120R CAN termination resistor into two 240R
Increase the thermal clearances on copper fills
Parts:
- U602: LCSC (none) -> C587147
Changed lines of the file:
@@
 F 2 "Package_DFN_QFN:Diodes_UDFN-10_1.0x2.5mm_P0.5mm" H 2200 1600 50  0001 C CNN
 F 3 "" H 2200 1600 50  0001 C CNN
+F 4 "C587147" H 2200 1700 50  0001 C CNN "LCSC"
 	1    2200 1700
 	1    0    0    -1

Commit message: Change the MCU to ATTiny1614
Also:
- Rewired the PCB due to changed pins
- Cleaned up network names around the MCU
- Use a basic part Schottky for the buck converter
- Change MCP2515 crystal to 16MHz basic part
- Change BAT54C to two discrete schottkys
- Change the SOD-523 schottky to MSK4005
- Update the release script and rotation DB
Parts:
- removed D602: BAT54C, Package_TO_SOT_SMD:SOT-23, symbol Diode:BAT54C
- added D602, D603: MSK4005, Diode_SMD:D_SOD-523, symbol Device:D_Schottky
- D601: value PSBD521S-40 -> MSK4005; LCSC C168633 -> C345957
- U601: value ATtiny841-SSU -> ATtiny1614-SSNR; symbol MCU_Microchip_ATtiny:ATtiny841-SSU -> MCU_Microchip_ATtiny:ATtiny1614-SS; LCSC C219103 -> C481364
Connections:
- net labels added: EN5V, EXT_INT, LED_STATUS, LED_VCAP, LED_VIN, RXD, TXD
- net labels removed: PA0, PA3_EN5V, PA5, PA7_LED2, PB0_INT, PB1_LED0, PB2_LED1
- wire segments 54 -> 53
Other:
- note removed: "Pins SDA, SCL, and PA5 are used for reflashing.\n"
- moved on the sheet: C602, R603

Commit message: Finish PCB layout updates
Parts:
- J602: LCSC (none) -> C492401
Changed lines of the file:
@@
 F 2 "Connector_PinHeader_2.54mm:PinHeader_1x02_P2.54mm_Vertical" H 850 1150 50  0001 C CNN
 F 3 "~" H 850 1150 50  0001 C CNN
+F 4 "C492401" H 850 1150 50  0001 C CNN "LCSC"
 	1    850  1150
 	-1   0    0    -1
