File: IO.sch (KiCad schematic (older format))
At the start: 19 parts, among them J701 Screw_Terminal_01x02, J702 Raspberry_Pi_2_3, U701 RCLAMP0524P-N

Commit message: Make power connector identical to SH-ESP32 for consistency
Parts:
- J701: value Screw_Terminal_01x02 -> Screw_Terminal_01x03; footprint Connector_Phoenix_MC:PhoenixContact_MC_1,5_2-G-3.81_1x02_P3.81mm_Horizontal -> Connector_Phoenix_MC:PhoenixContact_MC_1,5_3-G-3.81_1x03_P3.81mm_Horizontal; symbol Connector:Screw_Terminal_01x02 -> Connector:Screw_Terminal_01x03
Connections:
- wire segments 45 -> 48
Changed lines of the file:
@@
 Supercaps are now behind a\nseparate connector (min. 8A)
 $Comp
-L Connector:Screw_Terminal_01x02 J?
+L Connector:Screw_Terminal_01x03 J?
 U 1 1 5FAF7481
-P 1700 5450
+P 1700 5550
 AR Path="/5FAF7481" Ref="J?"  Part="1"
 AR Path="/5FAD80E5/5FAF7481" Ref="J701"  Part="1"
-F 0 "J701" H 1780 5442 50  0000 L CNN
-F 1 "Screw_Terminal_01x02" H 1780 5351 50  0000 L CNN
-F 2 "Connector_Phoenix_MC:PhoenixContact_MC_1,5_2-G-3.81_1x02_P3.81mm_Horizontal" H 1700 5450 50  0001 C CNN
-F 3 "~" H 1700 5450 50  0001 C CNN
-F 4 "C8387" H 1700 5450 50  0001 C CNN "LCSC"
-	1    1700 5450
+F 0 "J701" H 1780 5542 50  0000 L CNN
+F 1 "Screw_Terminal_01x03" H 1780 5451 50  0000 L CNN
+F 2 "Connector_Phoenix_MC:PhoenixContact_MC_1,5_3-G-3.81_1x03_P3.81mm_Horizontal" H 1700 5550 50  0001 C CNN
+F 3 "~" H 1700 5550 50  0001 C CNN
+F 4 "C8387" H 1700 5550 50  0001 C CNN "LCSC"
+	1    1700 5550
 	-1   0    0    -1
 $EndComp
@@
 	6200 5450 6450 5450
 Wire Wire Line
-	1900 5550 2450 5550
+	1900 5550 2000 5550
 Wire Wire Line
 	2450 6050 2450 5950
@@
 	1    0    0    -1
 $EndComp
+Wire Wire Line
+	1900 5650 2000 5650
+Wire Wire Line
+	2000 5650 2000 5550
+Connection ~ 2000 5550
+Wire Wire Line
+	2000 5550 2450 5550
 $EndSCHEMATC

Commit message: Add missing LCSC part numbers
Parts:
- U701: LCSC (none) -> C316044
Changed lines of the file:
@@
 F 2 "Package_DFN_QFN:Diodes_UDFN-10_1.0x2.5mm_P0.5mm" H 2800 6050 50  0001 C CNN
 F 3 "" H 2800 6050 50  0001 C CNN
+F 4 "C316044" H 2800 6150 50  0001 C CNN "LCSC"
 	1    2800 6150
 	1    0    0    -1

Commit message: Rename project files to follow the conventions in SH-ESP32
Parts:
- U701: symbol sailor-hat:RCLAMP0524P-N -> SH-RPi:RCLAMP0524P-N
Connections:
- wire segments 48 -> 42
- no-connect marks 21 -> 25
Changed lines of the file:
@@
 SCL
 $Comp
-L sailor-hat:RCLAMP0524P-N U701
+L SH-RPi:RCLAMP0524P-N U701
 U 1 1 5FB6B31D
 P 2800 6150
@@
 	1    0    0    -1
 $EndComp
-Wire Wire Line
-	1900 5450 2050 5450
-Wire Wire Line
-	2450 6150 2150 6150
-Wire Wire Line
-	2150 6150 2150 5450
-Connection ~ 2150 5450
-Wire Wire Line
-	2150 5450 3450 5450
-Wire Wire Line
-	2450 6250 2050 6250
-Wire Wire Line
-	2050 6250 2050 5450
-Connection ~ 2050 5450
-Wire Wire Line
-	2050 5450 2150 5450
 Wire Wire Line
 	3150 6150 3450 6150
@@
 Wire Wire Line
 	1900 5550 2000 5550
-Wire Wire Line
-	2450 6050 2450 5950
-Connection ~ 2450 5550
-Wire Wire Line
-	2450 5550 3150 5550
-Connection ~ 2450 5950
-Wire Wire Line
-	2450 5950 2450 5550
-Wire Wire Line
-	3150 6050 3150 5950
-Connection ~ 3150 5550
-Wire Wire Line
-	3150 5550 3800 5550
-Connection ~ 3150 5950
-Wire Wire Line
-	3150 5950 3150 5550
 $Comp
 L power:+3.3V #PWR0103
@@
 	2000 5650 2000 5550
 Connection ~ 2000 5550
+Connection ~ 2050 5450
 Wire Wire Line
-	2000 5550 2450 5550
+	2150 5450 3450 5450
+Connection ~ 2150 5450
+Wire Wire Line
+	2050 5450 2150 5450
+Wire Wire Line
+	1900 5450 2050 5450
+Wire Wire Line
+	2050 6250 2050 5450
+Wire Wire Line
+	2450 6250 2050 6250
+Wire Wire Line
+	2150 6150 2150 5450
+Wire Wire Line
+	2450 6150 2150 6150
+Wire Wire Line
+	2000 5550 3800 5550
+NoConn ~ 2450 5950
+NoConn ~ 2450 6050
+NoConn ~ 3150 5950
+NoConn ~ 3150 6050
 $EndSCHEMATC

Commit message: Updated the title block and one THT terminal part number
Parts:
- J701: LCSC C8387 -> C8406
Changed lines of the file:
@@
 F 2 "Connector_Phoenix_MC:PhoenixContact_MC_1,5_3-G-3.81_1x03_P3.81mm_Horizontal" H 1700 5550 50  0001 C CNN
 F 3 "~" H 1700 5550 50  0001 C CNN
-F 4 "C8387" H 1700 5550 50  0001 C CNN "LCSC"
+F 4 "C8406" H 1700 5550 50  0001 C CNN "LCSC"
 	1    1700 5550
 	-1   0    0    -1

Commit message: Extend the PCB size to provide space for an onboard supercapacitor
The PCB was extended to the left by 21mm to provide room for a
18x40mm (max 18x42mm) 50/60F supercapacitor. The supercapacitor
is lodged in a slot on the PCB to provide mechanical stability and limit
the maximum height of the assembly. It now requires 14mm of headroom.

Additionally, the following changes were made:

- the external supercap connector was removed
- the power and CAN connectors were swapped to JST XH
- there is space for a wire link between CAN and power conx
- power protection circuitry was moved to the edge of the board
- 3.3V regulator was moved to improve the layout
- a 100pF cap was added to the boost feedback to improve loop stability
- rectangles were drawn around ground pins on the GPIO connector
Parts:
- removed C701: 10uF/50V, Capacitor_SMD:C_1206_3216Metric, symbol Device:C
- removed C702: 10uF, Capacitor_SMD:C_0402_1005Metric, symbol Device:C
- removed FB701: GZ2012D601TF, Inductor_SMD:L_0805_2012Metric, symbol Device:Ferrite_Bead
- removed J701: Screw_Terminal_01x03, Connector_Phoenix_MC:PhoenixContact_MC_1,5_3-G-3.81_1x03_P3.81mm_Horizontal, symbol Connector:Screw_Terminal_01x03
- removed U701: RCLAMP0524P-N, Package_DFN_QFN:Diodes_UDFN-10_1.0x2.5mm_P0.5mm, symbol SH-RPi:RCLAMP0524P-N
- J702: footprint Connector_PinHeader_2.54mm:PinHeader_2x20_P2.54mm_Vertical -> SH-RPi:PinHeader_RPi-GPIO
Connections:
- net labels removed: Vcap, Vcap_CONN
- wire segments 42 -> 19
- no-connect marks 25 -> 21
Other:
- note removed: "Supercaps are now behind a\nseparate connector (min. 8A)"
Changed lines of the file:
@@
 Title "Sailor Hat for Raspberry Pi"
 Date ""
-Rev "revL"
+Rev "revM"
 Comp "Hat Laboratories"
 Comment1 "https://creativecommons.org/licenses/by-sa/4.0"
@@
 F 0 "J702" H 2650 4400 50  0000 C CNN
 F 1 "Raspberry_Pi_2_3" H 2950 4300 50  0000 C CNN
-F 2 "Connector_PinHeader_2.54mm:PinHeader_2x20_P2.54mm_Vertical" H 2350 3000 50  0001 C CNN
+F 2 "SH-RPi:PinHeader_RPi-GPIO" H 2350 3000 50  0001 C CNN
 F 3 "https://www.raspberrypi.org/documentation/hardware/raspberrypi/schematics/rpi_SCH_3bplus_1p0_reduced.pdf" H 2350 3000 50  0001 C CNN
 	1    2350 3000
@@
 Text Notes 3950 2750 0    50   ~ 0
 Vin voltage
-$Comp
-L power:GND #PWR?
-U 1 1 5FAF7478
-P 3800 5550
-AR Path="/5FAF7478" Ref="#PWR?"  Part="1"
-AR Path="/5FAD80E5/5FAF7478" Ref="#PWR0711"  Part="1"
-F 0 "#PWR0711" H 3800 5300 50  0001 C CNN
-F 1 "GND" H 3805 5377 50  0000 C CNN
-F 2 "" H 3800 5550 50  0001 C CNN
-F 3 "" H 3800 5550 50  0001 C CNN
-	1    3800 5550
-	-1   0    0    -1
-$EndComp
-Text Notes 2950 5200 2    50   ~ 0
-Supercaps are now behind a\nseparate connector (min. 8A)
-$Comp
-L Connector:Screw_Terminal_01x03 J?
-U 1 1 5FAF7481
-P 1700 5550
-AR Path="/5FAF7481" Ref="J?"  Part="1"
-AR Path="/5FAD80E5/5FAF7481" Ref="J701"  Part="1"
-F 0 "J701" H 1780 5542 50  0000 L CNN
-F 1 "Screw_Terminal_01x03" H 1780 5451 50  0000 L CNN
-F 2 "Connector_Phoenix_MC:PhoenixContact_MC_1,5_3-G-3.81_1x03_P3.81mm_Horizontal" H 1700 5550 50  0001 C CNN
-F 3 "~" H 1700 5550 50  0001 C CNN
-F 4 "C8406" H 1700 5550 50  0001 C CNN "LCSC"
-	1    1700 5550
-	-1   0    0    -1
-$EndComp
 Text HLabel 4200 1600 1    50   Input ~ 0
 ATT_LED2
@@
 SCL
 $Comp
-L SH-RPi:RCLAMP0524P-N U701
-U 1 1 5FB6B31D
-P 2800 6150
-F 0 "U701" H 2800 6575 50  0000 C CNN
-F 1 "RCLAMP0524P-N" H 2800 6484 50  0000 C CNN
-F 2 "Package_DFN_QFN:Diodes_UDFN-10_1.0x2.5mm_P0.5mm" H 2800 6050 50  0001 C CNN
-F 3 "" H 2800 6050 50  0001 C CNN
-F 4 "C316044" H 2800 6150 50  0001 C CNN "LCSC"
-	1    2800 6150
-	1    0    0    -1
-$EndComp
-Wire Wire Line
-	3150 6150 3450 6150
-Wire Wire Line
-	3450 6150 3450 5450
-Connection ~ 3450 5450
-Wire Wire Line
-	3450 5450 3550 5450
-Wire Wire Line
-	3150 6250 3550 6250
-Wire Wire Line
-	3550 6250 3550 5450
-Connection ~ 3550 5450
-Wire Wire Line
-	3550 5450 3800 5450
-$Comp
-L power:GND #PWR?
-U 1 1 5FB78DB9
-P 2750 6600
-AR Path="/5FB78DB9" Ref="#PWR?"  Part="1"
-AR Path="/5FAD80E5/5FB78DB9" Ref="#PWR0709"  Part="1"
-F 0 "#PWR0709" H 2750 6350 50  0001 C CNN
-F 1 "GND" H 2755 6427 50  0000 C CNN
-F 2 "" H 2750 6600 50  0001 C CNN
-F 3 "" H 2750 6600 50  0001 C CNN
-	1    2750 6600
-	-1   0    0    -1
-$EndComp
-$Comp
-L power:GND #PWR?
-U 1 1 5FB793D5
-P 2850 6600
-AR Path="/5FB793D5" Ref="#PWR?"  Part="1"
-AR Path="/5FAD80E5/5FB793D5" Ref="#PWR0710"  Part="1"
-F 0 "#PWR0710" H 2850 6350 50  0001 C CNN
-F 1 "GND" H 2855 6427 50  0000 C CNN
-F 2 "" H 2850 6600 50  0001 C CNN
-F 3 "" H 2850 6600 50  0001 C CNN
-	1    2850 6600
-	-1   0    0    -1
-$EndComp
-Text Label 3800 5450 0    50   ~ 0
-Vcap_CONN
-$Comp
-L Device:Ferrite_Bead FB701
-U 1 1 5FB7E43C
-P 5900 5450
-F 0 "FB701" V 5626 5450 50  0000 C CNN
-F 1 "GZ2012D601TF" V 5717 5450 50  0000 C CNN
-F 2 "Inductor_SMD:L_0805_2012Metric" V 5830 5450 50  0001 C CNN
-F 3 "~" H 5900 5450 50  0001 C CNN
-F 4 "C1017" V 5900 5450 50  0001 C CNN "LCSC"
-	1    5900 5450
-	0    1    1    0
-$EndComp
-$Comp
-L Device:C C701
-U 1 1 5FB7F028
-P 5550 5650
-F 0 "C701" H 5665 5696 50  0000 L CNN
-F 1 "10uF/50V" H 5665 5605 50  0000 L CNN
-F 2 "Capacitor_SMD:C_1206_3216Metric" H 5588 5500 50  0001 C CNN
-F 3 "~" H 5550 5650 50  0001 C CNN
-F 4 "C13585" H 5550 5650 50  0001 C CNN "LCSC"
-	1    5550 5650
-	1    0    0    -1
-$EndComp
-$Comp
-L Device:C C702
-U 1 1 5FB7F7AF
-P 6200 5650
-F 0 "C702" H 6315 5696 50  0000 L CNN
-F 1 "10uF" H 6315 5605 50  0000 L CNN
-F 2 "Capacitor_SMD:C_0402_1005Metric" H 6238 5500 50  0001 C CNN
-F 3 "~" H 6200 5650 50  0001 C CNN
-F 4 "C15525" H 6200 5650 50  0001 C CNN "LCSC"
-	1    6200 5650
-	1    0    0    -1
-$EndComp
-Text Label 5350 5450 2    50   ~ 0
-Vcap_CONN
-Text HLabel 6450 5450 2    50   Input ~ 0
-Vcap
-Wire Wire Line
-	5750 5450 5550 5450
-Wire Wire Line
-	5550 5500 5550 5450
-Connection ~ 5550 5450
-Wire Wire Line
-	5550 5450 5350 5450
-$Comp
-L power:GND #PWR?
-U 1 1 5FB82711
-P 5550 5800
-AR Path="/5FB82711" Ref="#PWR?"  Part="1"
-AR Path="/5FAD80E5/5FB82711" Ref="#PWR0715"  Part="1"
-F 0 "#PWR0715" H 5550 5550 50  0001 C CNN
-F 1 "GND" H 5555 5627 50  0000 C CNN
-F 2 "" H 5550 5800 50  0001 C CNN
-F 3 "" H 5550 5800 50  0001 C CNN
-	1    5550 5800
-	-1   0    0    -1
-$EndComp
-$Comp
-L power:GND #PWR?
-U 1 1 5FB82BCB
-P 6200 5800
-AR Path="/5FB82BCB" Ref="#PWR?"  Part="1"
-AR Path="/5FAD80E5/5FB82BCB" Ref="#PWR0717"  Part="1"
-F 0 "#PWR0717" H 6200 5550 50  0001 C CNN
-F 1 "GND" H 6205 5627 50  0000 C CNN
-F 2 "" H 6200 5800 50  0001 C CNN
-F 3 "" H 6200 5800 50  0001 C CNN
-	1    6200 5800
-	-1   0    0    -1
-$EndComp
-Wire Wire Line
-	6050 5450 6200 5450
-Wire Wire Line
-	6200 5500 6200 5450
-Connection ~ 6200 5450
-Wire Wire Line
-	6200 5450 6450 5450
-Wire Wire Line
-	1900 5550 2000 5550
-$Comp
 L power:+3.3V #PWR0103
 U 1 1 5FB6095A
@@
 	1    0    0    -1
 $EndComp
-Wire Wire Line
-	1900 5650 2000 5650
-Wire Wire Line
-	2000 5650 2000 5550
-Connection ~ 2000 5550
-Connection ~ 2050 5450
-Wire Wire Line
-	2150 5450 3450 5450
-Connection ~ 2150 5450
-Wire Wire Line
-	2050 5450 2150 5450
-Wire Wire Line
-	1900 5450 2050 5450
-Wire Wire Line
-	2050 6250 2050 5450
-Wire Wire Line
-	2450 6250 2050 6250
-Wire Wire Line
-	2150 6150 2150 5450
-Wire Wire Line
-	2450 6150 2150 6150
-Wire Wire Line
-	2000 5550 3800 5550
-NoConn ~ 2450 5950
-NoConn ~ 2450 6050
-NoConn ~ 3150 5950
-NoConn ~ 3150 6050
 $EndSCHEMATC

Commit message: Route I2C to unique pins
Also:
- Connect RTC interrupt to ATtiny
- Break out the interrupt pin to a connector for external signaling
Parts:
- added R710, R711: 0, Resistor_SMD:R_0603_1608Metric, symbol Device:R
Connections:
- net labels added: GPIO12, GPIO13
Other:
- note added: "Note 2: Also SDA and SCL are on\nnon-standard GPIOs"
Changed lines of the file:
@@
 NoConn ~ 1550 3300
 NoConn ~ 1550 3400
-NoConn ~ 3150 3700
 NoConn ~ 3150 2700
 NoConn ~ 3150 2200
 NoConn ~ 3150 2100
 NoConn ~ 1550 3500
-NoConn ~ 3150 3800
 NoConn ~ 1550 2800
 NoConn ~ 1550 2900
@@
 Text HLabel 6600 1450 0    50   Input ~ 0
 SI
-Text HLabel 3150 2400 2    50   Input ~ 0
+Text HLabel 6600 2700 0    50   Input ~ 0
 SDA
-Text HLabel 3150 2500 2    50   Input ~ 0
+Text HLabel 6600 2950 0    50   Input ~ 0
 SCL
 $Comp
@@
 	1    0    0    -1
 $EndComp
+NoConn ~ 3150 2400
+NoConn ~ 3150 2500
+$Comp
+L Device:R R?
+U 1 1 5FD877B8
+P 6750 2950
+AR Path="/5FD877B8" Ref="R?"  Part="1"
+AR Path="/5FAD80E5/5FD877B8" Ref="R711"  Part="1"
+F 0 "R711" H 6820 2996 50  0000 L CNN
+F 1 "0" H 6820 2905 50  0000 L CNN
+F 2 "Resistor_SMD:R_0603_1608Metric" V 6680 2950 50  0001 C CNN
+F 3 "~" H 6750 2950 50  0001 C CNN
+F 4 "C21189" H 6750 2950 50  0001 C CNN "LCSC"
+	1    6750 2950
+	0    -1   -1   0
+$EndComp
+$Comp
+L Device:R R?
+U 1 1 5FD877BF
+P 6750 2700
+AR Path="/5FD877BF" Ref="R?"  Part="1"
+AR Path="/5FAD80E5/5FD877BF" Ref="R710"  Part="1"
+F 0 "R710" H 6820 2746 50  0000 L CNN
+F 1 "0" H 6820 2655 50  0000 L CNN
+F 2 "Resistor_SMD:R_0603_1608Metric" V 6680 2700 50  0001 C CNN
+F 3 "~" H 6750 2700 50  0001 C CNN
+F 4 "C21189" H 6750 2700 50  0001 C CNN "LCSC"
+	1    6750 2700
+	0    -1   -1   0
+$EndComp
+Text Label 3150 3700 0    50   ~ 0
+GPIO12
+Text Label 3150 3800 0    50   ~ 0
+GPIO13
+Text Label 6900 2700 0    50   ~ 0
+GPIO12
+Text Label 6900 2950 0    50   ~ 0
+GPIO13
+Text Notes 7250 2800 0    50   ~ 0
+Note 2: Also SDA and SCL are on\nnon-standard GPIOs
 $EndSCHEMATC

Commit message: Change the MCU to ATTiny1614
Also:
- Rewired the PCB due to changed pins
- Cleaned up network names around the MCU
- Use a basic part Schottky for the buck converter
- Change MCP2515 crystal to 16MHz basic part
- Change BAT54C to two discrete schottkys
- Change the SOD-523 schottky to MSK4005
- Update the release script and rotation DB
Connections:
- net labels added: ATT_LED_STATUS, ATT_LED_VCAP, ATT_LED_VIN
- net labels removed: ATT_LED0, ATT_LED1, ATT_LED2
Changed lines of the file:
@@
 Vin voltage
 Text HLabel 4200 1600 1    50   Input ~ 0
-ATT_LED2
+ATT_LED_VIN
 Text HLabel 4650 1600 1    50   Input ~ 0
 EN5V
 Text HLabel 5100 1600 1    50   Input ~ 0
-ATT_LED1
+ATT_LED_VCAP
 Text HLabel 5600 1600 1    50   Input ~ 0
-ATT_LED0
+ATT_LED_STATUS
 Text HLabel 6600 2450 0    50   Input ~ 0
 INT0
