File: boost.sch (KiCad schematic (older format))
At the start: 13 parts, among them SW201 SW_SPST, U201 TPS61022

Commit message: Modify boost stage design according to WEBENCH results
Parts:
- added C?: 1uF/25V, Capacitor_SMD:C_0402_1005Metric, symbol Device:C
- C201: value 22uF/6.3V -> 10uF/25V; LCSC C45783 -> C15850
- C202, C203, C204: value 22uF/6.3V -> 22uF/25V
- C205: value 100pF -> 1pF; LCSC C1546 -> C1550
- L201: value MWSA0603-1R0MT -> MWSA0402S-1R0MT; footprint Inductor_SMD:L_Abracon_ASPI-0630LR -> SH-RPi:L_MWSA0402; LCSC C112125 -> C408332; Notes Shun Xiang Nuo Elec SMMS0630-1R0M -> (none)
- R203: value 300k -> 750k; LCSC C25774 -> C122545
- R204: value 39k -> 100k; LCSC C25783 -> C25741
Connections:
- wire segments 38 -> 41
Other:
- note added: "FB voltage divider designed\nto provide 5.1V at Vout."
- note removed: "C205 sets an additional feedforward\nzero frequency at 5.3 kHz"
- note removed: "FB voltage divider designed\nto provide 5.21V at Vout."
- moved on the sheet: C202, C203, C204
Changed lines of the file:
@@
 L Device:C C?
 U 1 1 5CA6B4E8
-P 4850 2450
+P 5550 2450
 AR Path="/5CA6B4E8" Ref="C?"  Part="1"
 AR Path="/5C3480BB/5CA6B4E8" Ref="C?"  Part="1"
 AR Path="/5CA73F16/5CA6B4E8" Ref="C202"  Part="1"
-F 0 "C202" H 4968 2496 50  0000 L CNN
-F 1 "22uF/6.3V" H 4968 2405 50  0000 L CNN
-F 2 "Capacitor_SMD:C_0805_2012Metric" H 4888 2300 50  0001 C CNN
-F 3 "~" H 4850 2450 50  0001 C CNN
-F 4 "C45783" H 4850 2450 50  0001 C CNN "LCSC"
-	1    4850 2450
+F 0 "C202" H 5668 2496 50  0000 L CNN
+F 1 "22uF/25V" H 5668 2405 50  0000 L CNN
+F 2 "Capacitor_SMD:C_0805_2012Metric" H 5588 2300 50  0001 C CNN
+F 3 "~" H 5550 2450 50  0001 C CNN
+F 4 "C45783" H 5550 2450 50  0001 C CNN "LCSC"
+	1    5550 2450
 	1    0    0    -1
 $EndComp
@@
 AR Path="/5CA73F16/5CA6B4FC" Ref="L201"  Part="1"
 F 0 "L201" V 3540 1500 50  0000 C CNN
-F 1 "MWSA0603-1R0MT" V 3449 1500 50  0000 C CNN
-F 2 "Inductor_SMD:L_Abracon_ASPI-0630LR" H 3350 1500 50  0001 C CNN
+F 1 "MWSA0402S-1R0MT" V 3449 1500 50  0000 C CNN
+F 2 "SH-RPi:L_MWSA0402" H 3350 1500 50  0001 C CNN
 F 3 "" H 3350 1500 50  0001 C CNN
-F 4 "Shun Xiang Nuo Elec SMMS0630-1R0M" V 3350 1500 50  0001 C CNN "Notes"
-F 5 "C112125" H 3350 1500 50  0001 C CNN "LCSC"
+F 4 "" V 3350 1500 50  0001 C CNN "Notes"
+F 5 "C408332" H 3350 1500 50  0001 C CNN "LCSC"
 	1    3350 1500
 	0    -1   -1   0
@@
 AR Path="/5CA73F16/5CA6B51B" Ref="R203"  Part="1"
 F 0 "R203" H 4420 2496 50  0000 L CNN
-F 1 "300k" H 4420 2405 50  0000 L CNN
+F 1 "750k" H 4420 2405 50  0000 L CNN
 F 2 "Resistor_SMD:R_0402_1005Metric" V 4280 2450 50  0001 C CNN
 F 3 "~" H 4350 2450 50  0001 C CNN
-F 4 "C25774" H 4350 2450 50  0001 C CNN "LCSC"
+F 4 "C122545" H 4350 2450 50  0001 C CNN "LCSC"
 	1    4350 2450
 	1    0    0    -1
@@
 AR Path="/5CA73F16/5CA6B522" Ref="R204"  Part="1"
 F 0 "R204" H 4420 2896 50  0000 L CNN
-F 1 "39k" H 4420 2805 50  0000 L CNN
+F 1 "100k" H 4420 2805 50  0000 L CNN
 F 2 "Resistor_SMD:R_0402_1005Metric" V 4280 2850 50  0001 C CNN
 F 3 "~" H 4350 2850 50  0001 C CNN
-F 4 "C25783" H 4350 2850 50  0001 C CNN "LCSC"
+F 4 "C25741" H 4350 2850 50  0001 C CNN "LCSC"
 	1    4350 2850
 	1    0    0    -1
@@
 Vin
 Text Notes 4250 1800 0    50   ~ 0
-FB voltage divider designed\nto provide 5.21V at Vout.
-Text HLabel 6400 2300 2    50   Output ~ 0
+FB voltage divider designed\nto provide 5.1V at Vout.
+Text HLabel 7100 2300 2    50   Output ~ 0
 Vboost
 $Comp
@@
 AR Path="/5CA73F16/5CF608F8" Ref="C201"  Part="1"
 F 0 "C201" H 3218 1696 50  0000 L CNN
-F 1 "22uF/6.3V" H 3218 1605 50  0000 L CNN
+F 1 "10uF/25V" H 3218 1605 50  0000 L CNN
 F 2 "Capacitor_SMD:C_0805_2012Metric" H 3138 1500 50  0001 C CNN
 F 3 "~" H 3100 1650 50  0001 C CNN
-F 4 "C45783" H 3100 1650 50  0001 C CNN "LCSC"
+F 4 "C15850" H 3100 1650 50  0001 C CNN "LCSC"
 	1    3100 1650
 	1    0    0    -1
@@
 	3400 3050 3400 2800
 Connection ~ 4350 2300
-Connection ~ 4850 2300
-Wire Wire Line
-	4850 2300 4350 2300
+Connection ~ 5550 2300
+Wire Wire Line
+	5550 2300 4900 2300
 Wire Wire Line
 	2900 2500 3000 2500
@@
 L Device:C C?
 U 1 1 5D8155D9
-P 5400 2600
+P 6100 2600
 AR Path="/5D8155D9" Ref="C?"  Part="1"
 AR Path="/5C3480BB/5D8155D9" Ref="C?"  Part="1"
 AR Path="/5CA73F16/5D8155D9" Ref="C203"  Part="1"
-F 0 "C203" H 5518 2646 50  0000 L CNN
-F 1 "22uF/6.3V" H 5518 2555 50  0000 L CNN
-F 2 "Capacitor_SMD:C_0805_2012Metric" H 5438 2450 50  0001 C CNN
-F 3 "~" H 5400 2600 50  0001 C CNN
-F 4 "C45783" H 5400 2600 50  0001 C CNN "LCSC"
-	1    5400 2600
+F 0 "C203" H 6218 2646 50  0000 L CNN
+F 1 "22uF/25V" H 6218 2555 50  0000 L CNN
+F 2 "Capacitor_SMD:C_0805_2012Metric" H 6138 2450 50  0001 C CNN
+F 3 "~" H 6100 2600 50  0001 C CNN
+F 4 "C45783" H 6100 2600 50  0001 C CNN "LCSC"
+	1    6100 2600
 	1    0    0    -1
 $EndComp
@@
 	2900 1500 3100 1500
 Wire Wire Line
-	5400 2450 5400 2300
-Connection ~ 5400 2300
-Wire Wire Line
-	5400 2300 4850 2300
-Wire Wire Line
-	5400 2300 5950 2300
+	6100 2450 6100 2300
+Connection ~ 6100 2300
+Wire Wire Line
+	6100 2300 5550 2300
+Wire Wire Line
+	6100 2300 6650 2300
 $Comp
 L Device:C C?
 U 1 1 5E6767E0
-P 5950 2750
+P 6650 2750
 AR Path="/5E6767E0" Ref="C?"  Part="1"
 AR Path="/5C3480BB/5E6767E0" Ref="C?"  Part="1"
 AR Path="/5CA73F16/5E6767E0" Ref="C204"  Part="1"
-F 0 "C204" H 6068 2796 50  0000 L CNN
-F 1 "22uF/6.3V" H 6068 2705 50  0000 L CNN
-F 2 "Capacitor_SMD:C_0805_2012Metric" H 5988 2600 50  0001 C CNN
-F 3 "~" H 5950 2750 50  0001 C CNN
-F 4 "C45783" H 5950 2750 50  0001 C CNN "LCSC"
-	1    5950 2750
-	1    0    0    -1
-$EndComp
-Wire Wire Line
-	5950 2600 5950 2300
-Connection ~ 5950 2300
-Wire Wire Line
-	5950 2300 6400 2300
-Wire Wire Line
-	5950 2900 5950 3050
+F 0 "C204" H 6768 2796 50  0000 L CNN
+F 1 "22uF/25V" H 6768 2705 50  0000 L CNN
+F 2 "Capacitor_SMD:C_0805_2012Metric" H 6688 2600 50  0001 C CNN
+F 3 "~" H 6650 2750 50  0001 C CNN
+F 4 "C45783" H 6650 2750 50  0001 C CNN "LCSC"
+	1    6650 2750
+	1    0    0    -1
+$EndComp
+Wire Wire Line
+	6650 2600 6650 2300
+Connection ~ 6650 2300
+Wire Wire Line
+	6650 2300 7100 2300
+Wire Wire Line
+	6650 2900 6650 3050
 $Comp
 L power:GND #PWR?
 U 1 1 5E6767E6
-P 5950 3050
+P 6650 3050
 AR Path="/5E6767E6" Ref="#PWR?"  Part="1"
 AR Path="/5C3480BB/5E6767E6" Ref="#PWR?"  Part="1"
 AR Path="/5CA73F16/5E6767E6" Ref="#PWR0209"  Part="1"
-F 0 "#PWR0209" H 5950 2800 50  0001 C CNN
-F 1 "GND" H 5955 2877 50  0000 C CNN
-F 2 "" H 5950 3050 50  0001 C CNN
-F 3 "" H 5950 3050 50  0001 C CNN
-	1    5950 3050
-	1    0    0    -1
-$EndComp
-Wire Wire Line
-	5400 2750 5400 3050
+F 0 "#PWR0209" H 6650 2800 50  0001 C CNN
+F 1 "GND" H 6655 2877 50  0000 C CNN
+F 2 "" H 6650 3050 50  0001 C CNN
+F 3 "" H 6650 3050 50  0001 C CNN
+	1    6650 3050
+	1    0    0    -1
+$EndComp
+Wire Wire Line
+	6100 2750 6100 3050
 $Comp
 L power:GND #PWR?
 U 1 1 5D815A89
-P 5400 3050
+P 6100 3050
 AR Path="/5D815A89" Ref="#PWR?"  Part="1"
 AR Path="/5C3480BB/5D815A89" Ref="#PWR?"  Part="1"
 AR Path="/5CA73F16/5D815A89" Ref="#PWR0208"  Part="1"
-F 0 "#PWR0208" H 5400 2800 50  0001 C CNN
-F 1 "GND" H 5405 2877 50  0000 C CNN
-F 2 "" H 5400 3050 50  0001 C CNN
-F 3 "" H 5400 3050 50  0001 C CNN
-	1    5400 3050
+F 0 "#PWR0208" H 6100 2800 50  0001 C CNN
+F 1 "GND" H 6105 2877 50  0000 C CNN
+F 2 "" H 6100 3050 50  0001 C CNN
+F 3 "" H 6100 3050 50  0001 C CNN
+	1    6100 3050
 	1    0    0    -1
 $EndComp
@@
 L power:GND #PWR?
 U 1 1 5CA6B4EF
-P 4850 3050
+P 5550 3050
 AR Path="/5CA6B4EF" Ref="#PWR?"  Part="1"
 AR Path="/5C3480BB/5CA6B4EF" Ref="#PWR?"  Part="1"
 AR Path="/5CA73F16/5CA6B4EF" Ref="#PWR0207"  Part="1"
-F 0 "#PWR0207" H 4850 2800 50  0001 C CNN
-F 1 "GND" H 4855 2877 50  0000 C CNN
-F 2 "" H 4850 3050 50  0001 C CNN
-F 3 "" H 4850 3050 50  0001 C CNN
-	1    4850 3050
-	1    0    0    -1
-$EndComp
-Wire Wire Line
-	4850 3050 4850 2600
+F 0 "#PWR0207" H 5550 2800 50  0001 C CNN
+F 1 "GND" H 5555 2877 50  0000 C CNN
+F 2 "" H 5550 3050 50  0001 C CNN
+F 3 "" H 5550 3050 50  0001 C CNN
+	1    5550 3050
+	1    0    0    -1
+$EndComp
+Wire Wire Line
+	5550 3050 5550 2600
 Text Notes 600  3000 0    50   ~ 0
 Switch/header allows for\npower-cycling the RPi.
@@
 P 4100 2450
 F 0 "C205" H 3986 2404 50  0000 R CNN
-F 1 "100pF" H 3986 2495 50  0000 R CNN
+F 1 "1pF" H 3986 2495 50  0000 R CNN
 F 2 "Capacitor_SMD:C_0402_1005Metric" H 4138 2300 50  0001 C CNN
 F 3 "~" H 4100 2450 50  0001 C CNN
-F 4 "C1546" H 4100 2450 50  0001 C CNN "LCSC"
+F 4 "C1550" H 4100 2450 50  0001 C CNN "LCSC"
 	1    4100 2450
 	1    0    0    1
@@
 Wire Wire Line
 	4100 2300 4350 2300
-Text Notes 4000 2150 0    50   ~ 0
-C205 sets an additional feedforward\nzero frequency at 5.3 kHz
 $Comp
 L Device:C C206
@@
 Text Notes 2400 3850 0    50   ~ 0
 C206 limits switch bouncing and slows\nreset on poweron
+$Comp
+L Device:C C?
+U 1 1 60184DB1
+P 4900 2600
+AR Path="/60184DB1" Ref="C?"  Part="1"
+AR Path="/5C3480BB/60184DB1" Ref="C?"  Part="1"
+AR Path="/5CA73F16/60184DB1" Ref="C?"  Part="1"
+F 0 "C?" H 5018 2646 50  0000 L CNN
+F 1 "1uF/25V" H 5018 2555 50  0000 L CNN
+F 2 "Capacitor_SMD:C_0402_1005Metric" H 4938 2450 50  0001 C CNN
+F 3 "~" H 4900 2600 50  0001 C CNN
+F 4 "C52923" H 4900 2600 50  0001 C CNN "LCSC"
+	1    4900 2600
+	1    0    0    -1
+$EndComp
+$Comp
+L power:GND #PWR?
+U 1 1 60184DB7
+P 4900 3050
+AR Path="/60184DB7" Ref="#PWR?"  Part="1"
+AR Path="/5C3480BB/60184DB7" Ref="#PWR?"  Part="1"
+AR Path="/5CA73F16/60184DB7" Ref="#PWR?"  Part="1"
+F 0 "#PWR?" H 4900 2800 50  0001 C CNN
+F 1 "GND" H 4905 2877 50  0000 C CNN
+F 2 "" H 4900 3050 50  0001 C CNN
+F 3 "" H 4900 3050 50  0001 C CNN
+	1    4900 3050
+	1    0    0    -1
+$EndComp
+Wire Wire Line
+	4900 2450 4900 2300
+Connection ~ 4900 2300
+Wire Wire Line
+	4900 2300 4350 2300
+Wire Wire Line
+	4900 2750 4900 3050
 $EndSCHEMATC

Commit message: Buck converter changed to LMR16030
Parts:
- C206: footprint Resistor_SMD:R_0402_1005Metric -> Capacitor_SMD:C_0402_1005Metric
- gave numbers to parts that had none: 1
Changed lines of the file:
@@
 F 0 "C206" H 2415 2896 50  0000 L CNN
 F 1 "1uF" H 2415 2805 50  0000 L CNN
-F 2 "Resistor_SMD:R_0402_1005Metric" H 2338 2700 50  0001 C CNN
+F 2 "Capacitor_SMD:C_0402_1005Metric" H 2338 2700 50  0001 C CNN
 F 3 "~" H 2300 2850 50  0001 C CNN
 F 4 "C52923" H 2300 2850 50  0001 C CNN "LCSC"
@@
 AR Path="/60184DB1" Ref="C?"  Part="1"
 AR Path="/5C3480BB/60184DB1" Ref="C?"  Part="1"
-AR Path="/5CA73F16/60184DB1" Ref="C?"  Part="1"
-F 0 "C?" H 5018 2646 50  0000 L CNN
+AR Path="/5CA73F16/60184DB1" Ref="C207"  Part="1"
+F 0 "C207" H 5018 2646 50  0000 L CNN
 F 1 "1uF/25V" H 5018 2555 50  0000 L CNN
 F 2 "Capacitor_SMD:C_0402_1005Metric" H 4938 2450 50  0001 C CNN
@@
 AR Path="/60184DB7" Ref="#PWR?"  Part="1"
 AR Path="/5C3480BB/60184DB7" Ref="#PWR?"  Part="1"
-AR Path="/5CA73F16/60184DB7" Ref="#PWR?"  Part="1"
-F 0 "#PWR?" H 4900 2800 50  0001 C CNN
+AR Path="/5CA73F16/60184DB7" Ref="#PWR0101"  Part="1"
+F 0 "#PWR0101" H 4900 2800 50  0001 C CNN
 F 1 "GND" H 4905 2877 50  0000 C CNN
 F 2 "" H 4900 3050 50  0001 C CNN
