File: pcb.sch (KiCad schematic (older format))
At the start: 14 parts

Commit message: Remove undersized ferrite bead, shuffle power protection circuitry
Also add new logo & generic cleanup
Parts:
- added H901: MountingHole, SH-RPi:MountingHole_3.2mm_no_pad, symbol Mechanical:MountingHole
Changed lines of the file:
@@
 Wire Wire Line
 	1750 6400 1750 6000
+$Comp
+L Mechanical:MountingHole H901
+U 1 1 603EEE8F
+P 3100 1600
+F 0 "H901" H 3200 1646 50  0000 L CNN
+F 1 "MountingHole" H 3200 1555 50  0000 L CNN
+F 2 "SH-RPi:MountingHole_3.2mm_no_pad" H 3100 1600 50  0001 C CNN
+F 3 "~" H 3100 1600 50  0001 C CNN
+	1    3100 1600
+	1    0    0    -1
+$EndComp
 $EndSCHEMATC
