File: rtc.sch (KiCad schematic (older format))
At the start: 3 parts, among them U401 DS3231MZ

Commit message: Redesigned layout to take EMC issues better into account
Parts:
- removed BT401: CR1220 3V, custom:BatteryHolder_Linx_BAT-HLD-012-SMT, symbol Device:Battery_Cell
- added BT401: CR1220/3V, custom:BatteryHolder_Linx_BAT-HLD-012-SMT, symbol Connector_Generic:Conn_01x03
- C401: footprint Capacitor_SMD:C_0603_1608Metric -> Capacitor_SMD:C_0402_1005Metric; LCSC C14663 -> C1525
Connections:
- net labels added: ATT_Vcc
- net labels removed: 3.3V
- wire segments 11 -> 14
- no-connect marks 3 -> 4
Changed lines of the file:
@@
 $Descr A4 11693 8268
 encoding utf-8
-Sheet 5 8
+Sheet 4 9
 Title "Sailor Hat for Raspberry Pi"
 Date ""
@@
 F 0 "C401" H 3065 1396 50  0000 L CNN
 F 1 "100nF" H 3065 1305 50  0000 L CNN
-F 2 "Capacitor_SMD:C_0603_1608Metric" H 2988 1200 50  0001 C CNN
+F 2 "Capacitor_SMD:C_0402_1005Metric" H 2988 1200 50  0001 C CNN
 F 3 "~" H 2950 1350 50  0001 C CNN
-F 4 "C14663" H 2950 1350 50  0001 C CNN "LCSC"
+F 4 "C1525" H 2950 1350 50  0001 C CNN "LCSC"
 	1    2950 1350
 	0    -1   -1   0
 $EndComp
-Text GLabel 2600 1200 1    50   Input ~ 0
-3.3V
 $Comp
 L power:GND #PWR0402
@@
 	2600 2750 2600 2550
 $Comp
-L Device:Battery_Cell BT401
-U 1 1 5C354C49
-P 3550 2300
-F 0 "BT401" H 3668 2396 50  0000 L CNN
-F 1 "CR1220 3V" H 3668 2305 50  0000 L CNN
-F 2 "custom:BatteryHolder_Linx_BAT-HLD-012-SMT" V 3550 2360 50  0001 C CNN
-F 3 "~" V 3550 2360 50  0001 C CNN
-F 4 "712-BAT-HLD-012-SMT" H 3550 2300 50  0001 C CNN "Mouser"
-	1    3550 2300
-	1    0    0    -1
-$EndComp
-$Comp
 L power:GND #PWR0403
 U 1 1 5C354D0D
-P 3550 2400
-F 0 "#PWR0403" H 3550 2150 50  0001 C CNN
-F 1 "GND" H 3555 2227 50  0000 C CNN
-F 2 "" H 3550 2400 50  0001 C CNN
-F 3 "" H 3550 2400 50  0001 C CNN
-	1    3550 2400
+P 3600 2900
+F 0 "#PWR0403" H 3600 2650 50  0001 C CNN
+F 1 "GND" H 3605 2727 50  0000 C CNN
+F 2 "" H 3600 2900 50  0001 C CNN
+F 3 "" H 3600 2900 50  0001 C CNN
+	1    3600 2900
 	1    0    0    -1
 $EndComp
@@
 $EndComp
 Connection ~ 3550 2050
-Wire Wire Line
-	3550 2050 3550 2100
 Wire Wire Line
 	2600 1200 2600 1350
@@
 Wire Wire Line
 	2500 1650 2500 1750
+$Comp
+L Connector_Generic:Conn_01x03 BT401
+U 1 1 5FAFCA18
+P 3900 2650
+F 0 "BT401" H 3980 2692 50  0000 L CNN
+F 1 "CR1220/3V" H 3980 2601 50  0000 L CNN
+F 2 "custom:BatteryHolder_Linx_BAT-HLD-012-SMT" H 3900 2650 50  0001 C CNN
+F 3 "~" H 3900 2650 50  0001 C CNN
+	1    3900 2650
+	1    0    0    -1
+$EndComp
+Wire Wire Line
+	3600 2900 3600 2750
+Wire Wire Line
+	3600 2750 3700 2750
+Wire Wire Line
+	3550 2550 3700 2550
+Wire Wire Line
+	3550 2050 3550 2550
+NoConn ~ 3700 2650
+Text HLabel 2600 1200 1    50   Input ~ 0
+ATT_Vcc
 $EndSCHEMATC

Commit message: Make power connector identical to SH-ESP32 for consistency
Changed lines of the file:
@@
 Wire Wire Line
 	3600 2750 3700 2750
-Wire Wire Line
-	3550 2550 3700 2550
-Wire Wire Line
-	3550 2050 3550 2550
-NoConn ~ 3700 2650
 Text HLabel 2600 1200 1    50   Input ~ 0
 ATT_Vcc
+Wire Wire Line
+	3550 2650 3700 2650
+Wire Wire Line
+	3550 2050 3550 2650
+NoConn ~ 3700 2550
 $EndSCHEMATC

Commit message: Rename project files to follow the conventions in SH-ESP32
Parts:
- BT401: footprint custom:BatteryHolder_Linx_BAT-HLD-012-SMT -> SH-RPi:BatteryHolder_Linx_BAT-HLD-012-SMT
Changed lines of the file:
@@
 F 0 "BT401" H 3980 2692 50  0000 L CNN
 F 1 "CR1220/3V" H 3980 2601 50  0000 L CNN
-F 2 "custom:BatteryHolder_Linx_BAT-HLD-012-SMT" H 3900 2650 50  0001 C CNN
+F 2 "SH-RPi:BatteryHolder_Linx_BAT-HLD-012-SMT" H 3900 2650 50  0001 C CNN
 F 3 "~" H 3900 2650 50  0001 C CNN
 	1    3900 2650

Commit message: Split the 120R CAN termination resistor into two 240R
Increase the thermal clearances on copper fills
Connections:
- net labels added: RTC_INT
- wire segments 14 -> 15
- no-connect marks 4 -> 3
Other:
- moved on the sheet: C401, U401
Changed lines of the file:
@@
 L Device:C C401
 U 1 1 5C353CB0
-P 2950 1350
-F 0 "C401" H 3065 1396 50  0000 L CNN
-F 1 "100nF" H 3065 1305 50  0000 L CNN
-F 2 "Capacitor_SMD:C_0402_1005Metric" H 2988 1200 50  0001 C CNN
-F 3 "~" H 2950 1350 50  0001 C CNN
-F 4 "C1525" H 2950 1350 50  0001 C CNN "LCSC"
-	1    2950 1350
+P 5350 3000
+F 0 "C401" H 5465 3046 50  0000 L CNN
+F 1 "100nF" H 5465 2955 50  0000 L CNN
+F 2 "Capacitor_SMD:C_0402_1005Metric" H 5388 2850 50  0001 C CNN
+F 3 "~" H 5350 3000 50  0001 C CNN
+F 4 "C1525" H 5350 3000 50  0001 C CNN "LCSC"
+	1    5350 3000
 	0    -1   -1   0
 $EndComp
@@
 L power:GND #PWR0402
 U 1 1 5C354469
-P 3300 1350
-F 0 "#PWR0402" H 3300 1100 50  0001 C CNN
-F 1 "GND" H 3305 1177 50  0000 C CNN
-F 2 "" H 3300 1350 50  0001 C CNN
-F 3 "" H 3300 1350 50  0001 C CNN
-	1    3300 1350
+P 5700 3000
+F 0 "#PWR0402" H 5700 2750 50  0001 C CNN
+F 1 "GND" H 5705 2827 50  0000 C CNN
+F 2 "" H 5700 3000 50  0001 C CNN
+F 3 "" H 5700 3000 50  0001 C CNN
+	1    5700 3000
 	1    0    0    -1
 $EndComp
-Text HLabel 1800 1950 0    50   Input ~ 0
+Text HLabel 4200 3600 0    50   Input ~ 0
 SCL
-Text HLabel 1800 2050 0    50   BiDi ~ 0
+Text HLabel 4200 3700 0    50   BiDi ~ 0
 SDA
 Wire Wire Line
-	1800 1950 2100 1950
+	4200 3600 4500 3600
 Wire Wire Line
-	1800 2050 2100 2050
+	4200 3700 4500 3700
 $Comp
 L power:GND #PWR0401
 U 1 1 5C35498E
-P 2600 2750
-F 0 "#PWR0401" H 2600 2500 50  0001 C CNN
-F 1 "GND" H 2605 2577 50  0000 C CNN
-F 2 "" H 2600 2750 50  0001 C CNN
-F 3 "" H 2600 2750 50  0001 C CNN
-	1    2600 2750
+P 5000 4400
+F 0 "#PWR0401" H 5000 4150 50  0001 C CNN
+F 1 "GND" H 5005 4227 50  0000 C CNN
+F 2 "" H 5000 4400 50  0001 C CNN
+F 3 "" H 5000 4400 50  0001 C CNN
+	1    5000 4400
 	1    0    0    -1
 $EndComp
 Wire Wire Line
-	2600 2750 2600 2550
+	5000 4400 5000 4200
 $Comp
 L power:GND #PWR0403
 U 1 1 5C354D0D
-P 3600 2900
-F 0 "#PWR0403" H 3600 2650 50  0001 C CNN
-F 1 "GND" H 3605 2727 50  0000 C CNN
-F 2 "" H 3600 2900 50  0001 C CNN
-F 3 "" H 3600 2900 50  0001 C CNN
-	1    3600 2900
-	1    0    0    -1
+P 2900 4550
+F 0 "#PWR0403" H 2900 4300 50  0001 C CNN
+F 1 "GND" H 2905 4377 50  0000 C CNN
+F 2 "" H 2900 4550 50  0001 C CNN
+F 3 "" H 2900 4550 50  0001 C CNN
+	1    2900 4550
+	-1   0    0    -1
 $EndComp
 Wire Wire Line
-	2500 1650 3550 1650
+	4900 3300 2950 3300
 Wire Wire Line
-	3550 1650 3550 2050
-NoConn ~ 2100 2350
-NoConn ~ 3100 2250
-NoConn ~ 3100 1950
+	2950 3300 2950 3700
+NoConn ~ 4500 4000
+NoConn ~ 5500 3600
 $Comp
 L power:PWR_FLAG #FLG0401
 U 1 1 5C392B36
-P 3550 2050
-F 0 "#FLG0401" H 3550 2125 50  0001 C CNN
-F 1 "PWR_FLAG" V 3550 2178 50  0000 L CNN
-F 2 "" H 3550 2050 50  0001 C CNN
-F 3 "~" H 3550 2050 50  0001 C CNN
-	1    3550 2050
-	0    1    1    0
+P 2950 3700
+F 0 "#FLG0401" H 2950 3775 50  0001 C CNN
+F 1 "PWR_FLAG" V 2950 3828 50  0000 L CNN
+F 2 "" H 2950 3700 50  0001 C CNN
+F 3 "~" H 2950 3700 50  0001 C CNN
+	1    2950 3700
+	0    -1   1    0
 $EndComp
-Connection ~ 3550 2050
+Connection ~ 2950 3700
 Wire Wire Line
-	2600 1200 2600 1350
+	5000 2850 5000 3000
 Wire Wire Line
-	3300 1350 3100 1350
+	5700 3000 5500 3000
 Wire Wire Line
-	2800 1350 2600 1350
-Connection ~ 2600 1350
+	5200 3000 5000 3000
+Connection ~ 5000 3000
 Wire Wire Line
-	2600 1350 2600 1750
-Text Label 3550 1650 0    50   ~ 0
+	5000 3000 5000 3400
+Text Label 2950 3300 2    50   ~ 0
 VBAT
 $Comp
 L Timer_RTC:DS3231MZ U401
 U 1 1 5D77B733
-P 2600 2150
-F 0 "U401" H 2600 1661 50  0000 C CNN
-F 1 "DS3231MZ" H 2600 1570 50  0000 C CNN
-F 2 "Package_SO:SOIC-8_3.9x4.9mm_P1.27mm" H 2600 1650 50  0001 C CNN
-F 3 "http://datasheets.maximintegrated.com/en/ds/DS3231M.pdf" H 2600 1550 50  0001 C CNN
-F 4 "C107410" H 2600 2150 50  0001 C CNN "LCSC"
-	1    2600 2150
+P 5000 3800
+F 0 "U401" H 5000 3311 50  0000 C CNN
+F 1 "DS3231MZ" H 5000 3220 50  0000 C CNN
+F 2 "Package_SO:SOIC-8_3.9x4.9mm_P1.27mm" H 5000 3300 50  0001 C CNN
+F 3 "http://datasheets.maximintegrated.com/en/ds/DS3231M.pdf" H 5000 3200 50  0001 C CNN
+F 4 "C107410" H 5000 3800 50  0001 C CNN "LCSC"
+	1    5000 3800
 	1    0    0    -1
 $EndComp
 Wire Wire Line
-	2500 1650 2500 1750
+	4900 3300 4900 3400
 $Comp
 L Connector_Generic:Conn_01x03 BT401
 U 1 1 5FAFCA18
-P 3900 2650
-F 0 "BT401" H 3980 2692 50  0000 L CNN
-F 1 "CR1220/3V" H 3980 2601 50  0000 L CNN
-F 2 "SH-RPi:BatteryHolder_Linx_BAT-HLD-012-SMT" H 3900 2650 50  0001 C CNN
-F 3 "~" H 3900 2650 50  0001 C CNN
-	1    3900 2650
-	1    0    0    -1
+P 2600 4300
+F 0 "BT401" H 2680 4342 50  0000 L CNN
+F 1 "CR1220/3V" H 2680 4251 50  0000 L CNN
+F 2 "SH-RPi:BatteryHolder_Linx_BAT-HLD-012-SMT" H 2600 4300 50  0001 C CNN
+F 3 "~" H 2600 4300 50  0001 C CNN
+	1    2600 4300
+	-1   0    0    -1
 $EndComp
 Wire Wire Line
-	3600 2900 3600 2750
+	2900 4550 2900 4400
 Wire Wire Line
-	3600 2750 3700 2750
-Text HLabel 2600 1200 1    50   Input ~ 0
+	2900 4400 2800 4400
+Text HLabel 5000 2850 1    50   Input ~ 0
 ATT_Vcc
 Wire Wire Line
-	3550 2650 3700 2650
+	2950 4300 2800 4300
 Wire Wire Line
-	3550 2050 3550 2650
-NoConn ~ 3700 2550
+	2950 3700 2950 4300
+NoConn ~ 2800 4200
+Text HLabel 5800 3900 2    50   Output ~ 0
+RTC_INT
+Wire Wire Line
+	5800 3900 5500 3900
 $EndSCHEMATC

Commit message: Remove undersized ferrite bead, shuffle power protection circuitry
Also add new logo & generic cleanup
Parts:
- BT401: footprint SH-RPi:BatteryHolder_Linx_BAT-HLD-012-SMT -> SH-RPi:BatteryHolder_Myoung_MY-1220-03
Changed lines of the file:
@@
 F 0 "BT401" H 2680 4342 50  0000 L CNN
 F 1 "CR1220/3V" H 2680 4251 50  0000 L CNN
-F 2 "SH-RPi:BatteryHolder_Linx_BAT-HLD-012-SMT" H 2600 4300 50  0001 C CNN
+F 2 "SH-RPi:BatteryHolder_Myoung_MY-1220-03" H 2600 4300 50  0001 C CNN
 F 3 "~" H 2600 4300 50  0001 C CNN
 	1    2600 4300
