File: buck.kicad_sch (KiCad schematic)
At the start: 35 parts, among them U301 PJ75AL33SA, U302 LMR14050SDDA, U303 MD1322

Commit message: Fix broken symbols
Parts:
- C309: symbol Device:CP -> Device:C_Polarized
Connections:
- net GND: now also C309.2
- net Vcap: now also C309.1
Changed lines of the file:
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@@
     (effects (font (size 1.27 1.27)) (justify left))
   )
-  (symbol (lib_id "power:PWR_FLAG") (at 46.99 167.64 0)
+  (symbol (lib_id "power:PWR_FLAG") (at 46.99 167.64 0) (unit 1)
     (in_bom yes) (on_board yes)
     (property "Reference" "#FLG0302" (id 0) (at 46.99 165.735 0)
@@
     (pin "1")
   )
-  (symbol (lib_id "power:GND") (at 25.4 133.35 0) (mirror y)
+  (symbol (lib_id "power:GND") (at 25.4 133.35 0) (mirror y) (unit 1)
     (in_bom yes) (on_board yes)
     (property "Reference" "#PWR0111" (id 0) (at 25.4 139.7 0)
@@
     (pin "1")
   )
-  (symbol (lib_id "power:GND") (at 34.29 133.35 0)
+  (symbol (lib_id "power:GND") (at 34.29 133.35 0) (unit 1)
     (in_bom yes) (on_board yes)
     (property "Reference" "#PWR0304" (id 0) (at 34.29 139.7 0)
@@
     (pin "1")
   )
-  (symbol (lib_id "power:GND") (at 43.18 133.35 0)
+  (symbol (lib_id "power:GND") (at 43.18 133.35 0) (unit 1)
     (in_bom yes) (on_board yes)
     (property "Reference" "#PWR0303" (id 0) (at 43.18 139.7 0)
@@
     (pin "1")
   )
-  (symbol (lib_id "power:GND") (at 52.07 135.89 0)
+  (symbol (lib_id "power:GND") (at 52.07 135.89 0) (unit 1)
     (in_bom yes) (on_board yes)
     (property "Reference" "#PWR0309" (id 0) (at 52.07 142.24 0)
@@
     (pin "1")
   )
-  (symbol (lib_id "power:GND") (at 76.2 130.81 0)
+  (symbol (lib_id "power:GND") (at 76.2 130.81 0) (unit 1)
     (in_bom yes) (on_board yes)
     (property "Reference" "#PWR0113" (id 0) (at 76.2 137.16 0)
@@
     (pin "1")
   )
-  (symbol (lib_id "power:GND") (at 92.71 133.35 0)
+  (symbol (lib_id "power:GND") (at 92.71 133.35 0) (unit 1)
     (in_bom yes) (on_board yes)
     (property "Reference" "#PWR0301" (id 0) (at 92.71 139.7 0)
@@
     (pin "1")
   )
-  (symbol (lib_id "power:GND") (at 118.11 133.35 0)
+  (symbol (lib_id "power:GND") (at 118.11 133.35 0) (unit 1)
     (in_bom yes) (on_board yes)
     (property "Reference" "#PWR0305" (id 0) (at 118.11 139.7 0)
@@
     (pin "1")
   )
-  (symbol (lib_id "power:GND") (at 124.46 133.35 0) (mirror y)
+  (symbol (lib_id "power:GND") (at 124.46 133.35 0) (mirror y) (unit 1)
     (in_bom yes) (on_board yes)
     (property "Reference" "#PWR0310" (id 0) (at 124.46 139.7 0)
@@
     (pin "1")
   )
-  (symbol (lib_id "power:GND") (at 134.62 133.35 0)
+  (symbol (lib_id "power:GND") (at 134.62 133.35 0) (unit 1)
     (in_bom yes) (on_board yes)
     (property "Reference" "#PWR0115" (id 0) (at 134.62 139.7 0)
@@
     (pin "1")
   )
-  (symbol (lib_id "power:GND") (at 154.94 156.21 0)
+  (symbol (lib_id "power:GND") (at 154.94 156.21 0) (unit 1)
     (in_bom yes) (on_board yes)
     (property "Reference" "#PWR0306" (id 0) (at 154.94 162.56 0)
@@
     (pin "1")
   )
-  (symbol (lib_id "power:GND") (at 170.18 83.82 0)
+  (symbol (lib_id "power:GND") (at 170.18 83.82 0) (unit 1)
     (in_bom yes) (on_board yes)
     (property "Reference" "#PWR0117" (id 0) (at 170.18 90.17 0)
@@
     (pin "1")
   )
-  (symbol (lib_id "power:GND") (at 200.66 92.71 0)
+  (symbol (lib_id "power:GND") (at 200.66 92.71 0) (unit 1)
     (in_bom yes) (on_board yes)
     (property "Reference" "#PWR0118" (id 0) (at 200.66 99.06 0)
@@
     (pin "1")
   )
-  (symbol (lib_id "power:GND") (at 214.63 142.24 0)
+  (symbol (lib_id "power:GND") (at 214.63 142.24 0) (unit 1)
     (in_bom yes) (on_board yes)
     (property "Reference" "#PWR0313" (id 0) (at 214.63 148.59 0)
@@
     (pin "1")
   )
-  (symbol (lib_id "power:GND") (at 226.06 142.24 0)
+  (symbol (lib_id "power:GND") (at 226.06 142.24 0) (unit 1)
     (in_bom yes) (on_board yes)
     (property "Reference" "#PWR0312" (id 0) (at 226.06 148.59 0)
@@
     (pin "1")
   )
-  (symbol (lib_id "power:GND") (at 232.41 40.64 0)
+  (symbol (lib_id "power:GND") (at 232.41 40.64 0) (unit 1)
     (in_bom yes) (on_board yes)
     (property "Reference" "#PWR0307" (id 0) (at 232.41 46.99 0)
@@
     (pin "1")
   )
-  (symbol (lib_id "power:GND") (at 238.76 48.26 0)
+  (symbol (lib_id "power:GND") (at 238.76 48.26 0) (unit 1)
     (in_bom yes) (on_board yes)
     (property "Reference" "#PWR0116" (id 0) (at 238.76 54.61 0)
@@
     (pin "1")
   )
-  (symbol (lib_id "power:GND") (at 238.76 85.09 0)
+  (symbol (lib_id "power:GND") (at 238.76 85.09 0) (unit 1)
     (in_bom yes) (on_board yes)
     (property "Reference" "#PWR0308" (id 0) (at 238.76 91.44 0)
@@
     (pin "1")
   )
-  (symbol (lib_id "Device:L") (at 106.68 115.57 90)
+  (symbol (lib_id "Device:L") (at 106.68 115.57 90) (unit 1)
     (in_bom yes) (on_board yes)
     (property "Reference" "L301" (id 0) (at 106.68 110.744 90))
@@
     (pin "2")
   )
-  (symbol (lib_id "Device:R") (at 154.94 121.92 0)
+  (symbol (lib_id "Device:R") (at 154.94 121.92 0) (unit 1)
     (in_bom yes) (on_board yes)
     (property "Reference" "R302" (id 0) (at 158.75 120.65 0))
@@
     (pin "2")
   )
-  (symbol (lib_id "Device:R") (at 154.94 148.59 0)
+  (symbol (lib_id "Device:R") (at 154.94 148.59 0) (unit 1)
     (in_bom yes) (on_board yes)
     (property "Reference" "R303" (id 0) (at 156.718 147.4216 0)
@@
     (pin "2")
   )
-  (symbol (lib_id "Device:C") (at 25.4 121.92 0) (mirror y)
+  (symbol (lib_id "Device:C") (at 25.4 121.92 0) (mirror y) (unit 1)
     (in_bom yes) (on_board yes)
     (property "Reference" "C314" (id 0) (at 22.479 120.7516 0)
@@
     (pin "2")
   )
-  (symbol (lib_id "Device:C") (at 82.55 107.95 270)
+  (symbol (lib_id "Device:C") (at 82.55 107.95 270) (unit 1)
     (in_bom yes) (on_board yes)
     (property "Reference" "C304" (id 0) (at 82.55 101.5492 90))
@@
     (pin "2")
   )
-  (symbol (lib_id "Device:C") (at 118.11 121.92 0) (mirror y)
+  (symbol (lib_id "Device:C") (at 118.11 121.92 0) (mirror y) (unit 1)
     (in_bom yes) (on_board yes)
     (property "Reference" "C305" (id 0) (at 115.189 120.7516 0)
@@
     (pin "2")
   )
-  (symbol (lib_id "Device:C") (at 124.46 121.92 0)
+  (symbol (lib_id "Device:C") (at 124.46 121.92 0) (unit 1)
     (in_bom yes) (on_board yes)
     (property "Reference" "C311" (id 0) (at 127.381 120.7516 0)
@@
     (pin "2")
   )
-  (symbol (lib_id "Device:C") (at 232.41 36.83 180)
+  (symbol (lib_id "Device:C_Polarized") (at 226.06 135.89 0) (unit 1)
+    (in_bom yes) (on_board yes)
+    (property "Reference" "C309" (id 0) (at 229.0572 134.7216 0)
+      (effects (font (size 1.27 1.27)) (justify left))
+    )
+    (property "Value" "CXHP2R7606R-TW" (id 1) (at 229.0572 137.033 0)
+      (effects (font (size 1.27 1.27)) (justify left))
+    )
+    (property "Footprint" "SH-RPi:CP_Radial_D18.0mm_P7.50mm_flat" (id 2) (at 227.0252 139.7 0)
+      (effects (font (size 1.27 1.27)) hide)
+    )
+    (property "Datasheet" "~" (id 3) (at 226.06 135.89 0)
+      (effects (font (size 1.27 1.27)) hide)
+    )
+    (pin "1")
+    (pin "2")
+  )
+  (symbol (lib_id "Device:C") (at 232.41 36.83 180) (unit 1)
     (in_bom yes) (on_board yes)
     (property "Reference" "C307" (id 0) (at 227.33 35.56 0))
@@
     (pin "2")
   )
-  (symbol (lib_id "Device:C") (at 238.76 77.47 180)
+  (symbol (lib_id "Device:C") (at 238.76 77.47 180) (unit 1)
     (in_bom yes) (on_board yes)
     (property "Reference" "C301" (id 0) (at 233.68 76.2 0))
@@
     (pin "2")
   )
-  (symbol (lib_id "Device:CP") (at 226.06 135.89 0) (unit 1)
-    (in_bom yes) (on_board yes)
-    (property "Reference" "C309" (id 0) (at 229.0572 134.7216 0)
-      (effects (font (size 1.27 1.27)) (justify left))
-    )
-    (property "Value" "CXHP2R7606R-TW" (id 1) (at 229.0572 137.033 0)
-      (effects (font (size 1.27 1.27)) (justify left))
-    )
-    (property "Footprint" "SH-RPi:CP_Radial_D18.0mm_P7.50mm_flat" (id 2) (at 227.0252 139.7 0)
-      (effects (font (size 1.27 1.27)) hide)
-    )
-    (property "Datasheet" "~" (id 3) (at 226.06 135.89 0)
-      (effects (font (size 1.27 1.27)) hide)
-    )
-  )
   (symbol (lib_id "SH-RPi:HT75xx-1-SOT23") (at 58.42 173.99 0) (unit 1)

Commit message: Revert the Rev. 1.0.1 LDO change
The new part exhibited severe startup overshoot
which disabled or even damaged the MCU.
Parts:
- U301: value PJ75AL33SA -> H7533-H#; LCSC C411736 -> C277872
Changed lines of the file:
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@@
     (in_bom yes) (on_board yes)
     (property "Reference" "U301" (id 0) (at 58.42 164.6682 0))
-    (property "Value" "PJ75AL33SA" (id 1) (at 58.42 166.9796 0))
+    (property "Value" "H7533-H#" (id 1) (at 58.42 166.9796 0))
     (property "Footprint" "Package_TO_SOT_SMD:SOT-23" (id 2) (at 58.42 165.735 0)
       (effects (font (size 1.27 1.27) italic) hide)
     )
-    (property "Datasheet" "" (id 3) (at 58.42 171.45 0)
+    (property "Datasheet" "https://datasheet.lcsc.com/szlcsc/Siproin-H7533-H_C277872.pdf" (id 3) (at 58.42 171.45 0)
       (effects (font (size 1.27 1.27)) hide)
     )
-    (property "LCSC" "C411736" (id 4) (at 58.42 173.99 0)
+    (property "LCSC" "C277872" (id 4) (at 58.42 173.99 0)
       (effects (font (size 1.27 1.27)) hide)
     )
