File: canbus.kicad_sch (KiCad schematic)
At the start: 28 parts, among them J801 JST XH horiz, J802 Wire Link, U802 PJ75AL50SA, U803 MCP2515-xST, U804 ISO1050DUB, Y801 X322516MLB4SI

Commit message: Fix broken symbols
Parts:
- FB801: symbol Device:Ferrite_Bead -> Device:FerriteBead
Connections:
- net CAN12V_fused: now also FB801.1
- net at F801.1: now also FB801.2
Changed lines of the file:
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@@
     (pin "1")
   )
-  (symbol (lib_id "power:PWR_FLAG") (at 57.15 36.83 0)
+  (symbol (lib_id "power:PWR_FLAG") (at 57.15 36.83 0) (unit 1)
     (in_bom yes) (on_board yes)
     (property "Reference" "#FLG0801" (id 0) (at 57.15 34.925 0)
@@
     (pin "1")
   )
-  (symbol (lib_id "power:PWR_FLAG") (at 106.68 154.94 180)
+  (symbol (lib_id "power:PWR_FLAG") (at 106.68 154.94 180) (unit 1)
     (in_bom yes) (on_board yes)
     (property "Reference" "#FLG0802" (id 0) (at 106.68 156.845 0)
@@
     (pin "1")
   )
-  (symbol (lib_id "power:PWR_FLAG") (at 128.27 166.37 270)
+  (symbol (lib_id "power:PWR_FLAG") (at 128.27 166.37 270) (unit 1)
     (in_bom yes) (on_board yes)
     (property "Reference" "#FLG0803" (id 0) (at 130.175 166.37 0)
@@
     (pin "2")
   )
-  (symbol (lib_id "Device:R") (at 209.55 104.14 0)
+  (symbol (lib_id "Device:R") (at 209.55 104.14 0) (unit 1)
     (in_bom yes) (on_board yes)
     (property "Reference" "R804" (id 0) (at 211.328 102.9716 0)
@@
     (pin "2")
   )
-  (symbol (lib_id "Device:R") (at 222.25 104.14 0)
+  (symbol (lib_id "Device:R") (at 222.25 104.14 0) (unit 1)
     (in_bom yes) (on_board yes)
     (property "Reference" "R805" (id 0) (at 224.028 102.9716 0)
@@
     (pin "2")
   )
-  (symbol (lib_id "Device:R") (at 233.68 104.14 0)
+  (symbol (lib_id "Device:R") (at 233.68 104.14 0) (unit 1)
     (in_bom yes) (on_board yes)
     (property "Reference" "R806" (id 0) (at 235.458 102.9716 0)
@@
     (pin "2")
   )
-  (symbol (lib_id "Device:D_TVS") (at 87.63 162.56 270)
+  (symbol (lib_id "Device:D_TVS") (at 87.63 162.56 270) (unit 1)
     (in_bom yes) (on_board yes)
     (property "Reference" "D801" (id 0) (at 89.6366 161.3916 90)
@@
     (pin "2")
   )
-  (symbol (lib_id "Device:D") (at 97.79 154.94 180)
+  (symbol (lib_id "Device:D") (at 97.79 154.94 180) (unit 1)
     (in_bom yes) (on_board yes)
     (property "Reference" "D802" (id 0) (at 97.79 149.4536 0))
@@
     (pin "2")
   )
-  (symbol (lib_id "Device:Polyfuse") (at 44.45 154.94 270)
+  (symbol (lib_id "Device:Polyfuse") (at 44.45 154.94 270) (unit 1)
     (in_bom yes) (on_board yes)
     (property "Reference" "F801" (id 0) (at 44.45 149.225 90))
@@
     (pin "2")
   )
-  (symbol (lib_id "Device:LED") (at 209.55 115.57 90)
+  (symbol (lib_id "Device:LED") (at 209.55 115.57 90) (unit 1)
     (in_bom yes) (on_board yes)
     (property "Reference" "D803" (id 0) (at 212.5218 114.6048 90)
@@
     (pin "2")
   )
-  (symbol (lib_id "Device:LED") (at 222.25 115.57 90)
+  (symbol (lib_id "Device:LED") (at 222.25 115.57 90) (unit 1)
     (in_bom yes) (on_board yes)
     (property "Reference" "D804" (id 0) (at 225.2218 114.6048 90)
@@
     (pin "2")
   )
-  (symbol (lib_id "Device:LED") (at 233.68 115.57 90)
+  (symbol (lib_id "Device:LED") (at 233.68 115.57 90) (unit 1)
     (in_bom yes) (on_board yes)
     (property "Reference" "D805" (id 0) (at 236.6518 114.6048 90)
@@
     (pin "2")
   )
-  (symbol (lib_id "Device:C") (at 71.12 163.83 0)
+  (symbol (lib_id "Device:C") (at 71.12 163.83 0) (unit 1)
     (in_bom yes) (on_board yes)
     (property "Reference" "C801" (id 0) (at 74.041 162.6616 0)
@@
     (pin "2")
   )
-  (symbol (lib_id "Device:C") (at 113.03 163.83 0)
+  (symbol (lib_id "Device:C") (at 113.03 163.83 0) (unit 1)
     (in_bom yes) (on_board yes)
     (property "Reference" "C802" (id 0) (at 115.951 162.6616 0)
@@
     (pin "2")
   )
-  (symbol (lib_id "Device:C") (at 144.78 163.83 0)
+  (symbol (lib_id "Device:C") (at 144.78 163.83 0) (unit 1)
     (in_bom yes) (on_board yes)
     (property "Reference" "C805" (id 0) (at 147.701 162.6616 0)
@@
     (pin "2")
   )
-  (symbol (lib_id "Device:C") (at 167.64 39.37 0)
+  (symbol (lib_id "Device:C") (at 167.64 39.37 0) (unit 1)
     (in_bom yes) (on_board yes)
     (property "Reference" "C806" (id 0) (at 170.561 38.2016 0)
@@
     (pin "2")
   )
-  (symbol (lib_id "Device:C") (at 190.5 44.45 0)
+  (symbol (lib_id "Device:C") (at 190.5 44.45 0) (unit 1)
     (in_bom yes) (on_board yes)
     (property "Reference" "C807" (id 0) (at 193.421 43.2816 0)
@@
     (pin "2")
   )
-  (symbol (lib_id "Device:C") (at 238.76 60.96 0)
+  (symbol (lib_id "Device:C") (at 238.76 60.96 0) (unit 1)
     (in_bom yes) (on_board yes)
     (property "Reference" "C808" (id 0) (at 241.681 59.7916 0)
@@
     (pin "2")
   )
-  (symbol (lib_id "Connector_Generic:Conn_01x04") (at 35.56 41.91 0) (mirror y)
+  (symbol (lib_id "Device:FerriteBead") (at 60.96 154.94 270) (unit 1)
+    (in_bom yes) (on_board yes)
+    (property "Reference" "FB801" (id 0) (at 60.96 147.9804 90))
+    (property "Value" "GZ2012D601TF" (id 1) (at 60.96 150.2918 90))
+    (property "Footprint" "Inductor_SMD:L_0805_2012Metric" (id 2) (at 60.96 153.162 90)
+      (effects (font (size 1.27 1.27)) hide)
+    )
+    (property "Datasheet" "~" (id 3) (at 60.96 154.94 0)
+      (effects (font (size 1.27 1.27)) hide)
+    )
+    (property "LCSC" "C1017" (id 4) (at 60.96 154.94 90)
+      (effects (font (size 1.27 1.27)) hide)
+    )
+    (pin "1")
+    (pin "2")
+  )
+  (symbol (lib_id "Connector_Generic:Conn_01x04") (at 35.56 41.91 0) (mirror y) (unit 1)
     (in_bom yes) (on_board yes)
     (property "Reference" "J801" (id 0) (at 37.592 52.705 0))
@@
     (pin "4")
   )
-  (symbol (lib_id "Device:Ferrite_Bead") (at 60.96 154.94 270)
-    (in_bom yes) (on_board yes)
-    (property "Reference" "FB801" (id 0) (at 60.96 147.9804 90))
-    (property "Value" "GZ2012D601TF" (id 1) (at 60.96 150.2918 90))
-    (property "Footprint" "Inductor_SMD:L_0805_2012Metric" (id 2) (at 60.96 153.162 90)
-      (effects (font (size 1.27 1.27)) hide)
-    )
-    (property "Datasheet" "~" (id 3) (at 60.96 154.94 0)
-      (effects (font (size 1.27 1.27)) hide)
-    )
-    (property "LCSC" "C1017" (id 4) (at 60.96 154.94 90)
-      (effects (font (size 1.27 1.27)) hide)
-    )
-  )
-  (symbol (lib_id "SH-RPi:HT75xx-1-SOT23") (at 128.27 157.48 0)
+  (symbol (lib_id "SH-RPi:HT75xx-1-SOT23") (at 128.27 157.48 0) (unit 1)
     (in_bom yes) (on_board yes)
     (property "Reference" "U802" (id 0) (at 128.27 148.1582 0))

Commit message: Revert the Rev. 1.0.1 LDO change
The new part exhibited severe startup overshoot
which disabled or even damaged the MCU.
Parts:
- U802: value PJ75AL50SA -> H7550-H#; LCSC C411735 -> C277875
Changed lines of the file:
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@@
     (in_bom yes) (on_board yes)
     (property "Reference" "U802" (id 0) (at 128.27 148.1582 0))
-    (property "Value" "PJ75AL50SA" (id 1) (at 128.27 150.4696 0))
+    (property "Value" "H7550-H#" (id 1) (at 128.27 150.4696 0))
     (property "Footprint" "Package_TO_SOT_SMD:SOT-23" (id 2) (at 128.27 149.225 0)
       (effects (font (size 1.27 1.27) italic) hide)
@@
       (effects (font (size 1.27 1.27)) hide)
     )
-    (property "LCSC" "C411735" (id 4) (at 128.27 157.48 0)
+    (property "LCSC" "C277875" (id 4) (at 128.27 157.48 0)
       (effects (font (size 1.27 1.27)) hide)
     )
