File: IO.kicad_sch (KiCad schematic)
At the start: 18 parts, among them J501 Raspberry_Pi_2_3, J502 Conn_01x02, J503 Conn_01x02

Commit message: Finish PCB routing
Connections:
- net +3.3V is gone; now on net +3V3: J501.1 (3V3), J501.17 (3V3)
- net +5V: now also D502.2 (A2), D503.2 (A2), J502.2 (Pin_2), J503.1 (Pin_1)
- net GND: now also J502.1 (Pin_1); no longer J502.2 (Pin_2)
- removed net 5V: D502.2 (A2), D503.2 (A2), J502.1 (Pin_1), J503.1 (Pin_1)
Changed lines of the file:
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@@
     (effects (font (size 1.27 1.27)) (justify left bottom))
-  )
-  (global_label "5V" (shape bidirectional) (at 138.43 138.43 180) (fields_autoplaced)
-    (effects (font (size 1.27 1.27)) (justify right))
-    (property "Intersheet References" "${INTERSHEET_REFS}" (id 0) (at -25.4 38.1 0)
-      (effects (font (size 1.27 1.27)) hide)
-    )
-  )
-  (global_label "5V" (shape bidirectional) (at 138.43 115.57 180) (fields_autoplaced)
-    (effects (font (size 1.27 1.27)) (justify right))
-    (property "Intersheet References" "${INTERSHEET_REFS}" (id 0) (at -25.4 15.24 0)
-      (effects (font (size 1.27 1.27)) hide)
-    )
   )
   (hierarchical_label "SDA" (shape input) (at 80.01 60.96 0)
@@
     (pin "2")
   )
-  (symbol (lib_id "power:+3.3V") (at 62.23 25.4 0) (unit 1)
-    (in_bom yes) (on_board yes)
-    (property "Reference" "#PWR0507" (id 0) (at 62.23 29.21 0)
-      (effects (font (size 1.27 1.27)) hide)
-    )
-    (property "Value" "+3.3V" (id 1) (at 62.611 21.0058 0))
-    (property "Footprint" "" (id 2) (at 62.23 25.4 0)
-      (effects (font (size 1.27 1.27)) hide)
-    )
-    (property "Datasheet" "" (id 3) (at 62.23 25.4 0)
-      (effects (font (size 1.27 1.27)) hide)
-    )
-    (pin "1")
-  )
   (symbol (lib_id "Connector_Generic:Conn_01x02") (at 171.45 138.43 0) (unit 1)
     (in_bom yes) (on_board yes)
@@
     (pin "1")
   )
-  (symbol (lib_id "Connector_Generic:Conn_01x02") (at 171.45 115.57 0) (unit 1)
-    (in_bom yes) (on_board yes)
-    (property "Reference" "J502" (id 0) (at 169.3672 123.825 0))
-    (property "Value" "Conn_01x02" (id 1) (at 169.3672 121.5136 0))
-    (property "Footprint" "Connector_Phoenix_MC:PhoenixContact_MC_1,5_2-G-3.81_1x02_P3.81mm_Horizontal" (id 2) (at 171.45 115.57 0)
-      (effects (font (size 1.27 1.27)) hide)
-    )
-    (property "Datasheet" "~" (id 3) (at 171.45 115.57 0)
-      (effects (font (size 1.27 1.27)) hide)
-    )
-    (property "LCSC" "C8387" (id 4) (at 171.45 115.57 0)
+  (symbol (lib_id "Connector_Generic:Conn_01x02") (at 171.45 118.11 0) (mirror x) (unit 1)
+    (in_bom yes) (on_board yes)
+    (property "Reference" "J502" (id 0) (at 169.3672 109.855 0))
+    (property "Value" "Conn_01x02" (id 1) (at 169.3672 112.1664 0))
+    (property "Footprint" "Connector_Phoenix_MC:PhoenixContact_MC_1,5_2-G-3.81_1x02_P3.81mm_Horizontal" (id 2) (at 171.45 118.11 0)
+      (effects (font (size 1.27 1.27)) hide)
+    )
+    (property "Datasheet" "~" (id 3) (at 171.45 118.11 0)
+      (effects (font (size 1.27 1.27)) hide)
+    )
+    (property "LCSC" "C8387" (id 4) (at 171.45 118.11 0)
       (effects (font (size 1.27 1.27)) hide)
     )
@@
     (pin "1")
   )
+  (symbol (lib_id "power:+5V") (at 138.43 115.57 0) (unit 1)
+    (in_bom yes) (on_board yes) (fields_autoplaced)
+    (property "Reference" "#PWR0104" (id 0) (at 138.43 119.38 0)
+      (effects (font (size 1.27 1.27)) hide)
+    )
+    (property "Value" "+5V" (id 1) (at 138.43 110.49 0))
+    (property "Footprint" "" (id 2) (at 138.43 115.57 0)
+      (effects (font (size 1.27 1.27)) hide)
+    )
+    (property "Datasheet" "" (id 3) (at 138.43 115.57 0)
+      (effects (font (size 1.27 1.27)) hide)
+    )
+    (pin "1")
+  )
   (symbol (lib_id "power:+3V3") (at 171.45 29.21 0) (unit 1)
     (in_bom yes) (on_board yes) (fields_autoplaced)
@@
     (pin "2")
   )
+  (symbol (lib_id "power:+3V3") (at 62.23 25.4 0) (unit 1)
+    (in_bom yes) (on_board yes) (fields_autoplaced)
+    (property "Reference" "#PWR0103" (id 0) (at 62.23 29.21 0)
+      (effects (font (size 1.27 1.27)) hide)
+    )
+    (property "Value" "+3V3" (id 1) (at 62.23 20.32 0))
+    (property "Footprint" "" (id 2) (at 62.23 25.4 0)
+      (effects (font (size 1.27 1.27)) hide)
+    )
+    (property "Datasheet" "" (id 3) (at 62.23 25.4 0)
+      (effects (font (size 1.27 1.27)) hide)
+    )
+    (pin "1")
+  )
   (symbol (lib_id "Device:D_TVS") (at 120.65 49.53 90) (unit 1)
     (in_bom yes) (on_board yes) (fields_autoplaced)
@@
       (effects (font (size 1.27 1.27)) hide)
     )
+    (pin "1")
+  )
+  (symbol (lib_id "power:+5V") (at 138.43 138.43 0) (unit 1)
+    (in_bom yes) (on_board yes) (fields_autoplaced)
+    (property "Reference" "#PWR0105" (id 0) (at 138.43 142.24 0)
+      (effects (font (size 1.27 1.27)) hide)
+    )
+    (property "Value" "+5V" (id 1) (at 138.43 133.35 0))
+    (property "Footprint" "" (id 2) (at 138.43 138.43 0)
+      (effects (font (size 1.27 1.27)) hide)
+    )
+    (property "Datasheet" "" (id 3) (at 138.43 138.43 0)
+      (effects (font (size 1.27 1.27)) hide)
+    )

Commit message: Replace "ideal diode" with Schottky & other changes
Parts:
- added TP501: SDA, TestPoint:TestPoint_Pad_D2.0mm, symbol Connector:TestPoint
- added TP502: SCL, TestPoint:TestPoint_Pad_D2.0mm, symbol Connector:TestPoint
Connections:
- net SCL: now also TP502.1
- net SDA: now also TP501.1
Changed lines of the file:
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@@
   (title_block
     (title "Sailor Hat for Raspberry Pi")
-    (date "2022-10-14")
-    (rev "v2.0.0-alpha")
+    (date "2022-10-21")
+    (rev "v2.0.0-a1")
     (company "Hat Labs Ltd")
     (comment 1 "https://creativecommons.org/licenses/by/4.0")
@@
   )
   (junction (at 54.61 40.64) (diameter 0) (color 0 0 0 0)
-  )
-  (junction (at 64.77 33.02) (diameter 0) (color 0 0 0 0)
   )
   (junction (at 62.23 31.75) (diameter 0) (color 0 0 0 0)
@@
     (stroke (width 0) (type default) (color 0 0 0 0))
   )
+  (wire (pts (xy 118.11 82.55) (xy 121.92 82.55))
+    (stroke (width 0) (type default) (color 0 0 0 0))
+  )
   (wire (pts (xy 154.94 39.37) (xy 154.94 41.91))
     (stroke (width 0) (type default) (color 0 0 0 0))
   )
+  (wire (pts (xy 118.11 80.01) (xy 118.11 82.55))
+    (stroke (width 0) (type default) (color 0 0 0 0))
+  )
   (wire (pts (xy 57.15 40.64) (xy 54.61 40.64))
     (stroke (width 0) (type default) (color 0 0 0 0))
@@
     (stroke (width 0) (type default) (color 0 0 0 0))
   )
+  (wire (pts (xy 118.11 96.52) (xy 121.92 96.52))
+    (stroke (width 0) (type default) (color 0 0 0 0))
+  )
   (wire (pts (xy 62.23 31.75) (xy 62.23 43.18))
     (stroke (width 0) (type default) (color 0 0 0 0))
@@
     (stroke (width 0) (type default) (color 0 0 0 0))
   )
+  (wire (pts (xy 118.11 92.71) (xy 118.11 96.52))
+    (stroke (width 0) (type default) (color 0 0 0 0))
+  )
   (wire (pts (xy 171.45 53.34) (xy 171.45 57.15))
     (stroke (width 0) (type default) (color 0 0 0 0))
@@
     (stroke (width 0) (type default) (color 0 0 0 0))
   )
-  (wire (pts (xy 64.77 31.75) (xy 64.77 33.02))
-    (stroke (width 0) (type default) (color 0 0 0 0))
-  )
   (wire (pts (xy 219.71 54.61) (xy 219.71 57.15))
     (stroke (width 0) (type default) (color 0 0 0 0))
@@
     (stroke (width 0) (type default) (color 0 0 0 0))
   )
-  (wire (pts (xy 64.77 33.02) (xy 64.77 43.18))
+  (wire (pts (xy 64.77 31.75) (xy 64.77 43.18))
     (stroke (width 0) (type default) (color 0 0 0 0))
   )
@@
     (effects (font (size 1.27 1.27)) (justify right))
   )
+  (hierarchical_label "SCL" (shape input) (at 121.92 96.52 0)
+    (effects (font (size 1.27 1.27)) (justify left))
+  )
   (hierarchical_label "RXD0" (shape input) (at 39.37 55.88 180)
     (effects (font (size 1.27 1.27)) (justify right))
   )
   (hierarchical_label "RXD5" (shape input) (at 80.01 96.52 0)
+    (effects (font (size 1.27 1.27)) (justify left))
+  )
+  (hierarchical_label "SDA" (shape input) (at 121.92 82.55 0)
     (effects (font (size 1.27 1.27)) (justify left))
   )
@@
   (symbol (lib_id "power:GND") (at 265.43 66.04 0) (unit 1)
     (in_bom yes) (on_board yes)
-    (property "Reference" "#PWR0524" (id 0) (at 265.43 72.39 0)
+    (property "Reference" "#PWR0526" (id 0) (at 265.43 72.39 0)
       (effects (font (size 1.27 1.27)) hide)
     )
@@
   (symbol (lib_id "power:GND") (at 250.19 66.04 0) (unit 1)
     (in_bom yes) (on_board yes)
-    (property "Reference" "#PWR0523" (id 0) (at 250.19 72.39 0)
+    (property "Reference" "#PWR0525" (id 0) (at 250.19 72.39 0)
       (effects (font (size 1.27 1.27)) hide)
     )
@@
   (symbol (lib_id "power:GND") (at 234.95 66.04 0) (unit 1)
     (in_bom yes) (on_board yes)
-    (property "Reference" "#PWR0522" (id 0) (at 234.95 72.39 0)
+    (property "Reference" "#PWR0524" (id 0) (at 234.95 72.39 0)
       (effects (font (size 1.27 1.27)) hide)
     )
@@
   (symbol (lib_id "power:GND") (at 219.71 66.04 0) (unit 1)
     (in_bom yes) (on_board yes)
-    (property "Reference" "#PWR0521" (id 0) (at 219.71 72.39 0)
+    (property "Reference" "#PWR0523" (id 0) (at 219.71 72.39 0)
       (effects (font (size 1.27 1.27)) hide)
     )
@@
   (symbol (lib_id "power:GND") (at 162.56 147.32 0) (unit 1)
     (in_bom yes) (on_board yes)
-    (property "Reference" "#PWR0518" (id 0) (at 162.56 153.67 0)
+    (property "Reference" "#PWR0520" (id 0) (at 162.56 153.67 0)
       (effects (font (size 1.27 1.27)) hide)
     )
@@
   (symbol (lib_id "power:GND") (at 162.56 124.46 0) (unit 1)
     (in_bom yes) (on_board yes)
-    (property "Reference" "#PWR0517" (id 0) (at 162.56 130.81 0)
+    (property "Reference" "#PWR0519" (id 0) (at 162.56 130.81 0)
       (effects (font (size 1.27 1.27)) hide)
     )
@@
   (symbol (lib_id "power:GND") (at 146.05 124.46 0) (unit 1)
     (in_bom yes) (on_board yes)
-    (property "Reference" "#PWR0513" (id 0) (at 146.05 130.81 0)
+    (property "Reference" "#PWR0515" (id 0) (at 146.05 130.81 0)
       (effects (font (size 1.27 1.27)) hide)
     )
@@
   (symbol (lib_id "power:GND") (at 146.05 147.32 0) (unit 1)
     (in_bom yes) (on_board yes)
-    (property "Reference" "#PWR0514" (id 0) (at 146.05 153.67 0)
+    (property "Reference" "#PWR0516" (id 0) (at 146.05 153.67 0)
       (effects (font (size 1.27 1.27)) hide)
     )
@@
   (symbol (lib_id "power:GND") (at 154.94 57.15 0) (unit 1)
     (in_bom yes) (on_board yes)
-    (property "Reference" "#PWR0516" (id 0) (at 154.94 63.5 0)
+    (property "Reference" "#PWR0518" (id 0) (at 154.94 63.5 0)
       (effects (font (size 1.27 1.27)) hide)
     )
@@
   (symbol (lib_id "power:+5V") (at 138.43 115.57 0) (unit 1)
     (in_bom yes) (on_board yes) (fields_autoplaced)
-    (property "Reference" "#PWR0104" (id 0) (at 138.43 119.38 0)
+    (property "Reference" "#PWR0513" (id 0) (at 138.43 119.38 0)
       (effects (font (size 1.27 1.27)) hide)
     )
@@
   (symbol (lib_id "power:+3V3") (at 171.45 29.21 0) (unit 1)
     (in_bom yes) (on_board yes) (fields_autoplaced)
-    (property "Reference" "#PWR0519" (id 0) (at 171.45 33.02 0)
+    (property "Reference" "#PWR0521" (id 0) (at 171.45 33.02 0)
       (effects (font (size 1.27 1.27)) hide)
     )
@@
   (symbol (lib_id "power:+3V3") (at 62.23 25.4 0) (unit 1)
     (in_bom yes) (on_board yes) (fields_autoplaced)
-    (property "Reference" "#PWR0103" (id 0) (at 62.23 29.21 0)
+    (property "Reference" "#PWR0507" (id 0) (at 62.23 29.21 0)
       (effects (font (size 1.27 1.27)) hide)
     )
@@
     (pin "2")
   )
+  (symbol (lib_id "Connector:TestPoint") (at 118.11 92.71 0) (unit 1)
+    (in_bom yes) (on_board yes) (fields_autoplaced)
+    (property "Reference" "TP502" (id 0) (at 120.65 88.1379 0)
+      (effects (font (size 1.27 1.27)) (justify left))
+    )
+    (property "Value" "SCL" (id 1) (at 120.65 90.6779 0)
+      (effects (font (size 1.27 1.27)) (justify left))
+    )
+    (property "Footprint" "TestPoint:TestPoint_Pad_D2.0mm" (id 2) (at 123.19 92.71 0)
+      (effects (font (size 1.27 1.27)) hide)
+    )
+    (property "Datasheet" "~" (id 3) (at 123.19 92.71 0)
+      (effects (font (size 1.27 1.27)) hide)
+    )
+    (pin "1")
+  )
   (symbol (lib_id "Device:LED") (at 250.19 60.96 90) (unit 1)
     (in_bom yes) (on_board yes)
@@
   (symbol (lib_id "power:+3V3") (at 154.94 29.21 0) (unit 1)
     (in_bom yes) (on_board yes) (fields_autoplaced)
-    (property "Reference" "#PWR0515" (id 0) (at 154.94 33.02 0)
+    (property "Reference" "#PWR0517" (id 0) (at 154.94 33.02 0)
       (effects (font (size 1.27 1.27)) hide)
     )
@@
     (pin "2")
   )
-  (symbol (lib_id "power:PWR_FLAG") (at 64.77 33.02 270) (unit 1)
-    (in_bom yes) (on_board yes) (fields_autoplaced)
-    (property "Reference" "#FLG0501" (id 0) (at 66.675 33.02 0)
-      (effects (font (size 1.27 1.27)) hide)
-    )
-    (property "Value" "PWR_FLAG" (id 1) (at 68.58 33.0199 90)
-      (effects (font (size 1.27 1.27)) (justify left))
-    )
-    (property "Footprint" "" (id 2) (at 64.77 33.02 0)
-      (effects (font (size 1.27 1.27)) hide)
-    )
-    (property "Datasheet" "~" (id 3) (at 64.77 33.02 0)
+  (symbol (lib_id "Connector:TestPoint") (at 118.11 80.01 0) (unit 1)
+    (in_bom yes) (on_board yes) (fields_autoplaced)
+    (property "Reference" "TP501" (id 0) (at 120.65 75.4379 0)
+      (effects (font (size 1.27 1.27)) (justify left))
+    )
+    (property "Value" "SDA" (id 1) (at 120.65 77.9779 0)
+      (effects (font (size 1.27 1.27)) (justify left))
+    )
+    (property "Footprint" "TestPoint:TestPoint_Pad_D2.0mm" (id 2) (at 123.19 80.01 0)
+      (effects (font (size 1.27 1.27)) hide)
+    )
+    (property "Datasheet" "~" (id 3) (at 123.19 80.01 0)
       (effects (font (size 1.27 1.27)) hide)
     )
@@
   (symbol (lib_id "power:+5V") (at 138.43 138.43 0) (unit 1)
     (in_bom yes) (on_board yes) (fields_autoplaced)
-    (property "Reference" "#PWR0105" (id 0) (at 138.43 142.24 0)
+    (property "Reference" "#PWR0514" (id 0) (at 138.43 142.24 0)
       (effects (font (size 1.27 1.27)) hide)
     )
@@
   (symbol (lib_id "power:GND") (at 171.45 57.15 0) (unit 1)
     (in_bom yes) (on_board yes)
-    (property "Reference" "#PWR0520" (id 0) (at 171.45 63.5 0)
-      (effects (font (size 1.27 1.27)) hide)
-    )
+    (property "Reference" "#PWR0522" (id 0) (at 171.45 63.5 0)
+      (effects (font (size 1.27 1.27)) hide)
+    )
