File: ldo.kicad_sch (KiCad schematic)
At the start: 3 parts

Commit message: SH-RPi v2 schematic design
Parts:
- added C902: 1uF/50V, Capacitor_SMD:C_0603_1608Metric, symbol Device:C
- added C904: 10uF/10V, Capacitor_SMD:C_0603_1608Metric, symbol Device:C
- added D901, D902, D903: 1N5819WS, Diode_SMD:D_SOD-323, symbol Device:D_Schottky
- added U902: SE8633X2-HF, Package_TO_SOT_SMD:SOT-89-3, symbol SH-RPi:HT75xx-1-SOT23
- C901: renamed from C302; LCSC C13585 -> C15849
- C903: renamed from C303; LCSC C19702 -> C15849
- U901: renamed from U301; value (none) -> SE8633X2-HF; footprint (none) -> Package_TO_SOT_SMD:SOT-89-3; LCSC C277872 -> C496613
Connections:
- net GND: now also C902.2, C904.2, U902.1 (GND)
- net REG3.3V: no longer names the net of C903.1, U901.2 (VOUT)
- net REG3.3V: now also D901.2 (A)
- net Vin renamed HS_Vin
- new net: D901.1 (K), D903.2 (A)
- new net: C904.1, D902.2 (A), U902.2 (VOUT)
- new net +3V3: D902.1 (K), D903.1 (K)
- new net LS_Vin: C902.1, U902.3 (VIN)
Other:
- note added: "Due to the diodes, output is actually less than 3.3V."
- note added: "Due to two schottky forward voltage drops, LS_Vin will always be preferred if both are available."
- moved on the sheet: C901, C903, U901

Commit message: WIP: Assign footprints and LCSC part numbers
Parts:
- C901: value (none) -> 1uF/50V; footprint (none) -> Capacitor_SMD:C_0805_2012Metric; LCSC C15849 -> C28323
- C902: value 1uF/50V -> 1uF/16V; footprint Capacitor_SMD:C_0603_1608Metric -> Capacitor_SMD:C_0504_1310Metric; LCSC C15849 -> C52923
- C903: value (none) -> 10uF/6.3V; footprint (none) -> Capacitor_SMD:C_0603_1608Metric; LCSC C15849 -> C19702
- C904: value 10uF/10V -> 10uF/6.3V; LCSC C15849 -> C19702
Changed lines of the file:
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@@
       (effects (font (size 1.27 1.27)) (justify left))
     )
-    (property "Value" "" (id 1) (at 127.381 76.073 0)
+    (property "Value" "10uF/6.3V" (id 1) (at 127.381 76.073 0)
       (effects (font (size 1.27 1.27)) (justify left))
     )
-    (property "Footprint" "" (id 2) (at 125.4252 78.74 0)
+    (property "Footprint" "Capacitor_SMD:C_0603_1608Metric" (id 2) (at 125.4252 78.74 0)
       (effects (font (size 1.27 1.27)) hide)
     )
@@
       (effects (font (size 1.27 1.27)) hide)
     )
-    (property "LCSC" "C15849" (id 4) (at 124.46 74.93 0)
+    (property "LCSC" "C19702" (id 4) (at 124.46 74.93 0)
       (effects (font (size 1.27 1.27)) hide)
     )
@@
       (effects (font (size 1.27 1.27)) (justify left))
     )
-    (property "Value" "" (id 1) (at 98.679 76.073 0)
+    (property "Value" "1uF/50V" (id 1) (at 98.679 76.073 0)
       (effects (font (size 1.27 1.27)) (justify left))
     )
-    (property "Footprint" "" (id 2) (at 100.6348 78.74 0)
+    (property "Footprint" "Capacitor_SMD:C_0805_2012Metric" (id 2) (at 100.6348 78.74 0)
       (effects (font (size 1.27 1.27)) hide)
     )
@@
       (effects (font (size 1.27 1.27)) hide)
     )
-    (property "LCSC" "C15849" (id 4) (at 101.6 74.93 0)
+    (property "LCSC" "C28323" (id 4) (at 101.6 74.93 0)
       (effects (font (size 1.27 1.27)) hide)
     )
@@
       (effects (font (size 1.27 1.27)) (justify left))
     )
-    (property "Value" "1uF/50V" (id 1) (at 98.679 109.093 0)
+    (property "Value" "1uF/16V" (id 1) (at 98.679 109.093 0)
       (effects (font (size 1.27 1.27)) (justify left))
     )
-    (property "Footprint" "Capacitor_SMD:C_0603_1608Metric" (id 2) (at 100.6348 111.76 0)
+    (property "Footprint" "Capacitor_SMD:C_0504_1310Metric" (id 2) (at 100.6348 111.76 0)
       (effects (font (size 1.27 1.27)) hide)
     )
@@
       (effects (font (size 1.27 1.27)) hide)
     )
-    (property "LCSC" "C15849" (id 4) (at 101.6 107.95 0)
+    (property "LCSC" "C52923" (id 4) (at 101.6 107.95 0)
       (effects (font (size 1.27 1.27)) hide)
     )
@@
       (effects (font (size 1.27 1.27)) hide)
     )
-    (property "Value" "" (id 1) (at 93.98 60.3504 0))
+    (property "Value" "PWR_FLAG" (id 1) (at 93.98 60.3504 0))
     (property "Footprint" "" (id 2) (at 93.98 64.77 0)
       (effects (font (size 1.27 1.27)) hide)
@@
       (effects (font (size 1.27 1.27)) (justify left))
     )
-    (property "Value" "10uF/10V" (id 1) (at 127.381 109.093 0)
+    (property "Value" "10uF/6.3V" (id 1) (at 127.381 109.093 0)
       (effects (font (size 1.27 1.27)) (justify left))
     )
@@
       (effects (font (size 1.27 1.27)) hide)
     )
-    (property "LCSC" "C15849" (id 4) (at 124.46 107.95 0)
+    (property "LCSC" "C19702" (id 4) (at 124.46 107.95 0)
       (effects (font (size 1.27 1.27)) hide)
     )
@@
       (effects (font (size 1.27 1.27)) hide)
     )
-    (property "Value" "" (id 1) (at 113.157 84.4042 0))
+    (property "Value" "GND" (id 1) (at 113.157 84.4042 0))
     (property "Footprint" "" (id 2) (at 113.03 80.01 0)
       (effects (font (size 1.27 1.27)) hide)

Commit message: WIP: PCB layout
Parts:
- C902: footprint Capacitor_SMD:C_0504_1310Metric -> Capacitor_SMD:C_0402_1005Metric
- U901, U902: footprint Package_TO_SOT_SMD:SOT-89-3 -> Package_TO_SOT_SMD:SOT-23
Connections:
- net HLDO_OUT: now reaches C903.1, D901.2 (A), U901.2 (VOUT)
- net LLDO_OUT: now reaches C904.1, D902.2 (A), U902.2 (VOUT)
Changed lines of the file:
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@@
+    (effects (font (size 1.27 1.27)) (justify left bottom))
+  )
+  (label "LLDO_OUT" (at 127 101.6 0)
+    (effects (font (size 1.27 1.27)) (justify left bottom))
+  )
+  (label "HLDO_OUT" (at 123.19 68.58 0)
     (effects (font (size 1.27 1.27)) (justify left bottom))
   )
@@
     (property "Reference" "U901" (id 0) (at 113.03 61.7982 0))
     (property "Value" "SE8633X2-HF" (id 1) (at 113.03 64.1096 0))
-    (property "Footprint" "Package_TO_SOT_SMD:SOT-89-3" (id 2) (at 113.03 62.865 0)
+    (property "Footprint" "Package_TO_SOT_SMD:SOT-23" (id 2) (at 113.03 62.865 0)
       (effects (font (size 1.27 1.27) italic) hide)
     )
@@
       (effects (font (size 1.27 1.27)) (justify left))
     )
-    (property "Footprint" "Capacitor_SMD:C_0504_1310Metric" (id 2) (at 100.6348 111.76 0)
+    (property "Footprint" "Capacitor_SMD:C_0402_1005Metric" (id 2) (at 100.6348 111.76 0)
       (effects (font (size 1.27 1.27)) hide)
     )
@@
     (property "Reference" "U902" (id 0) (at 113.03 94.8182 0))
     (property "Value" "SE8633X2-HF" (id 1) (at 113.03 97.1296 0))
-    (property "Footprint" "Package_TO_SOT_SMD:SOT-89-3" (id 2) (at 113.03 95.885 0)
+    (property "Footprint" "Package_TO_SOT_SMD:SOT-23" (id 2) (at 113.03 95.885 0)
       (effects (font (size 1.27 1.27) italic) hide)
     )

Commit message: Initial PCB component layout done
Parts:
- C903, C904: footprint Capacitor_SMD:C_0603_1608Metric -> Capacitor_SMD:C_0402_1005Metric; LCSC C19702 -> C15525
Changed lines of the file:
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@@
     (in_bom yes) (on_board yes)
     (property "Reference" "C903" (id 0) (at 127.381 73.7616 0)
-      (effects (font (size 1.27 1.27)) (justify left))
+      (effects (font (size 0 0)) (justify left))
     )
     (property "Value" "10uF/6.3V" (id 1) (at 127.381 76.073 0)
       (effects (font (size 1.27 1.27)) (justify left))
     )
-    (property "Footprint" "Capacitor_SMD:C_0603_1608Metric" (id 2) (at 125.4252 78.74 0)
+    (property "Footprint" "Capacitor_SMD:C_0402_1005Metric" (id 2) (at 125.4252 78.74 0)
       (effects (font (size 1.27 1.27)) hide)
     )
@@
       (effects (font (size 1.27 1.27)) hide)
     )
-    (property "LCSC" "C19702" (id 4) (at 124.46 74.93 0)
+    (property "LCSC" "C15525" (id 4) (at 124.46 74.93 0)
       (effects (font (size 1.27 1.27)) hide)
     )
@@
       (effects (font (size 1.27 1.27)) (justify left))
     )
-    (property "Footprint" "Capacitor_SMD:C_0603_1608Metric" (id 2) (at 125.4252 111.76 0)
+    (property "Footprint" "Capacitor_SMD:C_0402_1005Metric" (id 2) (at 125.4252 111.76 0)
       (effects (font (size 1.27 1.27)) hide)
     )
@@
       (effects (font (size 1.27 1.27)) hide)
     )
-    (property "LCSC" "C19702" (id 4) (at 124.46 107.95 0)
+    (property "LCSC" "C15525" (id 4) (at 124.46 107.95 0)
       (effects (font (size 1.27 1.27)) hide)
     )

Commit message: Replace "ideal diode" with Schottky & other changes
Parts:
- added TP901: HLDO, TestPoint:TestPoint_Pad_D2.0mm, symbol Connector:TestPoint
- added TP902: LLDO, TestPoint:TestPoint_Pad_D2.0mm, symbol Connector:TestPoint
Connections:
- net HLDO_OUT: now also TP901.1
- net LLDO_OUT: now also TP902.1
Other:
- note added: "Due to the diodes, output is actually less than 3.3V. If the host provides 3.3V, that is always preferred."
- note removed: "Due to the diodes, output is actually less than 3.3V."
Changed lines of the file:
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@@
   (title_block
     (title "Sailor Hat for Raspberry Pi")
-    (date "2022-10-14")
-    (rev "v2.0.0-alpha")
+    (date "2022-10-21")
+    (rev "v2.0.0-a1")
     (company "Hat Labs Ltd")
     (comment 1 "https://creativecommons.org/licenses/by/4.0")
@@
   (junction (at 124.46 101.6) (diameter 0) (color 0 0 0 0)
   )
+  (junction (at 121.92 101.6) (diameter 0) (color 0 0 0 0)
+  )
   (junction (at 124.46 68.58) (diameter 0) (color 0 0 0 0)
   )
   (junction (at 113.03 111.76) (diameter 0) (color 0 0 0 0)
   )
+  (junction (at 121.92 68.58) (diameter 0) (color 0 0 0 0)
+  )
   (junction (at 99.06 101.6) (diameter 0) (color 0 0 0 0)
   )
   (junction (at 101.6 68.58) (diameter 0) (color 0 0 0 0)
   )
+  (wire (pts (xy 121.92 68.58) (xy 124.46 68.58))
+    (stroke (width 0) (type default) (color 0 0 0 0))
+  )
   (wire (pts (xy 101.6 68.58) (xy 105.41 68.58))
     (stroke (width 0) (type default) (color 0 0 0 0))
@@
     (stroke (width 0) (type default) (color 0 0 0 0))
   )
+  (wire (pts (xy 121.92 101.6) (xy 124.46 101.6))
+    (stroke (width 0) (type default) (color 0 0 0 0))
+  )
   (wire (pts (xy 83.82 101.6) (xy 99.06 101.6))
     (stroke (width 0) (type default) (color 0 0 0 0))
@@
     (stroke (width 0) (type default) (color 0 0 0 0))
   )
+  (wire (pts (xy 124.46 68.58) (xy 133.35 68.58))
+    (stroke (width 0) (type default) (color 0 0 0 0))
+  )
   (wire (pts (xy 101.6 111.76) (xy 113.03 111.76))
     (stroke (width 0) (type default) (color 0 0 0 0))
@@
     (stroke (width 0) (type default) (color 0 0 0 0))
   )
-  (wire (pts (xy 120.65 101.6) (xy 124.46 101.6))
+  (wire (pts (xy 120.65 101.6) (xy 121.92 101.6))
     (stroke (width 0) (type default) (color 0 0 0 0))
   )
@@
     (stroke (width 0) (type default) (color 0 0 0 0))
   )
+  (wire (pts (xy 121.92 97.79) (xy 121.92 101.6))
+    (stroke (width 0) (type default) (color 0 0 0 0))
+  )
+  (wire (pts (xy 121.92 64.77) (xy 121.92 68.58))
+    (stroke (width 0) (type default) (color 0 0 0 0))
+  )
   (wire (pts (xy 154.94 87.63) (xy 166.37 87.63))
     (stroke (width 0) (type default) (color 0 0 0 0))
@@
     (stroke (width 0) (type default) (color 0 0 0 0))
   )
-  (wire (pts (xy 124.46 68.58) (xy 133.35 68.58))
-    (stroke (width 0) (type default) (color 0 0 0 0))
-  )
   (wire (pts (xy 113.03 114.3) (xy 113.03 111.76))
     (stroke (width 0) (type default) (color 0 0 0 0))
@@
     (stroke (width 0) (type default) (color 0 0 0 0))
   )
-  (wire (pts (xy 120.65 68.58) (xy 124.46 68.58))
+  (wire (pts (xy 120.65 68.58) (xy 121.92 68.58))
     (stroke (width 0) (type default) (color 0 0 0 0))
   )
@@
     (effects (font (size 1.27 1.27)) (justify left bottom))
   )
-  (text "Due to the diodes, output is\nactually less than 3.3V."
+  (text "Due to the diodes, output is\nactually less than 3.3V.\nIf the host provides 3.3V, that\nis always preferred."
     (at 173.99 80.01 0)
     (effects (font (size 1.27 1.27)) (justify left bottom))
@@
     (pin "2")
   )
+  (symbol (lib_id "Connector:TestPoint") (at 121.92 64.77 0) (unit 1)
+    (in_bom yes) (on_board yes)
+    (property "Reference" "TP901" (id 0) (at 121.92 55.88 0)
+      (effects (font (size 1.27 1.27)) (justify left))
+    )
+    (property "Value" "HLDO" (id 1) (at 121.92 58.42 0)
+      (effects (font (size 1.27 1.27)) (justify left))
+    )
+    (property "Footprint" "TestPoint:TestPoint_Pad_D2.0mm" (id 2) (at 127 64.77 0)
+      (effects (font (size 1.27 1.27)) hide)
+    )
+    (property "Datasheet" "~" (id 3) (at 127 64.77 0)
+      (effects (font (size 1.27 1.27)) hide)
+    )
+    (pin "1")
+  )
   (symbol (lib_id "power:PWR_FLAG") (at 166.37 87.63 180) (unit 1)
     (in_bom yes) (on_board yes) (fields_autoplaced)
@@
       (effects (font (size 1.27 1.27)) hide)
     )
+    (pin "1")
+  )
+  (symbol (lib_id "Connector:TestPoint") (at 121.92 97.79 0) (unit 1)
+    (in_bom yes) (on_board yes)
+    (property "Reference" "TP902" (id 0) (at 121.92 88.9 0)
+      (effects (font (size 1.27 1.27)) (justify left))
+    )
+    (property "Value" "LLDO" (id 1) (at 121.92 91.44 0)
+      (effects (font (size 1.27 1.27)) (justify left))
+    )
+    (property "Footprint" "TestPoint:TestPoint_Pad_D2.0mm" (id 2) (at 127 97.79 0)
+      (effects (font (size 1.27 1.27)) hide)
+    )
+    (property "Datasheet" "~" (id 3) (at 127 97.79 0)
+      (effects (font (size 1.27 1.27)) hide)
+    )
