File: supercap.kicad_sch (KiCad schematic)
At the start: 2 parts

Commit message: SH-RPi v2 schematic design
Parts:
- removed C309: (no value), symbol Device:C_Polarized
- removed C310: (no value), symbol Device:C
- added C1001, C1002, C1003: 100nF, symbol Device:C
- added C1004, C1005, C1006: CAS SCAP 3.0V20F, symbol Device:C_Polarized
- added D1001, D1002, D1003: B5819W SL, Diode_SMD:D_SOD-123, symbol Device:D_Schottky
- added Q1001, Q1002, Q1003: SS8050, Package_TO_SOT_SMD:SOT-23, symbol Transistor_BJT:MMBT5551L
- added R1001, R1002, R1003: 220k, symbol Device:R
- added R1004, R1006, R1008, R1011, R1013, R1015: 2M, symbol Device:R
- added R1005, R1007, R1009: 1.8M, symbol Device:R
- added R1010, R1012, R1014: 2.2M, symbol Device:R
- added U1001, U1002, U1003: LMV321-TR, Package_TO_SOT_SMD:SOT-23-5, symbol Amplifier_Operational:LMV321
Connections:
- net GND: now also C1003.2, C1006.2, D1003.2 (A), Q1003.2 (E), R1003.2, R1009.2, R1015.2, U1003.2 (V-)
- net Vcap: now also C1001.1, C1004.1, D1001.1 (K), Q1001.3 (C), R1001.1, R1004.1, R1010.1, U1001.5 (V+)
- new net: R1006.2, R1007.1, U1002.1 (+)
- new net: C1002.2, C1003.1, C1005.2, C1006.1, D1002.2 (A), D1003.1 (K), Q1002.2 (E), Q1003.3 (C), R1008.1, R1013.2, U1002.2 (V-), U1003.5 (V+)
- new net: R1012.2, R1013.1, U1002.3 (-)
- new net: Q1002.1 (B), U1002.4
- new net: C1001.2, C1002.1, C1004.2, C1005.1, D1001.2 (A), D1002.1 (K), Q1001.2 (E), Q1002.3 (C), R1006.1, R1011.2, U1001.2 (V-), U1002.5 (V+)
- new net: R1010.2, R1011.1, U1001.3 (-)
- new net: R1014.2, R1015.1, U1003.3 (-)
- new net: R1004.2, R1005.1, U1001.1 (+)
- new net: Q1001.1 (B), U1001.4
- new net: R1001.2, R1002.1, R1005.2, R1012.1
- new net: R1002.2, R1003.1, R1007.2, R1014.1
- new net: Q1003.1 (B), U1003.4
- new net: R1008.2, R1009.1, U1003.1 (+)
Other:
- note added: "Balancing circuit modeled after https://www.eevblog.com/forum/renewable-energy/supercapacitor-balancer/"
- note removed: "60F (or thereabouts) supercapacitor, 2.7V, 18x40mm size"

Commit message: WIP: Assign footprints and LCSC part numbers
Parts:
- C1001, C1002, C1003: footprint (none) -> Capacitor_SMD:C_0402_1005Metric; LCSC (none) -> C307331
- C1004, C1005, C1006: footprint (none) -> SH-RPi:CP_Radial_D12.0mm_H25.0mm_P5.30mm_Horizontal
Changed lines of the file:
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@@
       (effects (font (size 1.27 1.27)) (justify left))
     )
-    (property "Footprint" "" (id 2) (at 126.6952 96.52 0)
+    (property "Footprint" "SH-RPi:CP_Radial_D12.0mm_H25.0mm_P5.30mm_Horizontal" (id 2) (at 126.6952 96.52 0)
       (effects (font (size 1.27 1.27)) hide)
     )
@@
       (effects (font (size 1.27 1.27)) (justify left))
     )
-    (property "Footprint" "" (id 2) (at 126.6952 58.42 0)
+    (property "Footprint" "SH-RPi:CP_Radial_D12.0mm_H25.0mm_P5.30mm_Horizontal" (id 2) (at 126.6952 58.42 0)
       (effects (font (size 1.27 1.27)) hide)
     )
@@
       (effects (font (size 1.27 1.27)) (justify left))
     )
-    (property "Footprint" "" (id 2) (at 116.5352 52.07 0)
+    (property "Footprint" "Capacitor_SMD:C_0402_1005Metric" (id 2) (at 116.5352 52.07 0)
       (effects (font (size 1.27 1.27)) hide)
     )
     (property "Datasheet" "~" (id 3) (at 115.57 48.26 0)
+      (effects (font (size 1.27 1.27)) hide)
+    )
+    (property "LCSC" "C307331" (id 4) (at 115.57 48.26 0)
       (effects (font (size 1.27 1.27)) hide)
     )
@@
       (effects (font (size 1.27 1.27)) (justify left))
     )
-    (property "Footprint" "" (id 2) (at 116.5352 90.17 0)
+    (property "Footprint" "Capacitor_SMD:C_0402_1005Metric" (id 2) (at 116.5352 90.17 0)
       (effects (font (size 1.27 1.27)) hide)
     )
@@
       (effects (font (size 1.27 1.27)) hide)
     )
+    (property "LCSC" "C307331" (id 4) (at 115.57 86.36 0)
+      (effects (font (size 1.27 1.27)) hide)
+    )
     (pin "1")
     (pin "2")
@@
       (effects (font (size 1.27 1.27)) (justify left))
     )
-    (property "Footprint" "" (id 2) (at 126.6952 134.62 0)
+    (property "Footprint" "SH-RPi:CP_Radial_D12.0mm_H25.0mm_P5.30mm_Horizontal" (id 2) (at 126.6952 134.62 0)
       (effects (font (size 1.27 1.27)) hide)
     )
@@
       (effects (font (size 1.27 1.27)) (justify left))
     )
-    (property "Footprint" "" (id 2) (at 116.5352 128.27 0)
+    (property "Footprint" "Capacitor_SMD:C_0402_1005Metric" (id 2) (at 116.5352 128.27 0)
       (effects (font (size 1.27 1.27)) hide)
     )
@@
       (effects (font (size 1.27 1.27)) hide)
     )
+    (property "LCSC" "C307331" (id 4) (at 115.57 124.46 0)
+      (effects (font (size 1.27 1.27)) hide)
+    )

Commit message: Assign footprints and part numbers to components
Parts:
- removed R1005, R1007, R1009: 1.8M, symbol Device:R
- added R1005, R1008, R1011: 1.5M, Resistor_SMD:R_0603_1608Metric, symbol Device:R_Small
- added R1006, R1009, R1012: 300k, Resistor_SMD:R_0603_1608Metric, symbol Device:R_Small
- C1001, C1002, C1003: LCSC C307331 -> C1525
- D1001, D1002, D1003: value B5819W SL -> 1N5819WS; LCSC C8598 -> C191023
- R1001, R1002, R1003: footprint (none) -> Resistor_SMD:R_0402_1005Metric; LCSC (none) -> C25767
- R1004: footprint (none) -> Resistor_SMD:R_0603_1608Metric; LCSC (none) -> C22976
- R1007: renamed from R1006; footprint (none) -> Resistor_SMD:R_0603_1608Metric; LCSC (none) -> C22976
- R1010: renamed from R1008; footprint (none) -> Resistor_SMD:R_0603_1608Metric; LCSC (none) -> C22976
- R1013: renamed from R1010; footprint (none) -> Resistor_SMD:R_0603_1608Metric; LCSC (none) -> C22938
- R1014: renamed from R1011; footprint (none) -> Resistor_SMD:R_0603_1608Metric; LCSC (none) -> C22976
- R1015: renamed from R1012; footprint (none) -> Resistor_SMD:R_0603_1608Metric; LCSC (none) -> C22938
- R1016: renamed from R1013; footprint (none) -> Resistor_SMD:R_0603_1608Metric; LCSC (none) -> C22976
- R1017: renamed from R1014; footprint (none) -> Resistor_SMD:R_0603_1608Metric; LCSC (none) -> C22938
- R1018: renamed from R1015; footprint (none) -> Resistor_SMD:R_0603_1608Metric; LCSC (none) -> C22976
Connections:
- net GND: now also R1012.2
- net at R1007.2, U1002.1 (+): now also R1008.1
- net at R1004.2, U1001.1 (+): now also R1005.1
- net at R1001.2, R1002.1, R1015.1: now also R1006.2
- net at R1002.2, R1003.1, R1017.1: now also R1009.2
- net at R1010.2, U1003.1 (+): now also R1011.1
- new net: R1008.2, R1009.1
- new net: R1011.2, R1012.1
- new net: R1005.2, R1006.1

Commit message: WIP: PCB layout
Parts:
- D1001, D1002, D1003: footprint Diode_SMD:D_SOD-123 -> Diode_SMD:D_SOD-323
- R1001, R1002, R1003: value 220k -> 33k; LCSC C25767 -> C25779
- R1004, R1007, R1010, R1014, R1016, R1018: value 2M -> 300k; footprint Resistor_SMD:R_0603_1608Metric -> Resistor_SMD:R_0402_1005Metric; LCSC C22976 -> C25774
- R1005, R1008, R1011: value 1.5M -> 150k; footprint Resistor_SMD:R_0603_1608Metric -> Resistor_SMD:R_0402_1005Metric; LCSC C4172 -> C25755
- R1006, R1009, R1012: value 300k -> 120k; footprint Resistor_SMD:R_0603_1608Metric -> Resistor_SMD:R_0402_1005Metric; LCSC C23024 -> C25750
- R1013, R1015, R1017: value 2.2M -> 330k; footprint Resistor_SMD:R_0603_1608Metric -> Resistor_SMD:R_0402_1005Metric; LCSC C22938 -> C25778
Connections:
- net BO2+: now reaches R1007.2, R1008.1, U1002.1 (+)
- net SC12: now reaches C1002.2, C1003.1, C1005.2, C1006.1, D1002.2 (A), D1003.1 (K), Q1002.2 (E), Q1003.3 (C), R1010.1, R1016.2, U1002.2 (V-), U1003.5 (V+)
- net BO2-: now reaches R1015.2, R1016.1, U1002.3 (-)
- net BO2o: now reaches Q1002.1 (B), U1002.4
- net SC23: now reaches C1001.2, C1002.1, C1004.2, C1005.1, D1001.2 (A), D1002.1 (K), Q1001.2 (E), Q1002.3 (C), R1007.1, R1014.2, U1001.2 (V-), U1002.5 (V+)
- net BO3-: now reaches R1013.2, R1014.1, U1001.3 (-)
- net BO1-: now reaches R1017.2, R1018.1, U1003.3 (-)
- net BO3+: now reaches R1004.2, R1005.1, U1001.1 (+)
- net BO3o: now reaches Q1001.1 (B), U1001.4
- net SC23R: now reaches R1001.2, R1002.1, R1006.2, R1015.1
- net SC12R: now reaches R1002.2, R1003.1, R1009.2, R1017.1
- net BO1o: now reaches Q1003.1 (B), U1003.4
- net BO1+: now reaches R1010.2, R1011.1, U1003.1 (+)

Commit message: Finish PCB routing
Changed lines of the file:
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@@
     (effects (font (size 1.27 1.27)) (justify right bottom))
   )
-  (hierarchical_label "Vcap" (shape input) (at 35.56 36.83 180)
+  (hierarchical_label "Vcap" (shape bidirectional) (at 35.56 36.83 180)
     (effects (font (size 1.27 1.27)) (justify right))
   )
