File: control_mcu.kicad_sch (KiCad schematic)
At the start: 23 parts, among them J401 Conn_02x02_Top_Bottom, J402 Conn_02x06_Odd_Even, U401 ATtiny1616-MNR

Commit message: Redesign the EMI input filter
Parts:
- J401: LCSC (none) -> C492419
Changed lines of the file:
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@@
   (symbol (lib_id "power:GND") (at 148.59 104.14 0) (unit 1)
     (in_bom yes) (on_board yes)
-    (property "Reference" "#PWR0414" (id 0) (at 148.59 110.49 0)
+    (property "Reference" "#PWR0413" (id 0) (at 148.59 110.49 0)
       (effects (font (size 1.27 1.27)) hide)
     )
@@
   (symbol (lib_id "power:GND") (at 165.1 48.26 0) (unit 1)
     (in_bom yes) (on_board yes)
-    (property "Reference" "#PWR0415" (id 0) (at 165.1 54.61 0)
+    (property "Reference" "#PWR0414" (id 0) (at 165.1 54.61 0)
       (effects (font (size 1.27 1.27)) hide)
     )
@@
   (symbol (lib_id "power:GND") (at 64.77 130.81 0) (unit 1)
     (in_bom yes) (on_board yes)
-    (property "Reference" "#PWR0408" (id 0) (at 64.77 137.16 0)
+    (property "Reference" "#PWR0407" (id 0) (at 64.77 137.16 0)
       (effects (font (size 1.27 1.27)) hide)
     )
@@
   (symbol (lib_id "power:GND") (at 80.01 130.81 0) (unit 1)
     (in_bom yes) (on_board yes)
-    (property "Reference" "#PWR0412" (id 0) (at 80.01 137.16 0)
+    (property "Reference" "#PWR0411" (id 0) (at 80.01 137.16 0)
       (effects (font (size 1.27 1.27)) hide)
     )
@@
   (symbol (lib_id "power:GND") (at 71.12 182.88 0) (unit 1)
     (in_bom yes) (on_board yes)
-    (property "Reference" "#PWR0409" (id 0) (at 71.12 189.23 0)
+    (property "Reference" "#PWR0408" (id 0) (at 71.12 189.23 0)
       (effects (font (size 1.27 1.27)) hide)
     )
@@
   (symbol (lib_id "power:GND") (at 58.42 45.72 0) (unit 1)
     (in_bom yes) (on_board yes)
-    (property "Reference" "#PWR0406" (id 0) (at 58.42 52.07 0)
+    (property "Reference" "#PWR0405" (id 0) (at 58.42 52.07 0)
       (effects (font (size 1.27 1.27)) hide)
     )
@@
   (symbol (lib_id "power:GND") (at 73.66 45.72 0) (unit 1)
     (in_bom yes) (on_board yes)
-    (property "Reference" "#PWR0410" (id 0) (at 73.66 52.07 0)
+    (property "Reference" "#PWR0409" (id 0) (at 73.66 52.07 0)
       (effects (font (size 1.27 1.27)) hide)
     )
@@
   (symbol (lib_id "power:+3V3") (at 175.26 48.26 0) (unit 1)
     (in_bom yes) (on_board yes) (fields_autoplaced)
-    (property "Reference" "#PWR0416" (id 0) (at 175.26 52.07 0)
+    (property "Reference" "#PWR0415" (id 0) (at 175.26 52.07 0)
       (effects (font (size 1.27 1.27)) hide)
     )
@@
   (symbol (lib_id "power:+3V3") (at 148.59 30.48 0) (unit 1)
     (in_bom yes) (on_board yes) (fields_autoplaced)
-    (property "Reference" "#PWR0413" (id 0) (at 148.59 34.29 0)
+    (property "Reference" "#PWR0412" (id 0) (at 148.59 34.29 0)
       (effects (font (size 1.27 1.27)) hide)
     )
@@
   (symbol (lib_id "power:GND") (at 241.3 38.1 0) (unit 1)
     (in_bom yes) (on_board yes)
-    (property "Reference" "#PWR0418" (id 0) (at 241.3 44.45 0)
+    (property "Reference" "#PWR0417" (id 0) (at 241.3 44.45 0)
       (effects (font (size 1.27 1.27)) hide)
     )
@@
   (symbol (lib_id "power:GND") (at 232.41 80.01 0) (unit 1)
     (in_bom yes) (on_board yes)
-    (property "Reference" "#PWR0417" (id 0) (at 232.41 86.36 0)
+    (property "Reference" "#PWR0416" (id 0) (at 232.41 86.36 0)
       (effects (font (size 1.27 1.27)) hide)
     )
@@
   (symbol (lib_id "power:GND") (at 265.43 80.01 0) (unit 1)
     (in_bom yes) (on_board yes)
-    (property "Reference" "#PWR0420" (id 0) (at 265.43 86.36 0)
+    (property "Reference" "#PWR0419" (id 0) (at 265.43 86.36 0)
       (effects (font (size 1.27 1.27)) hide)
     )
@@
   (symbol (lib_id "power:+3V3") (at 262.89 71.12 0) (unit 1)
     (in_bom yes) (on_board yes) (fields_autoplaced)
-    (property "Reference" "#PWR0419" (id 0) (at 262.89 74.93 0)
+    (property "Reference" "#PWR0418" (id 0) (at 262.89 74.93 0)
       (effects (font (size 1.27 1.27)) hide)
     )
@@
   (symbol (lib_id "power:GND") (at 73.66 76.2 0) (unit 1)
     (in_bom yes) (on_board yes)
-    (property "Reference" "#PWR0411" (id 0) (at 73.66 82.55 0)
+    (property "Reference" "#PWR0410" (id 0) (at 73.66 82.55 0)
       (effects (font (size 1.27 1.27)) hide)
     )
@@
   (symbol (lib_id "power:GND") (at 58.42 76.2 0) (unit 1)
     (in_bom yes) (on_board yes)
-    (property "Reference" "#PWR0407" (id 0) (at 58.42 82.55 0)
+    (property "Reference" "#PWR0406" (id 0) (at 58.42 82.55 0)
       (effects (font (size 1.27 1.27)) hide)
     )
@@
       (effects (font (size 1.27 1.27)) hide)
     )
+    (property "LCSC" "C492419" (id 4) (at 19.05 48.26 0)
+      (effects (font (size 1.27 1.27)) hide)
+    )
