File: control_mcu.kicad_sch (KiCad schematic)
At the start: 23 parts, among them J401 Conn_02x02_Top_Bottom, J402 Conn_02x06_Odd_Even, U401 ATtiny1616-MNR

Commit message: chore(bom): swap parts for better-stocked equivalents
Re-point LCSC part numbers for the 150k, 470k, 68k, 3.9k, 300k and 7.5k
resistors and the LMV321 op-amp to alternates that are in stock.

D202 changes from MSK340A to MBRA340T3G-FS, an equivalent 3A/40V
Schottky in the same SMA package.

Co-Authored-By: Claude Opus 5 (1M context) <noreply@anthropic.com>
Parts:
- R402: LCSC C25755 -> C93947
Changed lines of the file:
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@@
 			)
 		)
-		(property "LCSC" "C25755"
+		(property "LCSC" "C93947"
 			(at 71.12 163.83 0)
 			(hide yes)
