File: pcb.kicad_sch (KiCad schematic)
At the start: 18 parts

Commit message: SH-RPi v2 schematic design
Parts:
- removed C901, C902, C903, C904, C905, C906, C907, C908, C909, C910, C911, C912, C913, C914: 100nF, Capacitor_SMD:C_0402_1005Metric, symbol Device:C
- removed H901: MountingHole, SH-RPi:MountingHole_3.2mm_no_pad, symbol Mechanical:MountingHole
- renumbered H902 to H601, H903 to H602, H904 to H603
Other:
- note removed: "Decoupling caps"
- note removed: "This mounting hole meant for an optional zip tie support for the supercap"

Commit message: WIP: PCB layout
Parts:
- added H604: MountingHole, SH-RPi:MountingHole_Pi_2.75mm_M2.5, symbol Mechanical:MountingHole
- added P601: HL pictogram, SH-RPi:HL_pictogram_6.3mm, symbol SH-RPi:SilkScreenPicture
- added P602: Hat Labs logo, SH-RPi:Hat_Labs_63.5mm, symbol SH-RPi:SilkScreenPicture
- added P603: OSHW logo, Symbol:OSHW-Logo_11.4x12mm_SilkScreen, symbol SH-RPi:SilkScreenPicture
- added P604: WEEE logo, Symbol:WEEE-Logo_4.2x6mm_SilkScreen, symbol SH-RPi:SilkScreenPicture
- added P605: cc-by logo, SH-RPi:cc-by_5mm, symbol SH-RPi:SilkScreenPicture
- H601, H602, H603: footprint SH-RPi:JlcpcbToolingHole -> SH-RPi:MountingHole_Pi_2.75mm_M2.5
Other:
- note added: "Raspberry Pi mounting holes"
Changed lines of the file:
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@@
     (comment 3 "Sailor Hat for Raspberry Pi is licensed under CC BY 4.0.")
   )
-  (symbol (lib_id "Mechanical:MountingHole") (at 78.74 54.61 0) (unit 1)
-    (in_bom yes) (on_board yes)
-    (property "Reference" "H601" (id 0) (at 81.28 53.4416 0)
+  (text "Raspberry Pi\nmounting holes" (at 50.8 45.72 0)
+    (effects (font (size 1.27 1.27)) (justify left bottom))
+  )
+  (symbol (lib_id "SH-RPi:SilkScreenPicture") (at 162.56 80.01 0) (unit 1)
+    (in_bom yes) (on_board yes) (fields_autoplaced)
+    (property "Reference" "P603" (id 0) (at 168.91 81.2799 0)
       (effects (font (size 1.27 1.27)) (justify left))
     )
-    (property "Value" "MountingHole" (id 1) (at 81.28 55.753 0)
+    (property "Value" "OSHW logo" (id 1) (at 168.91 83.8199 0)
       (effects (font (size 1.27 1.27)) (justify left))
     )
-    (property "Footprint" "SH-RPi:JlcpcbToolingHole" (id 2) (at 78.74 54.61 0)
+    (property "Footprint" "Symbol:OSHW-Logo_11.4x12mm_SilkScreen" (id 2) (at 162.56 80.01 0)
       (effects (font (size 1.27 1.27)) hide)
     )
-    (property "Datasheet" "~" (id 3) (at 78.74 54.61 0)
+    (property "Datasheet" "" (id 3) (at 162.56 80.01 0)
       (effects (font (size 1.27 1.27)) hide)
     )
   )
-  (symbol (lib_id "Mechanical:MountingHole") (at 78.74 63.5 0) (unit 1)
-    (in_bom yes) (on_board yes)
-    (property "Reference" "H602" (id 0) (at 81.28 62.3316 0)
+  (symbol (lib_id "Mechanical:MountingHole") (at 53.34 53.34 0) (unit 1)
+    (in_bom yes) (on_board yes) (fields_autoplaced)
+    (property "Reference" "H601" (id 0) (at 55.88 52.0699 0)
       (effects (font (size 1.27 1.27)) (justify left))
     )
-    (property "Value" "MountingHole" (id 1) (at 81.28 64.643 0)
+    (property "Value" "MountingHole" (id 1) (at 55.88 54.6099 0)
       (effects (font (size 1.27 1.27)) (justify left))
     )
-    (property "Footprint" "SH-RPi:JlcpcbToolingHole" (id 2) (at 78.74 63.5 0)
+    (property "Footprint" "SH-RPi:MountingHole_Pi_2.75mm_M2.5" (id 2) (at 53.34 53.34 0)
       (effects (font (size 1.27 1.27)) hide)
     )
-    (property "Datasheet" "~" (id 3) (at 78.74 63.5 0)
+    (property "Datasheet" "~" (id 3) (at 53.34 53.34 0)
       (effects (font (size 1.27 1.27)) hide)
     )
   )
-  (symbol (lib_id "Mechanical:MountingHole") (at 78.74 72.39 0) (unit 1)
-    (in_bom yes) (on_board yes)
-    (property "Reference" "H603" (id 0) (at 81.28 71.2216 0)
+  (symbol (lib_id "Mechanical:MountingHole") (at 53.34 60.96 0) (unit 1)
+    (in_bom yes) (on_board yes) (fields_autoplaced)
+    (property "Reference" "H602" (id 0) (at 55.88 59.6899 0)
       (effects (font (size 1.27 1.27)) (justify left))
     )
-    (property "Value" "MountingHole" (id 1) (at 81.28 73.533 0)
+    (property "Value" "MountingHole" (id 1) (at 55.88 62.2299 0)
       (effects (font (size 1.27 1.27)) (justify left))
     )
-    (property "Footprint" "SH-RPi:JlcpcbToolingHole" (id 2) (at 78.74 72.39 0)
+    (property "Footprint" "SH-RPi:MountingHole_Pi_2.75mm_M2.5" (id 2) (at 53.34 60.96 0)
       (effects (font (size 1.27 1.27)) hide)
     )
-    (property "Datasheet" "~" (id 3) (at 78.74 72.39 0)
+    (property "Datasheet" "~" (id 3) (at 53.34 60.96 0)
       (effects (font (size 1.27 1.27)) hide)
     )
+  )
+  (symbol (lib_id "SH-RPi:SilkScreenPicture") (at 162.56 107.95 0) (unit 1)
+    (in_bom yes) (on_board yes) (fields_autoplaced)
+    (property "Reference" "P605" (id 0) (at 168.91 109.2199 0)
+      (effects (font (size 1.27 1.27)) (justify left))
+    )
+    (property "Value" "cc-by logo" (id 1) (at 168.91 111.7599 0)
+      (effects (font (size 1.27 1.27)) (justify left))
+    )
+    (property "Footprint" "SH-RPi:cc-by_5mm" (id 2) (at 162.56 107.95 0)
+      (effects (font (size 1.27 1.27)) hide)
+    )
+    (property "Datasheet" "" (id 3) (at 162.56 107.95 0)
+      (effects (font (size 1.27 1.27)) hide)
+    )
+  )
+  (symbol (lib_id "SH-RPi:SilkScreenPicture") (at 162.56 93.98 0) (unit 1)
+    (in_bom yes) (on_board yes) (fields_autoplaced)
+    (property "Reference" "P604" (id 0) (at 168.91 95.2499 0)
+      (effects (font (size 1.27 1.27)) (justify left))
+    )
+    (property "Value" "WEEE logo" (id 1) (at 168.91 97.7899 0)
+      (effects (font (size 1.27 1.27)) (justify left))
+    )
+    (property "Footprint" "Symbol:WEEE-Logo_4.2x6mm_SilkScreen" (id 2) (at 162.56 93.98 0)
+      (effects (font (size 1.27 1.27)) hide)
+    )
+    (property "Datasheet" "" (id 3) (at 162.56 93.98 0)
+      (effects (font (size 1.27 1.27)) hide)
+    )
+  )
+  (symbol (lib_id "SH-RPi:SilkScreenPicture") (at 162.56 52.07 0) (unit 1)
+    (in_bom yes) (on_board yes) (fields_autoplaced)
+    (property "Reference" "P601" (id 0) (at 168.91 53.3399 0)
+      (effects (font (size 1.27 1.27)) (justify left))
+    )
+    (property "Value" "HL pictogram" (id 1) (at 168.91 55.8799 0)
+      (effects (font (size 1.27 1.27)) (justify left))
+    )
+    (property "Footprint" "SH-RPi:HL_pictogram_6.3mm" (id 2) (at 162.56 52.07 0)
+      (effects (font (size 1.27 1.27)) hide)
+    )
+    (property "Datasheet" "" (id 3) (at 162.56 52.07 0)
+      (effects (font (size 1.27 1.27)) hide)
+    )
+  )
+  (symbol (lib_id "Mechanical:MountingHole") (at 53.34 76.2 0) (unit 1)
+    (in_bom yes) (on_board yes) (fields_autoplaced)
+    (property "Reference" "H604" (id 0) (at 55.88 74.9299 0)
+      (effects (font (size 1.27 1.27)) (justify left))
+    )
+    (property "Value" "MountingHole" (id 1) (at 55.88 77.4699 0)
+      (effects (font (size 1.27 1.27)) (justify left))
+    )
+    (property "Footprint" "SH-RPi:MountingHole_Pi_2.75mm_M2.5" (id 2) (at 53.34 76.2 0)
+      (effects (font (size 1.27 1.27)) hide)
+    )
+    (property "Datasheet" "~" (id 3) (at 53.34 76.2 0)
+      (effects (font (size 1.27 1.27)) hide)
+    )
+  )
+  (symbol (lib_id "Mechanical:MountingHole") (at 53.34 68.58 0) (unit 1)
+    (in_bom yes) (on_board yes) (fields_autoplaced)
+    (property "Reference" "H603" (id 0) (at 55.88 67.3099 0)
+      (effects (font (size 1.27 1.27)) (justify left))
+    )
+    (property "Value" "MountingHole" (id 1) (at 55.88 69.8499 0)
+      (effects (font (size 1.27 1.27)) (justify left))
+    )
+    (property "Footprint" "SH-RPi:MountingHole_Pi_2.75mm_M2.5" (id 2) (at 53.34 68.58 0)
+      (effects (font (size 1.27 1.27)) hide)
+    )
+    (property "Datasheet" "~" (id 3) (at 53.34 68.58 0)
+      (effects (font (size 1.27 1.27)) hide)
+    )
+  )
+  (symbol (lib_id "SH-RPi:SilkScreenPicture") (at 162.56 66.04 0) (unit 1)
+    (in_bom yes) (on_board yes) (fields_autoplaced)
+    (property "Reference" "P602" (id 0) (at 168.91 67.3099 0)
+      (effects (font (size 1.27 1.27)) (justify left))
+    )
+    (property "Value" "Hat Labs logo" (id 1) (at 168.91 69.8499 0)
+      (effects (font (size 1.27 1.27)) (justify left))
+    )
+    (property "Footprint" "SH-RPi:Hat_Labs_63.5mm" (id 2) (at 162.56 66.04 0)
+      (effects (font (size 1.27 1.27)) hide)
+    )
+    (property "Datasheet" "" (id 3) (at 162.56 66.04 0)
+      (effects (font (size 1.27 1.27)) hide)
+    )

Commit message: Remove silk screen graphics from the BOM
Parts:
- P601, P602, P603, P604, P605: now left out of the parts list
Changed lines of the file:
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@@
   )
   (symbol (lib_id "SH-RPi:SilkScreenPicture") (at 162.56 80.01 0) (unit 1)
-    (in_bom yes) (on_board yes) (fields_autoplaced)
+    (in_bom no) (on_board yes) (fields_autoplaced)
     (property "Reference" "P603" (id 0) (at 168.91 81.2799 0)
       (effects (font (size 1.27 1.27)) (justify left))
@@
   )
   (symbol (lib_id "SH-RPi:SilkScreenPicture") (at 162.56 107.95 0) (unit 1)
-    (in_bom yes) (on_board yes) (fields_autoplaced)
+    (in_bom no) (on_board yes) (fields_autoplaced)
     (property "Reference" "P605" (id 0) (at 168.91 109.2199 0)
       (effects (font (size 1.27 1.27)) (justify left))
@@
   )
   (symbol (lib_id "SH-RPi:SilkScreenPicture") (at 162.56 93.98 0) (unit 1)
-    (in_bom yes) (on_board yes) (fields_autoplaced)
+    (in_bom no) (on_board yes) (fields_autoplaced)
     (property "Reference" "P604" (id 0) (at 168.91 95.2499 0)
       (effects (font (size 1.27 1.27)) (justify left))
@@
   )
   (symbol (lib_id "SH-RPi:SilkScreenPicture") (at 162.56 52.07 0) (unit 1)
-    (in_bom yes) (on_board yes) (fields_autoplaced)
+    (in_bom no) (on_board yes) (fields_autoplaced)
     (property "Reference" "P601" (id 0) (at 168.91 53.3399 0)
       (effects (font (size 1.27 1.27)) (justify left))
@@
   )
   (symbol (lib_id "SH-RPi:SilkScreenPicture") (at 162.56 66.04 0) (unit 1)
-    (in_bom yes) (on_board yes) (fields_autoplaced)
+    (in_bom no) (on_board yes) (fields_autoplaced)
     (property "Reference" "P602" (id 0) (at 168.91 67.3099 0)
       (effects (font (size 1.27 1.27)) (justify left))
