File: pcb.kicad_sch (KiCad schematic)
At the start: 9 parts, among them P601 HL pictogram, P602 Hat Labs logo, P603 OSHW logo, P604 WEEE logo, P605 cc-by logo

Commit message: v2.0.0
Parts:
- added P606: CE logo, Symbol:CE-Logo_8.5x6mm_SilkScreen, symbol SH-RPi:SilkScreenPicture
- renumbered P605 to P604, P604 to P605
Other:
- moved on the sheet: P604, P605
Changed lines of the file:
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@@
   (title_block
     (title "Sailor Hat for Raspberry Pi")
-    (date "2023-01-28")
-    (rev "v2.0.0-a4")
+    (date "2023-02-12")
+    (rev "v2.0.0")
     (company "Hat Labs Ltd")
     (comment 1 "https://creativecommons.org/licenses/by/4.0")
@@
     )
   )
+  (symbol (lib_id "SH-RPi:SilkScreenPicture") (at 162.56 93.98 0) (unit 1)
+    (in_bom no) (on_board yes) (fields_autoplaced)
+    (property "Reference" "P604" (id 0) (at 168.91 95.2499 0)
+      (effects (font (size 1.27 1.27)) (justify left))
+    )
+    (property "Value" "cc-by logo" (id 1) (at 168.91 97.7899 0)
+      (effects (font (size 1.27 1.27)) (justify left))
+    )
+    (property "Footprint" "SH-RPi:cc-by_5mm" (id 2) (at 162.56 93.98 0)
+      (effects (font (size 1.27 1.27)) hide)
+    )
+    (property "Datasheet" "" (id 3) (at 162.56 93.98 0)
+      (effects (font (size 1.27 1.27)) hide)
+    )
+  )
+  (symbol (lib_id "SH-RPi:SilkScreenPicture") (at 162.56 121.92 0) (unit 1)
+    (in_bom no) (on_board yes) (fields_autoplaced)
+    (property "Reference" "P606" (id 0) (at 168.91 123.1899 0)
+      (effects (font (size 1.27 1.27)) (justify left))
+    )
+    (property "Value" "CE logo" (id 1) (at 168.91 125.7299 0)
+      (effects (font (size 1.27 1.27)) (justify left))
+    )
+    (property "Footprint" "Symbol:CE-Logo_8.5x6mm_SilkScreen" (id 2) (at 162.56 121.92 0)
+      (effects (font (size 1.27 1.27)) hide)
+    )
+    (property "Datasheet" "" (id 3) (at 162.56 121.92 0)
+      (effects (font (size 1.27 1.27)) hide)
+    )
+  )
   (symbol (lib_id "SH-RPi:SilkScreenPicture") (at 162.56 107.95 0) (unit 1)
     (in_bom no) (on_board yes) (fields_autoplaced)
@@
       (effects (font (size 1.27 1.27)) (justify left))
     )
-    (property "Value" "cc-by logo" (id 1) (at 168.91 111.7599 0)
+    (property "Value" "WEEE logo" (id 1) (at 168.91 111.7599 0)
       (effects (font (size 1.27 1.27)) (justify left))
     )
-    (property "Footprint" "SH-RPi:cc-by_5mm" (id 2) (at 162.56 107.95 0)
+    (property "Footprint" "Symbol:WEEE-Logo_4.2x6mm_SilkScreen" (id 2) (at 162.56 107.95 0)
       (effects (font (size 1.27 1.27)) hide)
     )
@@
       (effects (font (size 1.27 1.27)) hide)
     )
-  )
-  (symbol (lib_id "SH-RPi:SilkScreenPicture") (at 162.56 93.98 0) (unit 1)
-    (in_bom no) (on_board yes) (fields_autoplaced)
-    (property "Reference" "P604" (id 0) (at 168.91 95.2499 0)
-      (effects (font (size 1.27 1.27)) (justify left))
-    )
-    (property "Value" "WEEE logo" (id 1) (at 168.91 97.7899 0)
-      (effects (font (size 1.27 1.27)) (justify left))
-    )
-    (property "Footprint" "Symbol:WEEE-Logo_4.2x6mm_SilkScreen" (id 2) (at 162.56 93.98 0)
-      (effects (font (size 1.27 1.27)) hide)
-    )
-    (property "Datasheet" "" (id 3) (at 162.56 93.98 0)
-      (effects (font (size 1.27 1.27)) hide)
-    )
