File: buck_stage_2.kicad_sch (KiCad schematic)
At the start: 15 parts, among them U201 RT6365

Commit message: Update stage 2 output caps
Parts:
- C204, C205: footprint Capacitor_SMD:C_0805_2012Metric -> Capacitor_SMD:C_1210_3225Metric; LCSC C16780 -> (none)
Changed lines of the file:
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@@
       (effects (font (size 1.27 1.27)) (justify left))
     )
-    (property "Footprint" "Capacitor_SMD:C_0805_2012Metric" (id 2) (at 178.1048 143.51 0)
+    (property "Footprint" "Capacitor_SMD:C_1210_3225Metric" (id 2) (at 178.1048 143.51 0)
       (effects (font (size 1.27 1.27)) hide)
     )
@@
       (effects (font (size 1.27 1.27)) hide)
     )
-    (property "LCSC" "C16780" (id 5) (at 179.07 139.7 0)
+    (property "LCSC" "" (id 5) (at 179.07 139.7 0)
       (effects (font (size 1.27 1.27)) hide)
     )
@@
       (effects (font (size 1.27 1.27)) (justify left))
     )
-    (property "Footprint" "Capacitor_SMD:C_0805_2012Metric" (id 2) (at 167.9448 139.7 0)
+    (property "Footprint" "Capacitor_SMD:C_1210_3225Metric" (id 2) (at 167.9448 139.7 0)
       (effects (font (size 1.27 1.27)) hide)
     )
@@
       (effects (font (size 1.27 1.27)) hide)
     )
-    (property "LCSC" "C16780" (id 5) (at 168.91 135.89 0)
-      (effects (font (size 1.27 1.27)) hide)
-    )
+    (property "LCSC" "" (id 5) (at 168.91 135.89 0)
+      (effects (font (size 1.27 1.27)) hide)
+    )

Commit message: Pick LCSC part numbers for changed components
Parts:
- C204, C205: LCSC (none) -> C2918513
Changed lines of the file:
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@@
       (effects (font (size 1.27 1.27)) hide)
     )
-    (property "LCSC" "" (id 5) (at 179.07 139.7 0)
+    (property "LCSC" "C2918513" (id 5) (at 179.07 139.7 0)
       (effects (font (size 1.27 1.27)) hide)
     )
@@
       (effects (font (size 1.27 1.27)) hide)
     )
-    (property "LCSC" "" (id 5) (at 168.91 135.89 0)
-      (effects (font (size 1.27 1.27)) hide)
-    )
+    (property "LCSC" "C2918513" (id 5) (at 168.91 135.89 0)
+      (effects (font (size 1.27 1.27)) hide)
+    )

Commit message: Tweak the layout and reroute tracks
Parts:
- C204, C205: value 47uF/6.3V -> 47uF 6.3V
- D202: value SS54 -> SSL54F; LCSC C22452 -> C3033287
Changed lines of the file:
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@@
   (junction (at 146.05 129.54) (diameter 0) (color 0 0 0 0)
   )
+  (junction (at 130.81 160.02) (diameter 0) (color 0 0 0 0)
+  )
+  (junction (at 87.63 129.54) (diameter 0) (color 0 0 0 0)
+  )
   (junction (at 203.2 140.97) (diameter 0) (color 0 0 0 0)
   )
@@
   (junction (at 168.91 129.54) (diameter 0) (color 0 0 0 0)
   )
-  (wire (pts (xy 130.81 157.48) (xy 130.81 163.83))
+  (wire (pts (xy 130.81 157.48) (xy 130.81 160.02))
     (stroke (width 0) (type default) (color 0 0 0 0))
   )
@@
     (stroke (width 0) (type default) (color 0 0 0 0))
   )
-  (wire (pts (xy 80.01 129.54) (xy 102.87 129.54))
+  (wire (pts (xy 130.81 160.02) (xy 130.81 163.83))
+    (stroke (width 0) (type default) (color 0 0 0 0))
+  )
+  (wire (pts (xy 80.01 129.54) (xy 87.63 129.54))
+    (stroke (width 0) (type default) (color 0 0 0 0))
+  )
+  (wire (pts (xy 87.63 129.54) (xy 102.87 129.54))
     (stroke (width 0) (type default) (color 0 0 0 0))
   )
@@
       (effects (font (size 1.27 1.27)) (justify left))
     )
-    (property "Value" "SS54" (id 1) (at 148.082 140.843 90)
+    (property "Value" "SSL54F" (id 1) (at 148.082 140.843 90)
       (effects (font (size 1.27 1.27)) (justify left))
     )
@@
       (effects (font (size 1.27 1.27)) hide)
     )
-    (property "LCSC" "C22452" (id 4) (at 146.05 139.7 0)
+    (property "LCSC" "C3033287" (id 4) (at 146.05 139.7 0)
       (effects (font (size 1.27 1.27)) hide)
     )
@@
       (effects (font (size 1.27 1.27)) (justify left))
     )
-    (property "Value" "47uF/6.3V" (id 1) (at 176.149 140.843 0)
+    (property "Value" "47uF 6.3V" (id 1) (at 176.149 140.843 0)
       (effects (font (size 1.27 1.27)) (justify left))
     )
@@
     (pin "9")
   )
+  (symbol (lib_id "power:PWR_FLAG") (at 87.63 129.54 0) (unit 1)
+    (in_bom yes) (on_board yes) (fields_autoplaced)
+    (property "Reference" "#FLG0201" (id 0) (at 87.63 127.635 0)
+      (effects (font (size 1.27 1.27)) hide)
+    )
+    (property "Value" "PWR_FLAG" (id 1) (at 87.63 124.46 0))
+    (property "Footprint" "" (id 2) (at 87.63 129.54 0)
+      (effects (font (size 1.27 1.27)) hide)
+    )
+    (property "Datasheet" "~" (id 3) (at 87.63 129.54 0)
+      (effects (font (size 1.27 1.27)) hide)
+    )
+    (pin "1")
+  )
   (symbol (lib_id "Device:D_Small") (at 133.35 118.11 90) (unit 1)
     (in_bom yes) (on_board yes)
@@
       (effects (font (size 1.27 1.27)) (justify left))
     )
-    (property "Value" "47uF/6.3V" (id 1) (at 165.989 137.033 0)
+    (property "Value" "47uF 6.3V" (id 1) (at 165.989 137.033 0)
       (effects (font (size 1.27 1.27)) (justify left))
     )
@@
     (pin "2")
   )
+  (symbol (lib_id "power:PWR_FLAG") (at 130.81 160.02 270) (unit 1)
+    (in_bom yes) (on_board yes) (fields_autoplaced)
+    (property "Reference" "#FLG0202" (id 0) (at 132.715 160.02 0)
+      (effects (font (size 1.27 1.27)) hide)
+    )
+    (property "Value" "PWR_FLAG" (id 1) (at 134.62 160.0199 90)
+      (effects (font (size 1.27 1.27)) (justify left))
+    )
+    (property "Footprint" "" (id 2) (at 130.81 160.02 0)
+      (effects (font (size 1.27 1.27)) hide)
+    )
+    (property "Datasheet" "~" (id 3) (at 130.81 160.02 0)
+      (effects (font (size 1.27 1.27)) hide)
+    )
+    (pin "1")
+  )
   (symbol (lib_id "power:GND") (at 146.05 147.32 0) (unit 1)
     (in_bom yes) (on_board yes)
@@
   (symbol (lib_id "power:PWR_FLAG") (at 191.77 129.54 0) (unit 1)
     (in_bom yes) (on_board yes) (fields_autoplaced)
-    (property "Reference" "#FLG0201" (id 0) (at 191.77 127.635 0)
-      (effects (font (size 1.27 1.27)) hide)
-    )
+    (property "Reference" "#FLG0203" (id 0) (at 191.77 127.635 0)
+      (effects (font (size 1.27 1.27)) hide)
+    )

Commit message: Add test points, test footprints, GND vias
Parts:
- added TP201: SW2, TestPoint:TestPoint_Pad_D2.0mm, symbol Connector:TestPoint
Connections:
- net SW: now also TP201.1
Changed lines of the file:
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@@
   (junction (at 203.2 129.54) (diameter 0) (color 0 0 0 0)
   )
+  (junction (at 137.16 129.54) (diameter 0) (color 0 0 0 0)
+  )
   (junction (at 191.77 129.54) (diameter 0) (color 0 0 0 0)
   )
@@
     (stroke (width 0) (type default) (color 0 0 0 0))
   )
+  (wire (pts (xy 137.16 129.54) (xy 146.05 129.54))
+    (stroke (width 0) (type default) (color 0 0 0 0))
+  )
   (wire (pts (xy 130.81 137.16) (xy 130.81 144.78))
     (stroke (width 0) (type default) (color 0 0 0 0))
@@
     (stroke (width 0) (type default) (color 0 0 0 0))
   )
-  (wire (pts (xy 125.73 129.54) (xy 146.05 129.54))
+  (wire (pts (xy 125.73 129.54) (xy 137.16 129.54))
     (stroke (width 0) (type default) (color 0 0 0 0))
   )
@@
     (pin "2")
   )
+  (symbol (lib_id "Connector:TestPoint") (at 137.16 129.54 180) (unit 1)
+    (in_bom yes) (on_board yes)
+    (property "Reference" "TP201" (id 0) (at 139.7 131.5719 0)
+      (effects (font (size 1.27 1.27)) (justify right))
+    )
+    (property "Value" "SW2" (id 1) (at 139.7 133.35 0)
+      (effects (font (size 1.27 1.27)) (justify right))
+    )
+    (property "Footprint" "TestPoint:TestPoint_Pad_D2.0mm" (id 2) (at 132.08 129.54 0)
+      (effects (font (size 1.27 1.27)) hide)
+    )
+    (property "Datasheet" "~" (id 3) (at 132.08 129.54 0)
+      (effects (font (size 1.27 1.27)) hide)
+    )
+    (pin "1")
+  )
   (symbol (lib_id "power:+5V") (at 133.35 114.3 0) (unit 1)
