File: SH-RPi.kicad_pcb (KiCad board)
At the start: 4 copper layers, 65 x 56.5 mm, 183 parts, among them J101 Conn_01x02, J301 Conn_01x04, J401 Conn_02x02_Top_Bottom, J402 Conn_02x06_Odd_Even, J501 Raspberry_Pi_2_3, J502 Conn_01x02, J801 Conn_01x03, P601 HL pictogram, P602 Hat Labs logo, P603 OSHW logo, P604 WEEE logo, P605 cc-by logo, Q1001 SS8050, Q1002 SS8050, Q1003 SS8050, Q301 MMBT5551, Q302 MMBT5551, Q303 LBSS84LT1G, U1001 LMV321-TR, U1002 LMV321-TR, U1003 LMV321-TR, U201 RT6365, U301 RT6365, U302 COS1333TR, U303 LMV321-TR, U401 ATtiny1616-MNR, U801 PCF8563T, U901 H7533-1, Y801 X1A000061000200

Commit message: Update passthrough socket footprint to fit in copper area
Routing:
- net +5V: track 148.8 -> 148.1 mm
- net GND: vias 214 -> 213

Commit message: Change stage 1 switching diode due to part availability
Parts:
- D303: value SSL56F -> SS56FL
Changed lines of the file:
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@@
     (descr "Diode SMA (DO-214AC)")
     (tags "Diode SMA (DO-214AC)")
-    (property "LCSC" "C5125733")
+    (property "LCSC" "C122865")
     (property "Sheetfile" "buck_stage_1.kicad_sch")
     (property "Sheetname" "Buck converter stage 1")
@@
       (effects (font (size 1 1) (thickness 0.15)))
     )
-    (fp_text value "SSL56F" (at 0 2.6) (layer "F.Fab") hide
+    (fp_text value "SS56FL" (at 0 2.6) (layer "F.Fab") hide
       (effects (font (size 1 1) (thickness 0.15)))
     )
@@
     (property "Sheetfile" "pcb.kicad_sch")
     (property "Sheetname" "PCB")
-    (attr exclude_from_pos_files)
+    (property "exclude_from_bom" "")
+    (attr exclude_from_pos_files exclude_from_bom)
     (fp_text reference "H601" (at 0 -3.7) (layer "F.SilkS") hide
       (effects (font (size 1 1) (thickness 0.15)))
@@
     (descr "CP, Radial series, Radial, pin pitch=5.00mm, , diameter=10mm, Electrolytic Capacitor")
     (tags "CP Radial series Radial pin pitch 5.00mm  diameter 10mm Electrolytic Capacitor")
+    (property "JLCPCB_IGNORE" "1")
     (property "Sheetfile" "supercap.kicad_sch")
     (property "Sheetname" "Supercapacitor")
@@
     (property "Sheetfile" "pcb.kicad_sch")
     (property "Sheetname" "PCB")
-    (attr exclude_from_pos_files)
+    (property "exclude_from_bom" "")
+    (attr exclude_from_pos_files exclude_from_bom)
     (fp_text reference "H602" (at 0 -3.7) (layer "F.SilkS") hide
       (effects (font (size 1 1) (thickness 0.15)))
@@
     (property "Sheetfile" "pcb.kicad_sch")
     (property "Sheetname" "PCB")
-    (attr exclude_from_pos_files)
+    (property "exclude_from_bom" "")
+    (attr exclude_from_pos_files exclude_from_bom)
     (fp_text reference "H604" (at 0 -3.7) (layer "F.SilkS") hide
       (effects (font (size 1 1) (thickness 0.15)))
@@
     (descr "CP, Radial series, Radial, pin pitch=5.00mm, , diameter=10mm, Electrolytic Capacitor")
     (tags "CP Radial series Radial pin pitch 5.00mm  diameter 10mm Electrolytic Capacitor")
+    (property "JLCPCB_IGNORE" "1")
     (property "Sheetfile" "supercap.kicad_sch")
     (property "Sheetname" "Supercapacitor")
@@
     (property "Sheetfile" "pcb.kicad_sch")
     (property "Sheetname" "PCB")
-    (attr exclude_from_pos_files)
+    (property "exclude_from_bom" "")
+    (attr exclude_from_pos_files exclude_from_bom)
     (fp_text reference "H603" (at 0 -3.7) (layer "F.SilkS") hide
       (effects (font (size 1 1) (thickness 0.15)))
@@
     (descr "CP, Radial series, Radial, pin pitch=5.00mm, , diameter=10mm, Electrolytic Capacitor")
     (tags "CP Radial series Radial pin pitch 5.00mm  diameter 10mm Electrolytic Capacitor")
+    (property "JLCPCB_IGNORE" "1")
     (property "Sheetfile" "supercap.kicad_sch")
     (property "Sheetname" "Supercapacitor")

Commit message: Fix J301 part number
Parts:
- J301: value Conn_01x04 -> Conn_02x02
Changed lines of the file:
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@@
     (descr "Through hole straight pin header, 2x02, 2.54mm pitch, double rows")
     (tags "Through hole pin header THT 2x02 2.54mm double row")
-    (property "LCSC" "C152150")
+    (property "LCSC" "C492419")
     (property "Sheetfile" "buck_stage_1.kicad_sch")
     (property "Sheetname" "Buck converter stage 1")
@@
       (effects (font (size 1 1) (thickness 0.15)))
     )
-    (fp_text value "Conn_01x04" (at 1.27 4.87) (layer "F.Fab") hide
+    (fp_text value "Conn_02x02" (at 1.27 4.87) (layer "F.Fab") hide
       (effects (font (size 1 1) (thickness 0.15)))
     )

Commit message: Remove debugging pads
Parts:
- removed C313: CG, Capacitor_SMD:C_0603_1608Metric_Pad1.08x0.95mm_HandSolder
- removed C314: CFB, Capacitor_SMD:C_0603_1608Metric_Pad1.08x0.95mm_HandSolder
- removed C315: Ccomp, Capacitor_SMD:C_0603_1608Metric_Pad1.08x0.95mm_HandSolder
- removed R315: RG, Resistor_SMD:R_0603_1608Metric_Pad0.98x0.95mm_HandSolder
- removed R316: ROut, Resistor_SMD:R_0603_1608Metric_Pad0.98x0.95mm_HandSolder
- removed R317: RFBH, Resistor_SMD:R_0603_1608Metric_Pad0.98x0.95mm_HandSolder
- removed R318: RFBL, Resistor_SMD:R_0603_1608Metric_Pad0.98x0.95mm_HandSolder
- removed R321: Rcomp, Resistor_SMD:R_0603_1608Metric_Pad0.98x0.95mm_HandSolder
Routing:
- net /Buck converter stage 1/FB: track 22.6 -> 10.3 mm, vias 1 -> 0
- net GND: track 119.2 -> 127.4 mm, vias 213 -> 209
- net /Vcap: track 111.7 -> 107.1 mm, vias 14 -> 13
- net /Buck converter stage 1/COMP1_: track 5.48 -> 1.40 mm, vias 2 -> 0
- net +5V: track 148.1 -> 151.6 mm
- net /Buck converter stage 1/COMP1: track 5.82 -> 3.22 mm, vias 1 -> 0
- net /Iin: track 81.3 -> 79.1 mm
- net /Buck converter stage 1/VF-: track 6.42 -> 4.30 mm, vias 1 -> 0
- net /TXD5: track 61.4 -> 63.2 mm
- net /RXD5: track 63.1 -> 64.8 mm
- net unconnected-(J501-Pad40): track 0.00 -> 1.71 mm
- net unconnected-(J501-Pad38): track 0.00 -> 1.71 mm
- net unconnected-(J501-Pad37): track 0.00 -> 1.71 mm
- net unconnected-(J501-Pad36): track 0.00 -> 1.71 mm
- net unconnected-(J501-Pad35): track 0.00 -> 1.71 mm
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
Commit message: Bump board version number
Other:
- board text added: "v2.0.0-a4"
- board text removed: "v2.0.0-a2"
Changed lines of the file:
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@@
   (title_block
     (title "Sailor Hat for Raspberry Pi")
-    (date "2022-12-26")
-    (rev "v2.0.0-a2")
+    (date "2023-01-15")
+    (rev "v2.0.0-a4")
     (company "Hat Labs Ltd")
     (comment 1 "https://creativecommons.org/licenses/by/4.0")
@@
     (effects (font (size 1 1) (thickness 0.15)) (justify right mirror))
   )
-  (gr_text "v2.0.0-a2" (at 85.32 71.5) (layer "B.SilkS")
+  (gr_text "v2.0.0-a4" (at 85.32 71.5) (layer "B.SilkS")
     (effects (font (size 1.2 1.2) (thickness 0.2)) (justify left mirror))
   )
@@
     (effects (font (size 1 1) (thickness 0.2)))
   )
-  (gr_text "v2.0.0-a2" (at 79.1 91.4 90) (layer "F.SilkS")
+  (gr_text "v2.0.0-a4" (at 79.1 91.4 90) (layer "F.SilkS")
     (effects (font (size 1.5 1.5) (thickness 0.3)) (justify left))
   )

Commit message: Replace the GPIO connector with FH-00339
Parts:
- J501: footprint SH-RPi:PassthroughPinSocket_2x40_P2.54mm_Vertical_Bottom -> SH-RPi:PassthroughPinSocket_FH-00339_2x40_P2.54mm_Vertical_Bottom
Routing:
- net +5V: track 151.6 -> 148.9 mm
