File: buck_5V.kicad_sch (KiCad schematic)
At the start: 16 parts, among them U201 RT6365

Commit message: chore(bom): swap parts for better-stocked equivalents
Re-point LCSC part numbers for the 150k, 470k, 68k, 3.9k, 300k and 7.5k
resistors and the LMV321 op-amp to alternates that are in stock.

D202 changes from MSK340A to MBRA340T3G-FS, an equivalent 3A/40V
Schottky in the same SMA package.

Co-Authored-By: Claude Opus 5 (1M context) <noreply@anthropic.com>
Parts:
- D202: value MSK340A -> MBRA340T3G-FS; LCSC C434027 -> C5563736
- R204: LCSC C36871 -> C137947
Changed lines of the file:
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@@
 			)
 		)
-		(property "Value" "MSK340A"
+		(property "Value" "MBRA340T3G-FS"
 			(at 148.082 140.843 90)
 			(show_name no)
@@
 			)
 		)
-		(property "LCSC" "C434027"
+		(property "LCSC" "C5563736"
 			(at 146.05 139.7 0)
 			(hide yes)
@@
 			)
 		)
-		(property "LCSC" "C36871"
+		(property "LCSC" "C137947"
 			(at 203.2 135.89 0)
 			(hide yes)
