File: buck_8.8V.kicad_sch (KiCad schematic)
At the start: 42 parts, among them J301 Conn_02x02, Q301 MMBT5551, Q302 MMBT5551, Q303 LBSS84LT1G, U301 RT6365, U302 COS1333TR, U303 LMV321-TR

Commit message: chore(bom): swap parts for better-stocked equivalents
Re-point LCSC part numbers for the 150k, 470k, 68k, 3.9k, 300k and 7.5k
resistors and the LMV321 op-amp to alternates that are in stock.

D202 changes from MSK340A to MBRA340T3G-FS, an equivalent 3A/40V
Schottky in the same SMA package.

Co-Authored-By: Claude Opus 5 (1M context) <noreply@anthropic.com>
Parts:
- R304: LCSC C306602 -> C25774
- R307: LCSC C36871 -> C137947
- R312: LCSC C25790 -> C137976
- R315: LCSC C25918 -> C137934
- R316: LCSC C51721 -> C131467
- U303: LCSC C362273 -> C3014306
Changed lines of the file:
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@@
 			)
 		)
-		(property "LCSC" "C25790"
+		(property "LCSC" "C137976"
 			(at 172.72 128.27 0)
 			(hide yes)
@@
 			)
 		)
-		(property "LCSC" "C36871"
+		(property "LCSC" "C137947"
 			(at 91.44 149.86 0)
 			(hide yes)
@@
 			)
 		)
-		(property "LCSC" "C362273"
+		(property "LCSC" "C3014306"
 			(at 167.64 64.77 0)
 			(hide yes)
@@
 			)
 		)
-		(property "LCSC" "C51721"
+		(property "LCSC" "C131467"
 			(at 256.54 71.12 0)
 			(hide yes)
@@
 			)
 		)
-		(property "LCSC" "C306602"
+		(property "LCSC" "C25774"
 			(at 83.82 125.73 0)
 			(hide yes)
@@
 			)
 		)
-		(property "LCSC" "C25918"
+		(property "LCSC" "C137934"
 			(at 248.92 71.12 0)
 			(hide yes)
